File: avionics_board/SD_CARD.sch (KiCad schematic (older format))
At the start: 10 parts, among them J1 Micro_SD_Card_Latching

Commit message: Removed unecessary footprint lib
Parts:
- J1: footprint avionics_board:microSD_HC_Molex_0472192001 -> footprint_custom:microSD_HC_Molex_0472192001
Changed lines of the file:
@@
 F 0 "J1" H 7575 4392 50  0000 C CNN
 F 1 "Micro_SD_Card_Latching" H 7575 4301 50  0000 C CNN
-F 2 "avionics_board:microSD_HC_Molex_0472192001" H 8775 3975 50  0001 C CNN
+F 2 "footprint_custom:microSD_HC_Molex_0472192001" H 8775 3975 50  0001 C CNN
 F 3 "https://www.molex.com/pdm_docs/sd/472192001_sd.pdf" H 7625 3675 50  0001 C CNN
 F 4 "0472192001" H 7625 2875 50  0001 C CNN "Mfr. #"

Commit message: Progress on EPS
Other:
- note added: "I haven't found the proper spec regarding bypass caps\nForums suggest a 45uF and a smaller cap as well. \n\nhttp://elm-chan.org/docs/mmc/mmc_e.html\n\nIt doesn't seem like one is always necessary. \n\nIf size constrains, go with small cap only"
- note removed: "I haven't found the proper spec regarding bypass caps\nForums suggest ~45uF and a smaller cap as well. \n\nhttp://elm-chan.org/docs/mmc/mmc_e.html\n\nIt doesn't seem like one is always necessary. \n\nIf size constrains, go with small cap only"
Changed lines of the file:
@@
 Layout Note: Decoupling\n
 Text Notes 1425 7000 0    39   ~ 0
-I haven't found the proper spec regarding bypass caps\nForums suggest ~45uF and a smaller cap as well. \n\nhttp://elm-chan.org/docs/mmc/mmc_e.html\n\nIt doesn't seem like one is always necessary. \n\nIf size constrains, go with small cap only
+I haven't found the proper spec regarding bypass caps\nForums suggest a 45uF and a smaller cap as well. \n\nhttp://elm-chan.org/docs/mmc/mmc_e.html\n\nIt doesn't seem like one is always necessary. \n\nIf size constrains, go with small cap only
 $Comp
 L Device:C C?
