File: avionics_board/CAN_TRANSCEIVER.sch (KiCad schematic (older format))
At the start: 11 parts, among them U8 SN65HVD230

Commit message: Essentially done with EPS schematic
Parts:
- R41: Mfr. # RMCF0603JG100K -> RMCF0603FT100K; Order https://www.digikey.com/product-detail/en/stackpole-electro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 -> https://www.digikey.com/en/products/detail/stackpole-electr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
Changed lines of the file:
@@
 $Descr A 11000 8500
 encoding utf-8
-Sheet 32 39
+Sheet 30 39
 Title "CAN Transceiver"
 Date "2020-05-25"
@@
 F 2 "Resistor_SMD:R_0603_1608Metric_Pad1.05x0.95mm_HandSolder" V 3930 3000 50  0001 C CNN
 F 3 "~" H 4000 3000 50  0001 C CNN
-F 4 "RMCF0603JG100K" H 4000 3000 50  0001 C CNN "Mfr. #"
-F 5 "https://www.digikey.com/product-detail/en/stackpole-electronics-inc/RMCF0603JG100K/RMCF0603JG100KCT-ND/4425127" H 4000 3000 50  0001 C CNN "Order"
+F 4 "RMCF0603FT100K" H 4000 3000 50  0001 C CNN "Mfr. #"
+F 5 "https://www.digikey.com/en/products/detail/stackpole-electronics-inc/RMCF0603FT100K/1761112" H 4000 3000 50  0001 C CNN "Order"
 	1    4000 3000
 	1    0    0    -1

Commit message: Update Avionics part names to match KiCad update. Update Avionics board to use new interboard connector
Parts:
- C38, C39: footprint Capacitor_SMD:C_0603_1608Metric_Pad1.05x0.95mm_HandSolder -> Capacitor_SMD:C_0603_1608Metric_Pad1.08x0.95mm_HandSolder
- R35, R36, R37, R38, R39, R40, R41: footprint Resistor_SMD:R_0603_1608Metric_Pad1.05x0.95mm_HandSolder -> Resistor_SMD:R_0603_1608Metric_Pad0.98x0.95mm_HandSolder
Changed lines of the file:
@@
 $Descr A 11000 8500
 encoding utf-8
-Sheet 30 39
+Sheet 21 23
 Title "CAN Transceiver"
 Date "2020-05-25"
@@
 F 0 "C38" H 2515 6846 50  0000 L CNN
 F 1 "0.1uF" H 2515 6755 50  0000 L CNN
-F 2 "Capacitor_SMD:C_0603_1608Metric_Pad1.05x0.95mm_HandSolder" H 2438 6650 50  0001 C CNN
+F 2 "Capacitor_SMD:C_0603_1608Metric_Pad1.08x0.95mm_HandSolder" H 2438 6650 50  0001 C CNN
 F 3 "~" H 2400 6800 50  0001 C CNN
 F 4 "25V" H 2400 6800 50  0001 C CNN "Voltage"
@@
 F 0 "R36" V 4368 3225 50  0000 C CNN
 F 1 "0" V 4459 3225 50  0000 C CNN
-F 2 "Resistor_SMD:R_0603_1608Metric_Pad1.05x0.95mm_HandSolder" V 4505 3225 50  0001 C CNN
+F 2 "Resistor_SMD:R_0603_1608Metric_Pad0.98x0.95mm_HandSolder" V 4505 3225 50  0001 C CNN
 F 3 "~" H 4575 3225 50  0001 C CNN
 F 4 "RK73Z1JTTD" H 4575 3225 50  0001 C CNN "Mfr. #"
@@
 F 0 "R37" V 4368 3525 50  0000 C CNN
 F 1 "0" V 4459 3525 50  0000 C CNN
-F 2 "Resistor_SMD:R_0603_1608Metric_Pad1.05x0.95mm_HandSolder" V 4505 3525 50  0001 C CNN
+F 2 "Resistor_SMD:R_0603_1608Metric_Pad0.98x0.95mm_HandSolder" V 4505 3525 50  0001 C CNN
 F 3 "~" H 4575 3525 50  0001 C CNN
 F 4 "RK73Z1JTTD" H 4575 3525 50  0001 C CNN "Mfr. #"
@@
 F 0 "C39" V 7000 3500 50  0000 L CNN
 F 1 "4.7nF" V 6725 3475 50  0000 L CNN
-F 2 "Capacitor_SMD:C_0603_1608Metric_Pad1.05x0.95mm_HandSolder" H 6913 3425 50  0001 C CNN
+F 2 "Capacitor_SMD:C_0603_1608Metric_Pad1.08x0.95mm_HandSolder" H 6913 3425 50  0001 C CNN
 F 3 "~" H 6875 3575 50  0001 C CNN
 F 4 "885012206087" H 6875 3575 50  0001 C CNN "Mfr. #"
@@
 F 0 "R39" H 6545 3471 50  0000 L CNN
 F 1 "60.4" H 6545 3380 50  0000 L CNN
-F 2 "Resistor_SMD:R_0603_1608Metric_Pad1.05x0.95mm_HandSolder" V 6405 3425 50  0001 C CNN
+F 2 "Resistor_SMD:R_0603_1608Metric_Pad0.98x0.95mm_HandSolder" V 6405 3425 50  0001 C CNN
 F 3 "~" H 6475 3425 50  0001 C CNN
 F 4 "RMCF0603FT60R4" H 6475 3425 50  0001 C CNN "Mfr. #"
@@
 F 0 "R40" H 6545 3771 50  0000 L CNN
 F 1 "60.4" H 6545 3680 50  0000 L CNN
-F 2 "Resistor_SMD:R_0603_1608Metric_Pad1.05x0.95mm_HandSolder" V 6405 3725 50  0001 C CNN
+F 2 "Resistor_SMD:R_0603_1608Metric_Pad0.98x0.95mm_HandSolder" V 6405 3725 50  0001 C CNN
 F 3 "~" H 6475 3725 50  0001 C CNN
 F 4 "RMCF0603FT60R4" H 6475 3725 50  0001 C CNN "Mfr. #"
@@
 F 0 "R38" V 6018 3575 50  0000 C CNN
 F 1 "0" V 6109 3575 50  0000 C CNN
-F 2 "Resistor_SMD:R_0603_1608Metric_Pad1.05x0.95mm_HandSolder" V 6155 3575 50  0001 C CNN
+F 2 "Resistor_SMD:R_0603_1608Metric_Pad0.98x0.95mm_HandSolder" V 6155 3575 50  0001 C CNN
 F 3 "~" H 6225 3575 50  0001 C CNN
 F 4 "RK73Z1JTTD" H 6225 3575 50  0001 C CNN "Mfr. #"
@@
 F 0 "R41" H 4070 3046 50  0000 L CNN
 F 1 "100K" H 4070 2955 50  0000 L CNN
-F 2 "Resistor_SMD:R_0603_1608Metric_Pad1.05x0.95mm_HandSolder" V 3930 3000 50  0001 C CNN
+F 2 "Resistor_SMD:R_0603_1608Metric_Pad0.98x0.95mm_HandSolder" V 3930 3000 50  0001 C CNN
 F 3 "~" H 4000 3000 50  0001 C CNN
 F 4 "RMCF0603FT100K" H 4000 3000 50  0001 C CNN "Mfr. #"
@@
 F 0 "R35" V 3900 3600 50  0000 C CNN
 F 1 "0" V 3900 3825 50  0000 C CNN
-F 2 "Resistor_SMD:R_0603_1608Metric_Pad1.05x0.95mm_HandSolder" V 3730 3725 50  0001 C CNN
+F 2 "Resistor_SMD:R_0603_1608Metric_Pad0.98x0.95mm_HandSolder" V 3730 3725 50  0001 C CNN
 F 3 "~" H 3800 3725 50  0001 C CNN
 F 4 "RK73Z1JTTD" H 3800 3725 50  0001 C CNN "Mfr. #"
