File: avionics_board/DEBUG_INTERFACE.sch (KiCad schematic (older format))
At the start: 25 parts, among them J12 Conn_01x05, J13 Conn_01x04_Male

Commit message: Essentially done with EPS schematic
Other:
- moved on the sheet: D1, D2, D3, D4, D5, D6, D7, D8, J12, J13, R19, R20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

Commit message: EPS V1.0 Complete
Parts:
- removed TP38, TP40, TP41: TP_1.5x1.5, TestPoint:TestPoint_THTPad_1.5x1.5mm_Drill0.7mm, symbol 1K_Custom_Symbol:TP_1.5x1.5
- J13: footprint Connector_PinHeader_2.54mm:PinHeader_1x04_P2.54mm_Horizontal -> Connector_PinHeader_2.54mm:PinHeader_1x04_P2.54mm_Vertical
- TP37, TP39: footprint TestPoint:TestPoint_THTPad_1.5x1.5mm_Drill0.7mm -> TestPoint:TestPoint_THTPad_1.0x1.0mm_Drill0.5mm
Changed lines of the file:
@@
 Text Notes 2375 4525 0    50   ~ 0
 SWD\n    SWCLK (Clock signal to target CPU)\n    SWDIO (Bi-directional data pin)\n    SWO  (Serial Wire output) optional
-Wire Wire Line
-	2775 1750 2900 1750
-Wire Wire Line
-	2775 1950 2825 1950
-Wire Wire Line
-	2775 2150 2900 2150
 $Comp
 L 1K_Custom_Symbol:TP_1.5x1.5 TP39
@@
 F 0 "TP39" V 2275 5525 50  0000 R CNN
 F 1 "TP_1.5x1.5" V 2400 5775 50  0000 R CNN
-F 2 "TestPoint:TestPoint_THTPad_1.5x1.5mm_Drill0.7mm" H 2550 5350 50  0001 C CNN
+F 2 "TestPoint:TestPoint_THTPad_1.0x1.0mm_Drill0.5mm" H 2550 5350 50  0001 C CNN
 F 3 "~" H 2550 5350 50  0001 C CNN
 	1    2350 5350
 	0    1    1    0
 $EndComp
-$Comp
-L 1K_Custom_Symbol:TP_1.5x1.5 TP41
-U 1 1 6310C54D
-P 2900 2175
-F 0 "TP41" H 2842 2201 50  0000 R CNN
-F 1 "TP_1.5x1.5" H 2842 2292 50  0000 R CNN
-F 2 "TestPoint:TestPoint_THTPad_1.5x1.5mm_Drill0.7mm" H 3100 2175 50  0001 C CNN
-F 3 "~" H 3100 2175 50  0001 C CNN
-	1    2900 2175
-	-1   0    0    1
-$EndComp
-Wire Wire Line
-	2900 2175 2900 2150
-Connection ~ 2900 2150
-Wire Wire Line
-	2900 2150 3600 2150
-$Comp
-L 1K_Custom_Symbol:TP_1.5x1.5 TP38
-U 1 1 5EB6E467
-P 2825 1975
-F 0 "TP38" H 2767 2001 50  0000 R CNN
-F 1 "TP_1.5x1.5" H 2767 2092 50  0000 R CNN
-F 2 "TestPoint:TestPoint_THTPad_1.5x1.5mm_Drill0.7mm" H 3025 1975 50  0001 C CNN
-F 3 "~" H 3025 1975 50  0001 C CNN
-	1    2825 1975
-	-1   0    0    1
-$EndComp
-Wire Wire Line
-	2825 1950 2825 1975
-Connection ~ 2825 1950
-Wire Wire Line
-	2825 1950 3525 1950
-$Comp
-L 1K_Custom_Symbol:TP_1.5x1.5 TP40
-U 1 1 5EB6F13C
-P 2900 1775
-F 0 "TP40" H 2842 1801 50  0000 R CNN
-F 1 "TP_1.5x1.5" H 2842 1892 50  0000 R CNN
-F 2 "TestPoint:TestPoint_THTPad_1.5x1.5mm_Drill0.7mm" H 3100 1775 50  0001 C CNN
-F 3 "~" H 3100 1775 50  0001 C CNN
-	1    2900 1775
-	-1   0    0    1
-$EndComp
-Wire Wire Line
-	2900 1750 2900 1775
-Connection ~ 2900 1750
 Text HLabel 2000 1750 0    50   Input ~ 0
 JTAG_TCK_SWD_SWCLK
@@
 F 0 "J13" H 8347 4057 50  0000 R CNN
 F 1 "Conn_01x04_Male" H 8347 4148 50  0000 R CNN
-F 2 "Connector_PinHeader_2.54mm:PinHeader_1x04_P2.54mm_Horizontal" H 8375 4175 50  0001 C CNN
+F 2 "Connector_PinHeader_2.54mm:PinHeader_1x04_P2.54mm_Vertical" H 8375 4175 50  0001 C CNN
 F 3 "~" H 8375 4175 50  0001 C CNN
 F 4 "PREC004SBAN-M71RC" H 8375 4175 50  0001 C CNN "Mfr. #"
@@
 F 0 "TP37" V 2275 5250 50  0000 R CNN
 F 1 "TP_1.5x1.5" V 2425 5500 50  0000 R CNN
-F 2 "TestPoint:TestPoint_THTPad_1.5x1.5mm_Drill0.7mm" H 2550 5075 50  0001 C CNN
+F 2 "TestPoint:TestPoint_THTPad_1.0x1.0mm_Drill0.5mm" H 2550 5075 50  0001 C CNN
 F 3 "~" H 2550 5075 50  0001 C CNN
 	1    2350 5075
@@
 $EndComp
 Wire Wire Line
-	2900 1750 4675 1750
-Wire Wire Line
 	3525 1950 3525 1850
 Wire Wire Line
@@
 Wire Notes Line width 20
 	6250 5550 6250 3825
+Wire Wire Line
+	2775 1950 3525 1950
+Wire Wire Line
+	2775 1750 4675 1750
+Wire Wire Line
+	2775 2150 3600 2150
 $EndSCHEMATC

Commit message: Update Avionics part names to match KiCad update. Update Avionics board to use new interboard connector
Parts:
- R19, R20, R21, R22, R23, R24, R25, R26, R27, R28: footprint Resistor_SMD:R_0603_1608Metric_Pad1.05x0.95mm_HandSolder -> Resistor_SMD:R_0603_1608Metric_Pad0.98x0.95mm_HandSolder
Changed lines of the file:
@@
 $Descr A 11000 8500
 encoding utf-8
-Sheet 29 39
+Sheet 8 23
 Title "DEBUG INTERFACE"
 Date "2020-05-02"
@@
 F 0 "R24" V 8593 1825 50  0000 C CNN
 F 1 "330" V 8684 1825 50  0000 C CNN
-F 2 "Resistor_SMD:R_0603_1608Metric_Pad1.05x0.95mm_HandSolder" V 8730 1825 50  0001 C CNN
+F 2 "Resistor_SMD:R_0603_1608Metric_Pad0.98x0.95mm_HandSolder" V 8730 1825 50  0001 C CNN
 F 3 "https://www.mouser.com/datasheet/2/427/dcrcwe3-1762152.pdf" H 8800 1825 50  0001 C CNN
 F 4 "CRCW0603330RJNEA" V 8800 1825 50  0001 C CNN "Mfr. #"
@@
 F 0 "R25" V 8593 2175 50  0000 C CNN
 F 1 "330" V 8684 2175 50  0000 C CNN
-F 2 "Resistor_SMD:R_0603_1608Metric_Pad1.05x0.95mm_HandSolder" V 8730 2175 50  0001 C CNN
+F 2 "Resistor_SMD:R_0603_1608Metric_Pad0.98x0.95mm_HandSolder" V 8730 2175 50  0001 C CNN
 F 3 "https://www.mouser.com/datasheet/2/427/dcrcwe3-1762152.pdf" H 8800 2175 50  0001 C CNN
 F 4 "CRCW0603330RJNEA" V 8800 2175 50  0001 C CNN "Mfr. #"
@@
 F 0 "R26" V 8593 2525 50  0000 C CNN
 F 1 "330" V 8684 2525 50  0000 C CNN
-F 2 "Resistor_SMD:R_0603_1608Metric_Pad1.05x0.95mm_HandSolder" V 8730 2525 50  0001 C CNN
+F 2 "Resistor_SMD:R_0603_1608Metric_Pad0.98x0.95mm_HandSolder" V 8730 2525 50  0001 C CNN
 F 3 "https://www.mouser.com/datasheet/2/427/dcrcwe3-1762152.pdf" H 8800 2525 50  0001 C CNN
 F 4 "CRCW0603330RJNEA" V 8800 2525 50  0001 C CNN "Mfr. #"
@@
 F 0 "R27" V 8593 2850 50  0000 C CNN
 F 1 "330" V 8684 2850 50  0000 C CNN
-F 2 "Resistor_SMD:R_0603_1608Metric_Pad1.05x0.95mm_HandSolder" V 8730 2850 50  0001 C CNN
+F 2 "Resistor_SMD:R_0603_1608Metric_Pad0.98x0.95mm_HandSolder" V 8730 2850 50  0001 C CNN
 F 3 "https://www.mouser.com/datasheet/2/427/dcrcwe3-1762152.pdf" H 8800 2850 50  0001 C CNN
 F 4 "CRCW0603330RJNEA" V 8800 2850 50  0001 C CNN "Mfr. #"
@@
 F 0 "R28" V 8593 3200 50  0000 C CNN
 F 1 "330" V 8684 3200 50  0000 C CNN
-F 2 "Resistor_SMD:R_0603_1608Metric_Pad1.05x0.95mm_HandSolder" V 8730 3200 50  0001 C CNN
+F 2 "Resistor_SMD:R_0603_1608Metric_Pad0.98x0.95mm_HandSolder" V 8730 3200 50  0001 C CNN
 F 3 "https://www.mouser.com/datasheet/2/427/dcrcwe3-1762152.pdf" H 8800 3200 50  0001 C CNN
 F 4 "CRCW0603330RJNEA" V 8800 3200 50  0001 C CNN "Mfr. #"
@@
 F 0 "R20" V 2725 1850 50  0000 C CNN
 F 1 "49.9" V 2725 1650 50  0000 C CNN
-F 2 "Resistor_SMD:R_0603_1608Metric_Pad1.05x0.95mm_HandSolder" V 2555 1750 50  0001 C CNN
+F 2 "Resistor_SMD:R_0603_1608Metric_Pad0.98x0.95mm_HandSolder" V 2555 1750 50  0001 C CNN
 F 3 "https://www.mouser.com/datasheet/2/392/susumu_RR_Data_Sheet-1206438.pdf" H 2625 1750 50  0001 C CNN
 F 4 "RR0816Q-49R9-D-68R " V 2625 1750 50  0001 C CNN "Mfr. #"
@@
 F 0 "R21" V 2725 2050 50  0000 C CNN
 F 1 "49.9" V 2725 1850 50  0000 C CNN
-F 2 "Resistor_SMD:R_0603_1608Metric_Pad1.05x0.95mm_HandSolder" V 2555 1950 50  0001 C CNN
+F 2 "Resistor_SMD:R_0603_1608Metric_Pad0.98x0.95mm_HandSolder" V 2555 1950 50  0001 C CNN
 F 3 "https://www.mouser.com/datasheet/2/392/susumu_RR_Data_Sheet-1206438.pdf" H 2625 1950 50  0001 C CNN
 F 4 "RR0816Q-49R9-D-68R " V 2625 1950 50  0001 C CNN "Mfr. #"
@@
 F 0 "R22" V 2725 2250 50  0000 C CNN
 F 1 "49.9" V 2725 2050 50  0000 C CNN
-F 2 "Resistor_SMD:R_0603_1608Metric_Pad1.05x0.95mm_HandSolder" V 2555 2150 50  0001 C CNN
+F 2 "Resistor_SMD:R_0603_1608Metric_Pad0.98x0.95mm_HandSolder" V 2555 2150 50  0001 C CNN
 F 3 "https://www.mouser.com/datasheet/2/392/susumu_RR_Data_Sheet-1206438.pdf" H 2625 2150 50  0001 C CNN
 F 4 "RR0816Q-49R9-D-68R " V 2625 2150 50  0001 C CNN "Mfr. #"
@@
 F 0 "R23" V 2125 5450 50  0000 C CNN
 F 1 "49.9" V 2125 5250 50  0000 C CNN
-F 2 "Resistor_SMD:R_0603_1608Metric_Pad1.05x0.95mm_HandSolder" V 1955 5350 50  0001 C CNN
+F 2 "Resistor_SMD:R_0603_1608Metric_Pad0.98x0.95mm_HandSolder" V 1955 5350 50  0001 C CNN
 F 3 "https://www.mouser.com/datasheet/2/392/susumu_RR_Data_Sheet-1206438.pdf" H 2025 5350 50  0001 C CNN
 F 4 "RR0816Q-49R9-D-68R " V 2025 5350 50  0001 C CNN "Mfr. #"
@@
 F 0 "R19" V 2125 5175 50  0000 C CNN
 F 1 "49.9" V 2125 4975 50  0000 C CNN
-F 2 "Resistor_SMD:R_0603_1608Metric_Pad1.05x0.95mm_HandSolder" V 1955 5075 50  0001 C CNN
+F 2 "Resistor_SMD:R_0603_1608Metric_Pad0.98x0.95mm_HandSolder" V 1955 5075 50  0001 C CNN
 F 3 "https://www.mouser.com/datasheet/2/392/susumu_RR_Data_Sheet-1206438.pdf" H 2025 5075 50  0001 C CNN
 F 4 "RR0816Q-49R9-D-68R " V 2025 5075 50  0001 C CNN "Mfr. #"
