File: avionics_board/OSC32_TCXO.sch (KiCad schematic (older format))
At the start: 5 parts, among them X1 TG-3541CE

Commit message: Removed unecessary footprint lib
Parts:
- X1: footprint avionics_board:Oscillator_SMD_SeikoEpson_TG3541CE-10Pin_3.2x2.5mm_HandSoldering -> footprint_custom:Oscillator_SMD_SeikoEpson_TG3541CE-10Pin_3.2x2.5mm_HandSoldering
Changed lines of the file:
@@
 F 0 "X1" H 5950 4040 50  0000 C CNN
 F 1 "TG-3541CE" H 5950 3949 50  0000 C CNN
-F 2 "avionics_board:Oscillator_SMD_SeikoEpson_TG3541CE-10Pin_3.2x2.5mm_HandSoldering" H 5900 3175 50  0001 C CNN
+F 2 "footprint_custom:Oscillator_SMD_SeikoEpson_TG3541CE-10Pin_3.2x2.5mm_HandSoldering" H 5900 3175 50  0001 C CNN
 F 3 "https://support.epson.biz/td/api/doc_check.php?dl=brief_TG-3541CE&lang=en" H 6050 3625 50  0001 C CNN
 F 4 "TG-3541CE 32.7680KXA3" H 5900 2925 50  0001 C CNN "Mfr. #"

Commit message: EPS V1.0 Complete
Connections:
- net PWR: no longer C36.1
- net at R30.1, R31.2, X1.2 (Vcc)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: now also C36.1
Other:
- note removed: "Layout Note: Decoupling\n"
- moved on the sheet: C36
Changed lines of the file:
@@
 	6550 3475 6550 3575
 Connection ~ 6550 3575
-Text Notes 2420 6455 2    50   ~ 0
-Layout Note: Decoupling\n
-Text HLabel 1625 6600 0    50   Input ~ 0
-PWR
-Text HLabel 1625 6900 0    50   Input ~ 0
-GND
 $Comp
 L Device:C C?
 U 1 1 5FEDE147
-P 2425 6750
+P 5100 4050
 AR Path="/5EA31C93/5EA7CBB1/5FEDE147" Ref="C?"  Part="1"
 AR Path="/5EA31C93/5EAB027D/5FEDE147" Ref="C?"  Part="1"
@@
 AR Path="/5EA31C93/6310C56A/5FEDE147" Ref="C36"  Part="1"
 AR Path="/5FBFFCB6/5FEDB823/5FEDE147" Ref="C36"  Part="1"
-F 0 "C36" H 2540 6796 50  0000 L CNN
-F 1 "0.1uF" H 2540 6705 50  0000 L CNN
-F 2 "Capacitor_SMD:C_0603_1608Metric_Pad1.05x0.95mm_HandSolder" H 2463 6600 50  0001 C CNN
-F 3 "~" H 2425 6750 50  0001 C CNN
-F 4 "25V" H 2425 6750 50  0001 C CNN "Voltage"
-F 5 "CL10B104KA8NNNC" H 2425 6750 50  0001 C CNN "Mfr. #"
-F 6 "https://www.digikey.com/product-detail/en/samsung-electro-mechanics/CL10B104KA8NNNC/1276-1006-1-ND/3889092" H 2425 6750 50  0001 C CNN "Order"
-	1    2425 6750
+F 0 "C36" H 5215 4096 50  0000 L CNN
+F 1 "0.1uF" H 5215 4005 50  0000 L CNN
+F 2 "Capacitor_SMD:C_0603_1608Metric_Pad1.05x0.95mm_HandSolder" H 5138 3900 50  0001 C CNN
+F 3 "~" H 5100 4050 50  0001 C CNN
+F 4 "25V" H 5100 4050 50  0001 C CNN "Voltage"
+F 5 "CL10B104KA8NNNC" H 5100 4050 50  0001 C CNN "Mfr. #"
+F 6 "https://www.digikey.com/product-detail/en/samsung-electro-mechanics/CL10B104KA8NNNC/1276-1006-1-ND/3889092" H 5100 4050 50  0001 C CNN "Order"
+	1    5100 4050
 	1    0    0    -1
 $EndComp
@@
 Text HLabel 3575 3575 0    50   Input ~ 0
 PWR
-Wire Wire Line
-	1625 6600 2425 6600
-Wire Wire Line
-	1625 6900 2425 6900
 Text HLabel 3575 4350 0    50   Input ~ 0
 GND
@@
 Connection ~ 5350 3575
 Wire Wire Line
-	5350 3575 4800 3575
+	5350 3575 5100 3575
 $Comp
 L Device:R R?
@@
 	4800 4025 4275 4025
 Wire Wire Line
-	3575 4350 6550 4350
+	3575 4350 5100 4350
 Wire Wire Line
 	6550 3775 6550 4350
@@
 Text Notes 3750 2825 0    50   ~ 0
 By default, OE is tied high so the chip is enabled immediatly
+Wire Wire Line
+	5100 3900 5100 3575
+Connection ~ 5100 3575
+Wire Wire Line
+	5100 3575 4800 3575
+Wire Wire Line
+	5100 4200 5100 4350
+Connection ~ 5100 4350
+Wire Wire Line
+	5100 4350 6550 4350
 $EndSCHEMATC

Commit message: Update Avionics part names to match KiCad update. Update Avionics board to use new interboard connector
Parts:
- C36: footprint Capacitor_SMD:C_0603_1608Metric_Pad1.05x0.95mm_HandSolder -> Capacitor_SMD:C_0603_1608Metric_Pad1.08x0.95mm_HandSolder
- R29, R30, R31: footprint Resistor_SMD:R_0603_1608Metric_Pad1.05x0.95mm_HandSolder -> Resistor_SMD:R_0603_1608Metric_Pad0.98x0.95mm_HandSolder
Changed lines of the file:
@@
 $Descr A 11000 8500
 encoding utf-8
-Sheet 32 39
+Sheet 9 23
 Title "32kHz TCXO"
 Date "2020-05-25"
@@
 F 0 "C36" H 5215 4096 50  0000 L CNN
 F 1 "0.1uF" H 5215 4005 50  0000 L CNN
-F 2 "Capacitor_SMD:C_0603_1608Metric_Pad1.05x0.95mm_HandSolder" H 5138 3900 50  0001 C CNN
+F 2 "Capacitor_SMD:C_0603_1608Metric_Pad1.08x0.95mm_HandSolder" H 5138 3900 50  0001 C CNN
 F 3 "~" H 5100 4050 50  0001 C CNN
 F 4 "25V" H 5100 4050 50  0001 C CNN "Voltage"
@@
 F 0 "R30" V 4318 3575 50  0000 C CNN
 F 1 "0" V 4409 3575 50  0000 C CNN
-F 2 "Resistor_SMD:R_0603_1608Metric_Pad1.05x0.95mm_HandSolder" V 4455 3575 50  0001 C CNN
+F 2 "Resistor_SMD:R_0603_1608Metric_Pad0.98x0.95mm_HandSolder" V 4455 3575 50  0001 C CNN
 F 3 "~" H 4525 3575 50  0001 C CNN
 F 4 "RK73Z1JTTD" H 4525 3575 50  0001 C CNN "Mfr. #"
@@
 F 0 "R31" V 4843 3475 50  0000 C CNN
 F 1 "0" V 4934 3475 50  0000 C CNN
-F 2 "Resistor_SMD:R_0603_1608Metric_Pad1.05x0.95mm_HandSolder" V 4980 3475 50  0001 C CNN
+F 2 "Resistor_SMD:R_0603_1608Metric_Pad0.98x0.95mm_HandSolder" V 4980 3475 50  0001 C CNN
 F 3 "~" H 5050 3475 50  0001 C CNN
 F 4 "RK73Z1JTTD" H 5050 3475 50  0001 C CNN "Mfr. #"
@@
 F 0 "R29" V 3918 4025 50  0000 C CNN
 F 1 "0" V 4009 4025 50  0000 C CNN
-F 2 "Resistor_SMD:R_0603_1608Metric_Pad1.05x0.95mm_HandSolder" V 4055 4025 50  0001 C CNN
+F 2 "Resistor_SMD:R_0603_1608Metric_Pad0.98x0.95mm_HandSolder" V 4055 4025 50  0001 C CNN
 F 3 "~" H 4125 4025 50  0001 C CNN
 F 4 "RK73Z1JTTD" H 4125 4025 50  0001 C CNN "Mfr. #"
