File: avionics_board/TEMPERATURE_ADC.sch (KiCad schematic (older format))
At the start: 0 parts

Commit message: Progress on EPS
Parts:
- added R?: 0, Resistor_SMD:R_0603_1608Metric_Pad1.05x0.95mm_HandSolder, symbol Device:R
Connections:
- net VDD: now also R?.2
- new net INTRNL_VDD: R?.1

Commit message: Essentially done with EPS schematic
Parts:
- gave numbers to parts that had none: 1
Changed lines of the file:
@@
 $Descr A 11000 8500
 encoding utf-8
-Sheet 12 24
+Sheet 12 23
 Title "Temperature Sensors"
 Date "2020-05-05"
@@
 P 1875 1250
 AR Path="/5EA31C93/5EAB13AE/63F792FA" Ref="R?"  Part="1"
-AR Path="/5EA31C93/5EAB0B79/63F792FA" Ref="R?"  Part="1"
-F 0 "R?" V 1668 1250 50  0000 C CNN
+AR Path="/5EA31C93/5EAB0B79/63F792FA" Ref="R8"  Part="1"
+F 0 "R8" V 1668 1250 50  0000 C CNN
 F 1 "0" V 1759 1250 50  0000 C CNN
 F 2 "Resistor_SMD:R_0603_1608Metric_Pad1.05x0.95mm_HandSolder" V 1805 1250 50  0001 C CNN

Commit message: Update Avionics part names to match KiCad update. Update Avionics board to use new interboard connector
Parts:
- R8: footprint Resistor_SMD:R_0603_1608Metric_Pad1.05x0.95mm_HandSolder -> Resistor_SMD:R_0603_1608Metric_Pad0.98x0.95mm_HandSolder
Changed lines of the file:
@@
 F 0 "R8" V 1668 1250 50  0000 C CNN
 F 1 "0" V 1759 1250 50  0000 C CNN
-F 2 "Resistor_SMD:R_0603_1608Metric_Pad1.05x0.95mm_HandSolder" V 1805 1250 50  0001 C CNN
+F 2 "Resistor_SMD:R_0603_1608Metric_Pad0.98x0.95mm_HandSolder" V 1805 1250 50  0001 C CNN
 F 3 "~" H 1875 1250 50  0001 C CNN
 F 4 "RK73Z1JTTD" H 1875 1250 50  0001 C CNN "Mfr. #"
