File: avionics_board/WATCHDOG.sch (KiCad schematic (older format))
At the start: 9 parts, among them SW1 SW_DIP_x01, SW2 SW_Push, U3 TPL5010

Commit message: Progress on EPS
Parts:
- removed TP10: TP_1.5x1.5, TestPoint:TestPoint_THTPad_1.5x1.5mm_Drill0.7mm, symbol 1K_Custom_Symbol:TP_1.5x1.5
Changed lines of the file:
@@
 $Descr A 11000 8500
 encoding utf-8
-Sheet 5 25
+Sheet 4 39
 Title "EXTERNAL WATCHDOG"
 Date "2020-05-02"
@@
 $Comp
 L Timer:TPL5010 U3
-U 1 1 5EB1B3D3
+U 1 1 6310C545
 P 5550 3475
 F 0 "U3" H 5300 3925 50  0000 R CNN
@@
 $Comp
 L Device:C C?
-U 1 1 5EB1E933
+U 1 1 6310C546
 P 1900 5500
-AR Path="/5EA31C93/5EA7CBB1/5EB1E933" Ref="C?"  Part="1"
-AR Path="/5EA31C93/5EAB027D/5EB1E933" Ref="C?"  Part="1"
-AR Path="/5EA31C93/5EAB163E/5EB1E933" Ref="C?"  Part="1"
-AR Path="/5EA31C93/5EAB0A1F/5EB1E933" Ref="C21"  Part="1"
+AR Path="/5EA31C93/5EA7CBB1/6310C546" Ref="C?"  Part="1"
+AR Path="/5EA31C93/5EAB027D/6310C546" Ref="C?"  Part="1"
+AR Path="/5EA31C93/5EAB163E/6310C546" Ref="C?"  Part="1"
+AR Path="/5EA31C93/5EAB0A1F/6310C546" Ref="C21"  Part="1"
+AR Path="/5FBFFCB6/5EAB0A1F/6310C546" Ref="C21"  Part="1"
 F 0 "C21" H 2015 5546 50  0000 L CNN
 F 1 "0.1uF" H 2015 5455 50  0000 L CNN
@@
 $Comp
 L Switch:SW_DIP_x01 SW1
-U 1 1 5EB20C87
+U 1 1 6310C547
 P 3800 3375
 F 0 "SW1" H 3800 3642 50  0000 C CNN
@@
 $Comp
 L Device:R R14
-U 1 1 5EB21A87
+U 1 1 6310C548
 P 3200 3025
 F 0 "R14" H 3270 3071 50  0000 L CNN
@@
 $Comp
 L Device:R R15
-U 1 1 5EB25535
+U 1 1 6310C549
 P 6900 3900
 F 0 "R15" H 6970 3946 50  0000 L CNN
@@
 $Comp
 L Switch:SW_Push SW2
-U 1 1 5EB263A3
+U 1 1 6310C54A
 P 6900 3025
 F 0 "SW2" V 6854 3173 50  0000 L CNN
@@
 	3200 2825 5550 2825
 Wire Wire Line
-	4100 3375 4650 3375
-Wire Wire Line
 	4700 3475 5050 3475
 Wire Wire Line
@@
 Text Notes 4025 3600 2    50   ~ 0
 Disable switch
-$Comp
-L 1K_Custom_Symbol:TP_1.5x1.5 TP?
-U 1 1 5EB2E7B0
-P 4550 3275
-AR Path="/5EA31C93/5EAB163E/5EB2E7B0" Ref="TP?"  Part="1"
-AR Path="/5EA31C93/5EAB0A1F/5EB2E7B0" Ref="TP10"  Part="1"
-F 0 "TP10" V 4745 3347 50  0000 C CNN
-F 1 "TP_1.5x1.5" V 4654 3347 50  0000 C CNN
-F 2 "TestPoint:TestPoint_THTPad_1.5x1.5mm_Drill0.7mm" H 4750 3275 50  0001 C CNN
-F 3 "~" H 4750 3275 50  0001 C CNN
-	1    4550 3275
-	0    -1   -1   0
-$EndComp
-Wire Wire Line
-	4550 3275 4650 3275
-Wire Wire Line
-	4650 3275 4650 3375
-Connection ~ 4650 3375
-Wire Wire Line
-	4650 3375 5050 3375
 $Comp
 L 1K_Custom_Symbol:TP_smt_1x1 TP9
@@
 	0    1    1    0
 $EndComp
+Wire Wire Line
+	4100 3375 5050 3375
 $EndSCHEMATC

Commit message: Essentially done with EPS schematic
Parts:
- R14: Mfr. # RMCF0603JG100K -> RMCF0603FT100K; Order https://www.digikey.com/product-detail/en/stackpole-electro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 -> https://www.digikey.com/en/products/detail/stackpole-electr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
Changed lines of the file:
@@
 $Descr A 11000 8500
 encoding utf-8
-Sheet 4 39
+Sheet 28 39
 Title "EXTERNAL WATCHDOG"
 Date "2020-05-02"
@@
 F 2 "Resistor_SMD:R_0603_1608Metric_Pad1.05x0.95mm_HandSolder" V 3130 3025 50  0001 C CNN
 F 3 "~" H 3200 3025 50  0001 C CNN
-F 4 "RMCF0603JG100K" H 3200 3025 50  0001 C CNN "Mfr. #"
-F 5 "https://www.digikey.com/product-detail/en/stackpole-electronics-inc/RMCF0603JG100K/RMCF0603JG100KCT-ND/4425127" H 3200 3025 50  0001 C CNN "Order"
+F 4 "RMCF0603FT100K" H 3200 3025 50  0001 C CNN "Mfr. #"
+F 5 "https://www.digikey.com/en/products/detail/stackpole-electronics-inc/RMCF0603FT100K/1761112" H 3200 3025 50  0001 C CNN "Order"
 	1    3200 3025
 	1    0    0    -1

Commit message: EPS V1.0 Complete
Parts:
- TP8, TP9: footprint TestPoint:TestPoint_Pad_1.0x1.0mm -> TestPoint:TestPoint_THTPad_1.0x1.0mm_Drill0.5mm
Changed lines of the file:
@@
 F 0 "TP9" V 2604 2013 50  0000 L CNN
 F 1 "TP_smt_1x1" V 2695 2013 50  0000 L CNN
-F 2 "TestPoint:TestPoint_Pad_1.0x1.0mm" H 2850 1825 50  0001 C CNN
+F 2 "TestPoint:TestPoint_THTPad_1.0x1.0mm_Drill0.5mm" H 2850 1825 50  0001 C CNN
 F 3 "~" H 2850 1825 50  0001 C CNN
 	1    2650 1825
@@
 F 0 "TP8" V 1929 2113 50  0000 L CNN
 F 1 "TP_smt_1x1" V 2020 2113 50  0000 L CNN
-F 2 "TestPoint:TestPoint_Pad_1.0x1.0mm" H 2175 1925 50  0001 C CNN
+F 2 "TestPoint:TestPoint_THTPad_1.0x1.0mm_Drill0.5mm" H 2175 1925 50  0001 C CNN
 F 3 "~" H 2175 1925 50  0001 C CNN
 	1    1975 1925

Commit message: Update Avionics part names to match KiCad update. Update Avionics board to use new interboard connector
Parts:
- C21: footprint Capacitor_SMD:C_0603_1608Metric_Pad1.05x0.95mm_HandSolder -> Capacitor_SMD:C_0603_1608Metric_Pad1.08x0.95mm_HandSolder
- R14, R15: footprint Resistor_SMD:R_0603_1608Metric_Pad1.05x0.95mm_HandSolder -> Resistor_SMD:R_0603_1608Metric_Pad0.98x0.95mm_HandSolder
Changed lines of the file:
@@
 $Descr A 11000 8500
 encoding utf-8
-Sheet 28 39
+Sheet 4 23
 Title "EXTERNAL WATCHDOG"
 Date "2020-05-02"
@@
 F 0 "C21" H 2015 5546 50  0000 L CNN
 F 1 "0.1uF" H 2015 5455 50  0000 L CNN
-F 2 "Capacitor_SMD:C_0603_1608Metric_Pad1.05x0.95mm_HandSolder" H 1938 5350 50  0001 C CNN
+F 2 "Capacitor_SMD:C_0603_1608Metric_Pad1.08x0.95mm_HandSolder" H 1938 5350 50  0001 C CNN
 F 3 "~" H 1900 5500 50  0001 C CNN
 F 4 "25V" H 1900 5500 50  0001 C CNN "Voltage"
@@
 F 0 "R14" H 3270 3071 50  0000 L CNN
 F 1 "100K" H 3270 2980 50  0000 L CNN
-F 2 "Resistor_SMD:R_0603_1608Metric_Pad1.05x0.95mm_HandSolder" V 3130 3025 50  0001 C CNN
+F 2 "Resistor_SMD:R_0603_1608Metric_Pad0.98x0.95mm_HandSolder" V 3130 3025 50  0001 C CNN
 F 3 "~" H 3200 3025 50  0001 C CNN
 F 4 "RMCF0603FT100K" H 3200 3025 50  0001 C CNN "Mfr. #"
@@
 F 0 "R15" H 6970 3946 50  0000 L CNN
 F 1 "8.85K" H 6970 3855 50  0000 L CNN
-F 2 "Resistor_SMD:R_0603_1608Metric_Pad1.05x0.95mm_HandSolder" V 6830 3900 50  0001 C CNN
+F 2 "Resistor_SMD:R_0603_1608Metric_Pad0.98x0.95mm_HandSolder" V 6830 3900 50  0001 C CNN
 F 3 "~" H 6900 3900 50  0001 C CNN
 F 4 "RMCF0603FT8K87" H 6900 3900 50  0001 C CNN "Mfr. #"
