File: avionics_board/MAG.sch (KiCad schematic (older format))
At the start: 13 parts, among them U9 MMC5983MA

Commit message: Update Avionics part names to match KiCad update. Update Avionics board to use new interboard connector
Parts:
- C44, C45: footprint Capacitor_SMD:C_0603_1608Metric_Pad1.05x0.95mm_HandSolder -> Capacitor_SMD:C_0603_1608Metric_Pad1.08x0.95mm_HandSolder
- R43, R44: footprint Resistor_SMD:R_0603_1608Metric_Pad1.05x0.95mm_HandSolder -> Resistor_SMD:R_0603_1608Metric_Pad0.98x0.95mm_HandSolder
Changed lines of the file:
@@
 F 0 "C45" H 6200 3425 50  0000 R CNN
 F 1 "10uF" H 6200 3500 50  0000 R CNN
-F 2 "Capacitor_SMD:C_0603_1608Metric_Pad1.05x0.95mm_HandSolder" H 6363 3300 50  0001 C CNN
+F 2 "Capacitor_SMD:C_0603_1608Metric_Pad1.08x0.95mm_HandSolder" H 6363 3300 50  0001 C CNN
 F 3 "~" H 6325 3450 50  0001 C CNN
 F 4 "CL10X106MO8NRNC" H 6325 3450 50  0001 C CNN "Mfr. #"
@@
 F 0 "C44" H 2090 5471 50  0000 L CNN
 F 1 "1uF" H 2090 5380 50  0000 L CNN
-F 2 "Capacitor_SMD:C_0603_1608Metric_Pad1.05x0.95mm_HandSolder" H 2013 5275 50  0001 C CNN
+F 2 "Capacitor_SMD:C_0603_1608Metric_Pad1.08x0.95mm_HandSolder" H 2013 5275 50  0001 C CNN
 F 3 "~" H 1975 5425 50  0001 C CNN
 F 4 "CL10B105KP8NFNC" H 1975 5425 50  0001 C CNN "Mfr. #"
@@
 F 0 "R44" V 4493 2875 50  0000 C CNN
 F 1 "0" V 4584 2875 50  0000 C CNN
-F 2 "Resistor_SMD:R_0603_1608Metric_Pad1.05x0.95mm_HandSolder" V 4630 2875 50  0001 C CNN
+F 2 "Resistor_SMD:R_0603_1608Metric_Pad0.98x0.95mm_HandSolder" V 4630 2875 50  0001 C CNN
 F 3 "~" H 4700 2875 50  0001 C CNN
 F 4 "RK73Z1JTTD" H 4700 2875 50  0001 C CNN "Mfr. #"
@@
 F 0 "R43" V 4493 2500 50  0000 C CNN
 F 1 "0" V 4584 2500 50  0000 C CNN
-F 2 "Resistor_SMD:R_0603_1608Metric_Pad1.05x0.95mm_HandSolder" V 4630 2500 50  0001 C CNN
+F 2 "Resistor_SMD:R_0603_1608Metric_Pad0.98x0.95mm_HandSolder" V 4630 2500 50  0001 C CNN
 F 3 "~" H 4700 2500 50  0001 C CNN
 F 4 "RK73Z1JTTD" H 4700 2500 50  0001 C CNN "Mfr. #"

Commit message: Avionics Board layout done
Parts:
- removed TP55, TP58, TP59: TP_1.5x1.5, TestPoint:TestPoint_THTPad_1.5x1.5mm_Drill0.7mm, symbol 1K_Custom_Symbol:TP_1.5x1.5
Connections:
- net VDD: no longer C44.1
- net at R44.1, U9.2 (VDD): now also C44.1
Other:
- note removed: "Layout Note: Decoupling\n"
- moved on the sheet: C44, R44
Changed lines of the file:
@@
 Comment4 ""
 $EndDescr
-Text HLabel 1650 5275 0    50   Output ~ 0
-VDD
-Text HLabel 1650 5575 0    50   Output ~ 0
-VSS
-Text Notes 2320 5130 2    50   ~ 0
-Layout Note: Decoupling\n
-Wire Wire Line
-	1650 5275 1975 5275
-Wire Wire Line
-	1650 5575 1975 5575
 $Comp
 L Device:C C45
@@
 Text Notes 8375 3400 2    50   ~ 0
 Low ESR cap, close proximity to the chip
-Wire Wire Line
-	5200 3050 5200 2875
 Text HLabel 5025 4675 0    50   Output ~ 0
 VSS
 Wire Wire Line
 	5350 4675 5350 4400
-Text HLabel 4450 2875 0    50   Output ~ 0
+Text HLabel 4450 2725 0    50   Output ~ 0
 VDD
 Wire Wire Line
@@
 L Device:C C?
 U 1 1 5EB37DF9
-P 1975 5425
+P 6100 2875
 AR Path="/5EA31C93/5EA7CBB1/5EB37DF9" Ref="C?"  Part="1"
 AR Path="/5EA31C93/5EAB027D/5EB37DF9" Ref="C?"  Part="1"
@@
 AR Path="/5EA31C93/5EAB0A1F/5EB37DF9" Ref="C?"  Part="1"
 AR Path="/5EA31C93/5EAB13AE/5EB37DF9" Ref="C44"  Part="1"
-F 0 "C44" H 2090 5471 50  0000 L CNN
-F 1 "1uF" H 2090 5380 50  0000 L CNN
-F 2 "Capacitor_SMD:C_0603_1608Metric_Pad1.08x0.95mm_HandSolder" H 2013 5275 50  0001 C CNN
-F 3 "~" H 1975 5425 50  0001 C CNN
-F 4 "CL10B105KP8NFNC" H 1975 5425 50  0001 C CNN "Mfr. #"
-F 5 "https://www.digikey.com/product-detail/en/samsung-electro-mechanics/CL10B105KP8NFNC/1276-1945-1-ND/3890031" H 1975 5425 50  0001 C CNN "Order"
-F 6 "10V" H 1975 5425 50  0001 C CNN "Voltage"
-	1    1975 5425
+F 0 "C44" H 6215 2921 50  0000 L CNN
+F 1 "1uF" H 6215 2830 50  0000 L CNN
+F 2 "Capacitor_SMD:C_0603_1608Metric_Pad1.08x0.95mm_HandSolder" H 6138 2725 50  0001 C CNN
+F 3 "~" H 6100 2875 50  0001 C CNN
+F 4 "CL10B105KP8NFNC" H 6100 2875 50  0001 C CNN "Mfr. #"
+F 5 "https://www.digikey.com/product-detail/en/samsung-electro-mechanics/CL10B105KP8NFNC/1276-1945-1-ND/3890031" H 6100 2875 50  0001 C CNN "Order"
+F 6 "10V" H 6100 2875 50  0001 C CNN "Voltage"
+	1    6100 2875
 	1    0    0    -1
 $EndComp
@@
 L Device:R R44
 U 1 1 5EB3A638
-P 4700 2875
-F 0 "R44" V 4493 2875 50  0000 C CNN
-F 1 "0" V 4584 2875 50  0000 C CNN
-F 2 "Resistor_SMD:R_0603_1608Metric_Pad0.98x0.95mm_HandSolder" V 4630 2875 50  0001 C CNN
-F 3 "~" H 4700 2875 50  0001 C CNN
-F 4 "RK73Z1JTTD" H 4700 2875 50  0001 C CNN "Mfr. #"
-F 5 "https://www.digikey.com/product-detail/en/koa-speer-electronics-inc/RK73Z1JTTD/2019-RK73Z1JTTDCT-ND/9847522" H 4700 2875 50  0001 C CNN "Order"
-	1    4700 2875
-	0    1    1    0
-$EndComp
-Wire Wire Line
-	4450 2875 4550 2875
-Wire Wire Line
-	4850 2875 5200 2875
+P 4700 2725
+F 0 "R44" V 4600 2725 50  0000 C CNN
+F 1 "0" V 4800 2725 50  0000 C CNN
+F 2 "Resistor_SMD:R_0603_1608Metric_Pad0.98x0.95mm_HandSolder" V 4630 2725 50  0001 C CNN
+F 3 "~" H 4700 2725 50  0001 C CNN
+F 4 "RK73Z1JTTD" H 4700 2725 50  0001 C CNN "Mfr. #"
+F 5 "https://www.digikey.com/product-detail/en/koa-speer-electronics-inc/RK73Z1JTTD/2019-RK73Z1JTTDCT-ND/9847522" H 4700 2725 50  0001 C CNN "Order"
+	1    4700 2725
+	0    1    1    0
+$EndComp
+Wire Wire Line
+	4450 2725 4550 2725
 Text HLabel 1600 1325 0    50   Input ~ 0
 CLK
@@
 Text HLabel 1600 1725 0    50   Input ~ 0
 MOSI_SDA
-Text HLabel 1600 1825 0    50   Output ~ 0
-VDD
-$Comp
-L 1K_Custom_Symbol:TP_1.5x1.5 TP58
-U 1 1 5EB3E3D1
-P 2675 1825
-F 0 "TP58" V 2629 2013 50  0000 L CNN
-F 1 "TP_1.5x1.5" V 2720 2013 50  0000 L CNN
-F 2 "TestPoint:TestPoint_THTPad_1.5x1.5mm_Drill0.7mm" H 2875 1825 50  0001 C CNN
-F 3 "~" H 2875 1825 50  0001 C CNN
-	1    2675 1825
-	0    1    1    0
-$EndComp
 Wire Wire Line
 	1600 1325 2050 1325
@@
 Wire Wire Line
 	1600 1725 2050 1725
-Wire Wire Line
-	2675 1825 1600 1825
 $Comp
 L 1K_Custom_Symbol:TP_smt_1x1 TP52
@@
 Wire Wire Line
 	5500 2500 5500 3050
-Wire Wire Line
-	1600 1925 2050 1925
-$Comp
-L 1K_Custom_Symbol:TP_1.5x1.5 TP55
-U 1 1 5EB3E735
-P 2050 1925
-F 0 "TP55" V 2004 2113 50  0000 L CNN
-F 1 "TP_1.5x1.5" V 2095 2113 50  0000 L CNN
-F 2 "TestPoint:TestPoint_THTPad_1.5x1.5mm_Drill0.7mm" H 2250 1925 50  0001 C CNN
-F 3 "~" H 2250 1925 50  0001 C CNN
-	1    2050 1925
-	0    1    1    0
-$EndComp
-Text HLabel 1600 1925 0    50   Output ~ 0
-VDDIO
-Text HLabel 1600 2025 0    50   Output ~ 0
-VSS
-$Comp
-L 1K_Custom_Symbol:TP_1.5x1.5 TP59
-U 1 1 5ECDBF03
-P 2675 2025
-F 0 "TP59" V 2629 2213 50  0000 L CNN
-F 1 "TP_1.5x1.5" V 2720 2213 50  0000 L CNN
-F 2 "TestPoint:TestPoint_THTPad_1.5x1.5mm_Drill0.7mm" H 2875 2025 50  0001 C CNN
-F 3 "~" H 2875 2025 50  0001 C CNN
-	1    2675 2025
-	0    1    1    0
-$EndComp
-Wire Wire Line
-	2675 2025 1600 2025
 $Comp
 L 1K_Custom_Symbol:MMC5983MA U9
@@
 	1    0    0    -1
 $EndComp
+Wire Wire Line
+	4850 2725 5200 2725
+Wire Wire Line
+	5200 2725 5200 3050
+Wire Wire Line
+	5200 2725 6100 2725
+Connection ~ 5200 2725
+Text HLabel 5925 3025 0    50   Output ~ 0
+VSS
+Wire Wire Line
+	5925 3025 6100 3025
 $EndSCHEMATC
