File: avionics_board/STM32L4.sch (KiCad schematic (older format))
At the start: 22 parts, among them U1 STM32L496ZGTx

Commit message: Progress on EPS
Parts:
- added C? (x2): 0.1uF, Capacitor_SMD:C_0603_1608Metric_Pad1.05x0.95mm_HandSolder, symbol Device:C
- added U? (x2): 74LVC1G07, Package_TO_SOT_SMD:SOT-353_SC-70-5_Handsoldering, symbol 74xGxx:74LVC1G07
Connections:
- net GND: now also C?.1, C?.1, U?.3 (GND), U?.3 (GND)
- net RST: now also U?.2
- net MANUAL_RST: now reaches U1.96 (PC6)
- net MANUAL_RST: now also U?.2
- net EPS_RST: now reaches U1.97 (PC7)
- net 3.3V_STM_CORE renamed VCC
- net VCC: now also C?.2, C?.2, U?.5 (VCC), U?.5 (VCC)
- net SDMMC1_CK: no longer names the net of U1.113 (PC12)
- net SDMMC1_CMD: no longer names the net of U1.116 (PD2)
- net SDMMC1_D1: no longer names the net of U1.99 (PC9)
- net SDMMC1_D2: no longer names the net of U1.111 (PC10)
- net SDMMC1_D3: no longer names the net of U1.112 (PC11)
- net SDMMC1_DO renamed TEMP_PWR
- new net AVI_RST: U?.4, U?.4
- no-connect marks 22 -> 25
Other:
- note added: "STM Reset Triggers"
- note added: "STM32L496ZGT3 \nis the high (+125) temperature version\n\nSTM32L496ZGT6\nis the lower (+85) temperature version"
- note removed: "SD CARD\n"
- note removed: "TODO: Power to CAN"
- note removed: "VDD: 2.7V to 3.6V \n250mA peak"

Commit message: Essentially done with EPS schematic
Parts:
- C1, C13, C2: Mfr. # CL10B103KB8NCNC -> CL10B103KB8NNNC; Order https://www.digikey.com/product-detail/en/samsung-electro-m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 -> https://www.digikey.com/en/products/detail/samsung-electro-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
- C19, C20: renamed from C?; Mfr. # (none) -> CL10B104KA8NNNC; Order (none) -> https://www.digikey.com/product-detail/en/samsung-electro-m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; Voltage (none) -> 25V
- gave numbers to parts that had none: 2
Connections:
- net IRIDIUM_DCD: no longer names the net of U1.49 (PF11)
- net IRIDIUM_DSR: no longer names the net of U1.50 (PF12)
- net IRIDIUM_DTR: no longer names the net of U1.19 (PF7)
- net IRIDIUM_NET_AVAIL: no longer names the net of U1.90 (PG5)
- net IRIDIUM_ON_OFF: no longer names the net of U1.53 (PF13)
- net IRIDIUM_RING: no longer names the net of U1.89 (PG4)
- net RCC_OSC32_OUT: no longer names the net of U1.9 (PC15)
- net RCC_OSC_OUT: no longer names the net of U1.24 (PH1)
- no-connect marks 25 -> 35
Other:
- note removed: "3.3V Logic"
- note removed: "5.0V PWR \n2A. Softstart"
- note removed: "IRIDIUM"

Commit message: Update Avionics part names to match KiCad update. Update Avionics board to use new interboard connector
Parts:
- added H1, H2, H3, H4: MountingHole_Pad, MountingHole:MountingHole_3.2mm_M3_Pad_Via, symbol Mechanical:MountingHole_Pad
- C1, C10, C11, C12, C13, C14, C15, C16, C17, C19, C2, C20, C3, C4, C5, C6, C7, C8, C9: footprint Capacitor_SMD:C_0603_1608Metric_Pad1.05x0.95mm_HandSolder -> Capacitor_SMD:C_0603_1608Metric_Pad1.08x0.95mm_HandSolder
- R1, R2, R3, R4: footprint Resistor_SMD:R_0603_1608Metric_Pad1.05x0.95mm_HandSolder -> Resistor_SMD:R_0603_1608Metric_Pad0.98x0.95mm_HandSolder
Connections:
- wire segments 391 -> 399

Commit message: Avionics Board layout done
Parts:
- added H5, H6, H7: MountingHole, MountingHole:MountingHole_2.7mm, symbol Mechanical:MountingHole
- added R10, R11, R12, R9: DNP, Resistor_SMD:R_0603_1608Metric_Pad0.98x0.95mm_HandSolder, symbol Device:R
- added TP10, TP11, TP12, TP13, TP7: TP_tht_1x1, TestPoint:TestPoint_THTPad_1.0x1.0mm_Drill0.5mm, symbol 1K_Custom_Symbol:TP_smt_1x1
- added TP14, TP15, TP16: TP_smt_1x1, TestPoint:TestPoint_Pad_1.0x1.0mm, symbol 1K_Custom_Symbol:TP_smt_1x1
- added TP3, TP6: TP_smt_1x1, TestPoint:TestPoint_THTPad_1.0x1.0mm_Drill0.5mm, symbol 1K_Custom_Symbol:TP_smt_1x1
Connections:
- net labels added: 10MHZ_OE, ADC1_IN5, ADC1_IN6
- net labels removed: ADC1_IN1, ADC1_IN2, SUN_CS_3, SUN_FRAME_RDY_3
- wire segments 399 -> 409
- no-connect marks 35 -> 31
Other:
- note added: "I2C is currently unused, \nbut left available"
