File: eps_board/CURRENT_MONITORS.sch (KiCad schematic (older format))
At the start: 56 parts

Commit message: Essentially done with EPS schematic
Parts:
- C44, C45: renamed from C?; Mfr. # (none) -> CL10B105KP8NFNC; Order (none) -> https://www.digikey.com/product-detail/en/samsung-electro-m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; Voltage (none) -> 10V
- R100, R102, R104, R106, R112, R114, R116, R118, R124, R126, R128, R130, R136, R138, R140, R142: renamed from R?; value 3090 -> 3.09K; Mfr. # (none) -> RMCF0603FT3K09; Order (none) -> https://www.digikey.com/en/products/detail/stackpole-electr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
- R101, R103, R105, R123, R125, R127, R129, R135, R137, R139, R141: renamed from R?; value 140k -> 140K; Mfr. # ERJ-3RSFR10V -> RK73H1JTTD1403F; Order https://www.digikey.com/product-detail/en/panasonic-electro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 -> https://www.digikey.com/en/products/detail/koa-speer-electr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
- R111, R117: renamed from R?; value 700k -> 698K; Mfr. # ERJ-3RSFR10V -> RMCF0603FT698K; Order https://www.digikey.com/product-detail/en/panasonic-electro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 -> https://www.digikey.com/en/products/detail/stackpole-electr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
- R113, R115: renamed from R?; Mfr. # ERJ-3RSFR10V -> RC0603FR-071M5L; Order https://www.digikey.com/product-detail/en/panasonic-electro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 -> https://www.digikey.com/en/products/detail/yageo/RC0603FR-0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
- R91, R92: renamed from R?; value 1k -> 1K; Mfr. # (none) -> RMCF0603FT1K00; Order (none) -> https://www.digikey.com/en/products/detail/stackpole-electr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
- R94: renamed from R?; value 0.04 -> 0.039; Mfr. # ERJ-3RSFR10V -> ERJ-3BWFR039V; Order https://www.digikey.com/product-detail/en/panasonic-electro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 -> https://www.digikey.com/en/products/detail/panasonic-electr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
- R97, R98: renamed from R?; value 10k -> 10K; Mfr. # (none) -> RMCF0603FT10K0; Order (none) -> https://www.digikey.com/en/products/detail/stackpole-electr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
- R99: renamed from R?; value 20k -> 20K; Mfr. # ERJ-3RSFR10V -> RMCF0603FT20K0; Order https://www.digikey.com/product-detail/en/panasonic-electro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 -> https://www.digikey.com/en/products/detail/stackpole-electr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
- gave numbers to parts that had none: 17
