File: eps_board/PMIC.sch (KiCad schematic (older format))
At the start: 57 parts, among them U1 STM32L496ZGTx

Commit message: Essentially done with EPS schematic
Parts:
- C1, C13, C2: Mfr. # CL10B103KB8NCNC -> CL10B103KB8NNNC; Order https://www.digikey.com/product-detail/en/samsung-electro-m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 -> https://www.digikey.com/en/products/detail/samsung-electro-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
- R1: Mfr. # RK73Z1JTTD -> RK73Z1JTTD; Order https://www.digikey.com/product-detail/en/koa-speer-electronics-inc/RK73Z1JTTD/2019-RK73Z1JTTDCT-ND/9847522 -> https://www.digikey.com/product-detail/en/koa-speer-electronics-inc/RK73Z1JTTD/2019-RK73Z1JTTDCT-ND/9847522
- R271, R272, R273, R274, R275, R276, R277, R278, R279, R280, R281, R282, R283, R284, R285, R286, R287, R288, R289, R290, R291, R292, R293, R294, R295, R296, R297, R298, R299, R300, R301, R302, R303, R304, R305: renamed from R?; Mfr. # RK73Z1JTTD -> RK73Z1JTTD; Order https://www.digikey.com/product-detail/en/koa-speer-electronics-inc/RK73Z1JTTD/2019-RK73Z1JTTDCT-ND/9847522 -> https://www.digikey.com/product-detail/en/koa-speer-electronics-inc/RK73Z1JTTD/2019-RK73Z1JTTDCT-ND/9847522
Connections:
- net RCC_OSC32_OUT: no longer names the net of U1.9 (PC15)

Commit message: EPS layout in progress
Parts:
- removed R271, R272, R273, R274, R275, R276, R277, R278, R279, R280, R281, R282, R283, R284, R285, R286, R287, R288, R289, R290, R291, R292, R293, R294, R295, R296, R297, R298, R299, R300, R301, R302, R303: 0, Resistor_SMD:R_0603_1608Metric_Pad1.05x0.95mm_HandSolder, symbol Device:R_Small
Connections:
- net INT_1: now also U1.56 (PG0)
- net INT_10: now also U1.125 (PG10)
- net INT_11: now also U1.126 (PG11)
- net INT_12: now also U1.127 (PG12)
- net INT_13: now also U1.128 (PG13)
- net INT_14: now also U1.129 (PG14)
- net INT_15: now also U1.132 (PG15)
- net INT_2: now also U1.87 (PG2)
- net INT_3: now also U1.88 (PG3)
- net INT_4: now also U1.89 (PG4)
- net INT_5: now also U1.90 (PG5)
- net INT_6: now also U1.91 (PG6)
- net INT_7: now also U1.92 (PG7)
- net INT_8: now also U1.93 (PG8)
- net INT_9: now also U1.124 (PG9)
- net PWR1_10_ON: now also U1.142 (PE1)
- net PWR1_11_ON: now also U1.1 (PE2)
- net PWR1_12_ON: now also U1.2 (PE3)
- net PWR1_13_ON: now also U1.3 (PE4)
- net PWR1_14_ON: now also U1.4 (PE5)
- net PWR1_15_ON: now also U1.5 (PE6)
- net PWR1_16_ON: now also U1.58 (PE7)
- net PWR1_1_ON: now also U1.10 (PF0)
- net PWR1_2_ON: now also U1.11 (PF1)
- net PWR1_3_ON: now also U1.19 (PF7)
- net PWR1_4_ON: now also U1.21 (PF9)
- net PWR1_5_ON: now also U1.49 (PF11)
- net PWR1_6_ON: now also U1.50 (PF12)
- net PWR1_7_ON: now also U1.53 (PF13)
- net PWR1_8_ON: now also U1.54 (PF14)
- net PWR1_9_ON: now also U1.55 (PF15)
- net PWR2_1_ON: now also U1.59 (PE8)
- net PWR2_2_ON: now also U1.60 (PE9)
