File: eps_board/BATTERY.sch (KiCad schematic (older format))
At the start: 16 parts

Commit message: Progress on EPS
Parts:
- removed U?: FPF2000, Package_TO_SOT_SMD:SOT-353_SC-70-5_Handsoldering, symbol 1K_Custom_Symbol:FPF2000
- removed U?: MCP6541, Package_TO_SOT_SMD:SOT-23-5_HandSoldering, symbol 1K_Custom_Symbol:MCP6541
- added R?: 1M, Resistor_SMD:R_0603_1608Metric_Pad1.05x0.95mm_HandSolder, symbol Device:R
- added R?: 3090, Resistor_SMD:R_0603_1608Metric_Pad1.05x0.95mm_HandSolder, symbol Device:R
- added U?: MCP65R46, Package_TO_SOT_SMD:SOT-23-6_Handsoldering, symbol Comparator:MCP65R46
- added U?: FPF2123, Package_TO_SOT_SMD:SOT-23-5_HandSoldering, symbol 1K_Custom_Symbol:FPF2123
Connections:
- wire segments 58 -> 68
Other:
- note added: "150mA current Limit\nset by 3090 Ohm resistor"
- note added: "When %VNTC > NTC, the comparator will be open drain.\nThis indicates it is hot, and the heater sholdn't be on.\nWhen NTC > %VNTC, the comparator will be high impedance \nand the load switch will turn on."
- note removed: "Active High load switch"
- note removed: "When NTC > %VNTC, the comparator will pull high.\nThis indicates it is cold, and the heater should be on."
- moved on the sheet: R?

Commit message: Essentially done with EPS schematic
Parts:
- removed BT?: Battery_Cell, symbol Device:Battery_Cell
- removed F?: Polyfuse, Fuse:Fuse_1206_3216Metric_Pad1.42x1.75mm_HandSolder, symbol Device:Polyfuse
- removed J?: Conn_01x02_Female, symbol Connector:Conn_01x02_Female
- removed R?: R, Resistor_SMD:R_0603_1608Metric_Pad1.05x0.95mm_HandSolder, symbol Device:R
- added R68: 100K, Resistor_SMD:R_0603_1608Metric_Pad1.05x0.95mm_HandSolder, symbol Device:R
- BT1: renamed from BT?; footprint (none) -> footprint_custom:BatteryHolder_Keystone_54_1x18650; Mfr. # (none) -> 54; Order (none) -> https://www.digikey.com/en/products/detail/keystone-electro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
- C24, C26: renamed from C?; Mfr. # (none) -> CL10B104KA8NNNC; Order (none) -> https://www.digikey.com/product-detail/en/samsung-electro-m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; Voltage (none) -> 25V
- C25: renamed from C?; Mfr. # (none) -> C1608X7S1A475K080AC; Order (none) -> https://www.digikey.com/product-detail/en/tdk-corporation/C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; Voltage (none) -> 10V
- F1: renamed from F?; Mfr. # 1206L300SLTHYR -> 1206L380SLTHYR; Order https://www.digikey.com/product-detail/en/littelfuse-inc/12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 -> https://www.digikey.com/en/products/detail/littelfuse-inc/1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
- J2: renamed from J?; footprint (none) -> Connector_PinHeader_1.27mm:PinHeader_1x02_P1.27mm_Vertical
- R67: renamed from R?; value R -> 10K; Mfr. # (none) -> RMCF0603FT10K0; Order (none) -> https://www.digikey.com/en/products/detail/stackpole-electr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
- R69: renamed from R?; value R -> 280K; Mfr. # (none) -> RMCF0603FT280K; Order (none) -> https://www.digikey.com/en/products/detail/stackpole-electr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
- R71: renamed from R?; Mfr. # (none) -> RMCF0603JT1M00; Order (none) -> https://www.digikey.com/en/products/detail/stackpole-electr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
- R72: renamed from R?; value 3090 -> 3.09K; Mfr. # (none) -> RMCF0603FT3K09; Order (none) -> https://www.digikey.com/en/products/detail/stackpole-electr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
- TH1: renamed from TH?; footprint (none) -> Connector_PinHeader_1.27mm:PinHeader_1x02_P1.27mm_Vertical; Mfr. # (none) -> NXFT15XH103FA2B130; Order (none) -> https://www.digikey.com/en/products/detail/murata-electroni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
- gave numbers to parts that had none: 3
Connections:
- wire segments 68 -> 59
Other:
- note added: "2.82A Hold\n8A Trip"
- note added: "<== Rnom"
- note added: "Battery & Fuse"
- note added: "Cold Point= 0C = 2.82*Rnom"
- note added: "Hot point= 50C = 0.41*Rnom"
- note added: "When 73.7% VNTC > NTC, the comparator will be open drain.\nThis indicates it is hot, and the heater should not be on.\nWhen NTC > 73.7% VNTC, the comparator will be high impedance and the load switch will turn on.\nNotice this resistor divider has (nearly) the same ratio as when the NTC is at it's cold point"
- note removed: "Batteries & fuses"
- note removed: "NTC is placed on only 1 battery.\nIt is assumed that one battery's temperature\nwill closely follow the others."
- note removed: "One heater per battery."
- note removed: "When %VNTC > NTC, the comparator will be open drain.\nThis indicates it is hot, and the heater sholdn't be on.\nWhen NTC > %VNTC, the comparator will be high impedance \nand the load switch will turn on."
- moved on the sheet: BT2, F2, R79, TH2

Commit message: EPS layout in progress
Parts:
- BT1: footprint footprint_custom:BatteryHolder_Keystone_54_1x18650 -> footprint_custom:BatteryHolder_Keystone_54_v2_1x18650
Changed lines of the file:
@@
 $Descr A 11000 8500
 encoding utf-8
-Sheet 6 39
+Sheet 4 39
 Title "Battery, Battery Heater, NTC"
 Date "2020-08-11"
@@
 AR Path="/5F39A2F6/5F335E5F" Ref="TH?"  Part="1"
 AR Path="/5F4CFCF6/5F335E5F" Ref="TH2"  Part="1"
-F 0 "TH2" H 2523 4921 50  0000 L CNN
+F 0 "TH1" H 2523 4921 50  0000 L CNN
 F 1 "Thermistor_NTC" H 2523 4830 50  0000 L CNN
 F 2 "Connector_PinHeader_1.27mm:PinHeader_1x02_P1.27mm_Vertical" H 2425 4925 50  0001 C CNN
@@
 AR Path="/5F39A2F6/5F337E75" Ref="R?"  Part="1"
 AR Path="/5F4CFCF6/5F337E75" Ref="R79"  Part="1"
-F 0 "R79" H 2495 4446 50  0000 L CNN
+F 0 "R67" H 2495 4446 50  0000 L CNN
 F 1 "10K" H 2495 4355 50  0000 L CNN
 F 2 "Resistor_SMD:R_0603_1608Metric_Pad1.05x0.95mm_HandSolder" V 2355 4400 50  0001 C CNN
@@
 AR Path="/5F39A2F6/5F45A0CC" Ref="BT?"  Part="1"
 AR Path="/5F4CFCF6/5F45A0CC" Ref="BT2"  Part="1"
-F 0 "BT2" H 7900 4950 50  0000 L CNN
+F 0 "BT1" H 7900 4950 50  0000 L CNN
 F 1 "Battery_Cell" H 7900 4850 50  0000 L CNN
-F 2 "footprint_custom:BatteryHolder_Keystone_54_1x18650" V 7750 4935 50  0001 C CNN
+F 2 "footprint_custom:BatteryHolder_Keystone_54_v2_1x18650" V 7750 4935 50  0001 C CNN
 F 3 "https://www.keyelco.com/product.cfm/product_id/826" V 7750 4935 50  0001 C CNN
 F 4 "54" H 7750 4875 50  0001 C CNN "Mfr. #"
@@
 AR Path="/5F39A2F6/5F467DEB" Ref="R?"  Part="1"
 AR Path="/5F4CFCF6/5F467DEB" Ref="R81"  Part="1"
-F 0 "R81" H 2445 2446 50  0000 L CNN
+F 0 "R69" H 2445 2446 50  0000 L CNN
 F 1 "280K" H 2445 2355 50  0000 L CNN
 F 2 "Resistor_SMD:R_0603_1608Metric_Pad1.05x0.95mm_HandSolder" V 2305 2400 50  0001 C CNN
@@
 AR Path="/5F301C6D/5F47566D" Ref="F1"  Part="1"
 AR Path="/5F4CFCF6/5F47566D" Ref="F2"  Part="1"
-F 0 "F2" H 7850 4550 50  0000 L CNN
+F 0 "F1" H 7850 4550 50  0000 L CNN
 F 1 "Polyfuse" H 7850 4450 50  0000 L CNN
 F 2 "Fuse:Fuse_1206_3216Metric_Pad1.42x1.75mm_HandSolder" H 7800 4275 50  0001 L CNN
@@
 AR Path="/5F301C6D/5F4827E2" Ref="C26"  Part="1"
 AR Path="/5F4CFCF6/5F4827E2" Ref="C31"  Part="1"
-F 0 "C31" H 6800 2600 50  0000 L CNN
+F 0 "C26" H 6800 2600 50  0000 L CNN
 F 1 "0.1uF" H 6800 2500 50  0000 L CNN
 F 2 "Capacitor_SMD:C_0603_1608Metric_Pad1.05x0.95mm_HandSolder" H 6713 2400 50  0001 C CNN
@@
 AR Path="/5F301C6D/5F48BF1E" Ref="C25"  Part="1"
 AR Path="/5F4CFCF6/5F48BF1E" Ref="C30"  Part="1"
-F 0 "C30" H 5040 2596 50  0000 L CNN
+F 0 "C25" H 5040 2596 50  0000 L CNN
 F 1 "4.7uF" H 5040 2505 50  0000 L CNN
 F 2 "Capacitor_SMD:C_0603_1608Metric_Pad1.05x0.95mm_HandSolder" H 4963 2400 50  0001 C CNN
@@
 AR Path="/5F301C6D/5F48FA37" Ref="C24"  Part="1"
 AR Path="/5F4CFCF6/5F48FA37" Ref="C29"  Part="1"
-F 0 "C29" H 2915 1896 50  0000 L CNN
+F 0 "C24" H 2915 1896 50  0000 L CNN
 F 1 "0.1uF" H 2915 1805 50  0000 L CNN
 F 2 "Capacitor_SMD:C_0603_1608Metric_Pad1.05x0.95mm_HandSolder" H 2838 1700 50  0001 C CNN
@@
 AR Path="/5F39A2F6/5F493212" Ref="R?"  Part="1"
 AR Path="/5F4CFCF6/5F493212" Ref="R82"  Part="1"
-F 0 "R82" V 3975 1925 50  0000 C CNN
+F 0 "R70" V 3975 1925 50  0000 C CNN
 F 1 "DNP" V 4175 1925 50  0000 C CNN
 F 2 "Resistor_SMD:R_0603_1608Metric_Pad1.05x0.95mm_HandSolder" V 4005 1925 50  0001 C CNN
@@
 AR Path="/5F301C6D/5F4A0172" Ref="J2"  Part="1"
 AR Path="/5F4CFCF6/5F4A0172" Ref="J4"  Part="1"
-F 0 "J4" H 8503 2126 50  0000 L CNN
+F 0 "J2" H 8503 2126 50  0000 L CNN
 F 1 "Conn_01x02_Female" H 8503 2035 50  0000 L CNN
 F 2 "Connector_PinHeader_1.27mm:PinHeader_1x02_P1.27mm_Vertical" H 8475 2150 50  0001 C CNN
@@
 AR Path="/5F4CFCF6/5FB8079B" Ref="U13"  Part="1"
 AR Path="/5F301C6D/5FB8079B" Ref="U10"  Part="1"
-F 0 "U13" H 3775 2450 50  0000 L CNN
+F 0 "U10" H 3775 2450 50  0000 L CNN
 F 1 "MCP65R46" H 3775 2100 50  0000 L CNN
 F 2 "Package_TO_SOT_SMD:SOT-23-6_Handsoldering" H 3675 2300 50  0001 C CNN
@@
 AR Path="/5F4CFCF6/5FB89477" Ref="U14"  Part="1"
 AR Path="/5F301C6D/5FB89477" Ref="U11"  Part="1"
-F 0 "U14" H 5700 2475 50  0000 C CNN
+F 0 "U11" H 5700 2475 50  0000 C CNN
 F 1 "FPF2123" H 5700 2400 50  0000 C CNN
 F 2 "Package_TO_SOT_SMD:SOT-23-5_HandSoldering" H 5750 1000 50  0001 C CNN
@@
 AR Path="/5F39A2F6/5FB9809C" Ref="R?"  Part="1"
 AR Path="/5F4CFCF6/5FB9809C" Ref="R83"  Part="1"
-F 0 "R83" H 4670 2021 50  0000 L CNN
+F 0 "R71" H 4670 2021 50  0000 L CNN
 F 1 "1M" H 4670 1930 50  0000 L CNN
 F 2 "Resistor_SMD:R_0603_1608Metric_Pad1.05x0.95mm_HandSolder" V 4530 1975 50  0001 C CNN
@@
 AR Path="/5F301C6D/5FBAF948" Ref="R72"  Part="1"
 AR Path="/5F4CFCF6/5FBAF948" Ref="R84"  Part="1"
-F 0 "R84" H 6175 2025 50  0000 C CNN
+F 0 "R72" H 6175 2025 50  0000 C CNN
 F 1 "3.09K" H 6125 2125 50  0000 C CNN
 F 2 "Resistor_SMD:R_0603_1608Metric_Pad1.05x0.95mm_HandSolder" V 6230 2075 50  0001 C CNN
@@
 AR Path="/5F39A2F6/6392F1BF" Ref="R?"  Part="1"
 AR Path="/5F4CFCF6/6392F1BF" Ref="R80"  Part="1"
-F 0 "R80" H 2445 2046 50  0000 L CNN
+F 0 "R68" H 2445 2046 50  0000 L CNN
 F 1 "100K" H 2445 1955 50  0000 L CNN
 F 2 "Resistor_SMD:R_0603_1608Metric_Pad1.05x0.95mm_HandSolder" V 2305 2000 50  0001 C CNN

Commit message: EPS V1.0 Complete
Changed lines of the file:
@@
 $Descr A 11000 8500
 encoding utf-8
-Sheet 4 39
+Sheet 6 39
 Title "Battery, Battery Heater, NTC"
 Date "2020-08-11"
@@
 AR Path="/5F39A2F6/5F335E5F" Ref="TH?"  Part="1"
 AR Path="/5F4CFCF6/5F335E5F" Ref="TH2"  Part="1"
-F 0 "TH1" H 2523 4921 50  0000 L CNN
+F 0 "TH2" H 2523 4921 50  0000 L CNN
 F 1 "Thermistor_NTC" H 2523 4830 50  0000 L CNN
 F 2 "Connector_PinHeader_1.27mm:PinHeader_1x02_P1.27mm_Vertical" H 2425 4925 50  0001 C CNN
@@
 AR Path="/5F39A2F6/5F337E75" Ref="R?"  Part="1"
 AR Path="/5F4CFCF6/5F337E75" Ref="R79"  Part="1"
-F 0 "R67" H 2495 4446 50  0000 L CNN
+F 0 "R79" H 2495 4446 50  0000 L CNN
 F 1 "10K" H 2495 4355 50  0000 L CNN
 F 2 "Resistor_SMD:R_0603_1608Metric_Pad1.05x0.95mm_HandSolder" V 2355 4400 50  0001 C CNN
@@
 AR Path="/5F39A2F6/5F45A0CC" Ref="BT?"  Part="1"
 AR Path="/5F4CFCF6/5F45A0CC" Ref="BT2"  Part="1"
-F 0 "BT1" H 7900 4950 50  0000 L CNN
+F 0 "BT2" H 7900 4950 50  0000 L CNN
 F 1 "Battery_Cell" H 7900 4850 50  0000 L CNN
 F 2 "footprint_custom:BatteryHolder_Keystone_54_v2_1x18650" V 7750 4935 50  0001 C CNN
@@
 AR Path="/5F39A2F6/5F467DEB" Ref="R?"  Part="1"
 AR Path="/5F4CFCF6/5F467DEB" Ref="R81"  Part="1"
-F 0 "R69" H 2445 2446 50  0000 L CNN
+F 0 "R81" H 2445 2446 50  0000 L CNN
 F 1 "280K" H 2445 2355 50  0000 L CNN
 F 2 "Resistor_SMD:R_0603_1608Metric_Pad1.05x0.95mm_HandSolder" V 2305 2400 50  0001 C CNN
@@
 AR Path="/5F301C6D/5F47566D" Ref="F1"  Part="1"
 AR Path="/5F4CFCF6/5F47566D" Ref="F2"  Part="1"
-F 0 "F1" H 7850 4550 50  0000 L CNN
+F 0 "F2" H 7850 4550 50  0000 L CNN
 F 1 "Polyfuse" H 7850 4450 50  0000 L CNN
 F 2 "Fuse:Fuse_1206_3216Metric_Pad1.42x1.75mm_HandSolder" H 7800 4275 50  0001 L CNN
@@
 AR Path="/5F301C6D/5F4827E2" Ref="C26"  Part="1"
 AR Path="/5F4CFCF6/5F4827E2" Ref="C31"  Part="1"
-F 0 "C26" H 6800 2600 50  0000 L CNN
+F 0 "C31" H 6800 2600 50  0000 L CNN
 F 1 "0.1uF" H 6800 2500 50  0000 L CNN
 F 2 "Capacitor_SMD:C_0603_1608Metric_Pad1.05x0.95mm_HandSolder" H 6713 2400 50  0001 C CNN
@@
 AR Path="/5F301C6D/5F48BF1E" Ref="C25"  Part="1"
 AR Path="/5F4CFCF6/5F48BF1E" Ref="C30"  Part="1"
-F 0 "C25" H 5040 2596 50  0000 L CNN
+F 0 "C30" H 5040 2596 50  0000 L CNN
 F 1 "4.7uF" H 5040 2505 50  0000 L CNN
 F 2 "Capacitor_SMD:C_0603_1608Metric_Pad1.05x0.95mm_HandSolder" H 4963 2400 50  0001 C CNN
@@
 AR Path="/5F301C6D/5F48FA37" Ref="C24"  Part="1"
 AR Path="/5F4CFCF6/5F48FA37" Ref="C29"  Part="1"
-F 0 "C24" H 2915 1896 50  0000 L CNN
+F 0 "C29" H 2915 1896 50  0000 L CNN
 F 1 "0.1uF" H 2915 1805 50  0000 L CNN
 F 2 "Capacitor_SMD:C_0603_1608Metric_Pad1.05x0.95mm_HandSolder" H 2838 1700 50  0001 C CNN
@@
 AR Path="/5F39A2F6/5F493212" Ref="R?"  Part="1"
 AR Path="/5F4CFCF6/5F493212" Ref="R82"  Part="1"
-F 0 "R70" V 3975 1925 50  0000 C CNN
+F 0 "R82" V 3975 1925 50  0000 C CNN
 F 1 "DNP" V 4175 1925 50  0000 C CNN
 F 2 "Resistor_SMD:R_0603_1608Metric_Pad1.05x0.95mm_HandSolder" V 4005 1925 50  0001 C CNN
@@
 AR Path="/5F301C6D/5F4A0172" Ref="J2"  Part="1"
 AR Path="/5F4CFCF6/5F4A0172" Ref="J4"  Part="1"
-F 0 "J2" H 8503 2126 50  0000 L CNN
+F 0 "J4" H 8503 2126 50  0000 L CNN
 F 1 "Conn_01x02_Female" H 8503 2035 50  0000 L CNN
 F 2 "Connector_PinHeader_1.27mm:PinHeader_1x02_P1.27mm_Vertical" H 8475 2150 50  0001 C CNN
@@
 AR Path="/5F4CFCF6/5FB8079B" Ref="U13"  Part="1"
 AR Path="/5F301C6D/5FB8079B" Ref="U10"  Part="1"
-F 0 "U10" H 3775 2450 50  0000 L CNN
+F 0 "U13" H 3775 2450 50  0000 L CNN
 F 1 "MCP65R46" H 3775 2100 50  0000 L CNN
 F 2 "Package_TO_SOT_SMD:SOT-23-6_Handsoldering" H 3675 2300 50  0001 C CNN
@@
 AR Path="/5F4CFCF6/5FB89477" Ref="U14"  Part="1"
 AR Path="/5F301C6D/5FB89477" Ref="U11"  Part="1"
-F 0 "U11" H 5700 2475 50  0000 C CNN
+F 0 "U14" H 5700 2475 50  0000 C CNN
 F 1 "FPF2123" H 5700 2400 50  0000 C CNN
 F 2 "Package_TO_SOT_SMD:SOT-23-5_HandSoldering" H 5750 1000 50  0001 C CNN
@@
 AR Path="/5F39A2F6/5FB9809C" Ref="R?"  Part="1"
 AR Path="/5F4CFCF6/5FB9809C" Ref="R83"  Part="1"
-F 0 "R71" H 4670 2021 50  0000 L CNN
+F 0 "R83" H 4670 2021 50  0000 L CNN
 F 1 "1M" H 4670 1930 50  0000 L CNN
 F 2 "Resistor_SMD:R_0603_1608Metric_Pad1.05x0.95mm_HandSolder" V 4530 1975 50  0001 C CNN
@@
 AR Path="/5F301C6D/5FBAF948" Ref="R72"  Part="1"
 AR Path="/5F4CFCF6/5FBAF948" Ref="R84"  Part="1"
-F 0 "R72" H 6175 2025 50  0000 C CNN
+F 0 "R84" H 6175 2025 50  0000 C CNN
 F 1 "3.09K" H 6125 2125 50  0000 C CNN
 F 2 "Resistor_SMD:R_0603_1608Metric_Pad1.05x0.95mm_HandSolder" V 6230 2075 50  0001 C CNN
@@
 AR Path="/5F39A2F6/6392F1BF" Ref="R?"  Part="1"
 AR Path="/5F4CFCF6/6392F1BF" Ref="R80"  Part="1"
-F 0 "R68" H 2445 2046 50  0000 L CNN
+F 0 "R80" H 2445 2046 50  0000 L CNN
 F 1 "100K" H 2445 1955 50  0000 L CNN
 F 2 "Resistor_SMD:R_0603_1608Metric_Pad1.05x0.95mm_HandSolder" V 2305 2000 50  0001 C CNN
