File: eps_board/BATTERY_CHARGER.sch (KiCad schematic (older format))
At the start: 15 parts

Commit message: Progress on EPS
Parts:
- removed D?: D_Schottky, symbol Device:D_Schottky
- removed TP?: TP_1x1, TestPoint:TestPoint_THTPad_1.0x1.0mm_Drill0.5mm, symbol 1K_Custom_Symbol:TP_1x1
- added C?: DNP, symbol Device:C
- added D?: NRVB120VLSFT1G, footprint_custom:D_SOD-123FL_handsolder, symbol Device:D_Schottky
- added R?: 10K, Resistor_SMD:R_0603_1608Metric_Pad1.05x0.95mm_HandSolder, symbol Device:R
- C?: value C -> 4.7uF
- R?: value R -> 10k
- R?: value R -> 1M
Connections:
- net EXT: now also D?.2 (A)
- net GND: now also C?.2, R?.1
- net ISTAT: now also R?.2
- net VOUT: now also D?.1 (K)
- net at C?.1, U?.21 (TIMER): now also C?.1
Other:
- note added: "10K = 10mA"
- note added: "Charge Timer: \n136hours = 3400mAh/25mA charge rate\n136*0.1uF*100k/Rprog/3.0 = Ctimer = 4.5uF"
- note added: "Charge current = 50mA\nIchg(A) = 50000V/1000000"
- note added: "Input current limit = 0.1A\nIcl(A) = 1000V/(10k ohms)"
- moved on the sheet: C?
Changed lines of the file:
@@
 $Descr A 11000 8500
 encoding utf-8
-Sheet 4 14
-Title "BATTERY_CHARGER"
+Sheet 5 39
+Title "LTC4066"
 Date "2020-08-09"
 Rev ""
@@
 $EndBitmap
 $Bitmap
-Pos 5475 7050
+Pos 9525 3450
 Scale 1.000000
 Data
@@
 AR Path="/5F4CFCEF/5F33B731" Ref="R?"  Part="1"
 F 0 "R?" H 3055 4729 50  0000 R CNN
-F 1 "R" H 3055 4820 50  0000 R CNN
+F 1 "10k" H 3055 4820 50  0000 R CNN
 F 2 "Resistor_SMD:R_0603_1608Metric_Pad1.05x0.95mm_HandSolder" V 3055 4775 50  0001 C CNN
 F 3 "~" H 3125 4775 50  0001 C CNN
@@
 L Device:C C?
 U 1 1 5F33BEE4
-P 3750 4775
+P 3550 4775
 AR Path="/5F301C23/5F33BEE4" Ref="C?"  Part="1"
 AR Path="/5F39A2F0/5F33BEE4" Ref="C?"  Part="1"
 AR Path="/5F4CFCEF/5F33BEE4" Ref="C?"  Part="1"
-F 0 "C?" H 3865 4821 50  0000 L CNN
-F 1 "C" H 3865 4730 50  0000 L CNN
-F 2 "" H 3788 4625 50  0001 C CNN
-F 3 "~" H 3750 4775 50  0001 C CNN
-	1    3750 4775
+F 0 "C?" H 3665 4821 50  0000 L CNN
+F 1 "4.7uF" H 3665 4730 50  0000 L CNN
+F 2 "" H 3588 4625 50  0001 C CNN
+F 3 "~" H 3550 4775 50  0001 C CNN
+	1    3550 4775
 	1    0    0    -1
 $EndComp
@@
 AR Path="/5F4CFCEF/5F33EC40" Ref="R?"  Part="1"
 F 0 "R?" H 2455 4729 50  0000 R CNN
-F 1 "R" H 2455 4820 50  0000 R CNN
+F 1 "1M" H 2455 4820 50  0000 R CNN
 F 2 "Resistor_SMD:R_0603_1608Metric_Pad1.05x0.95mm_HandSolder" V 2455 4775 50  0001 C CNN
 F 3 "~" H 2525 4775 50  0001 C CNN
@@
 Wire Wire Line
 	6425 4225 6525 4225
-Text HLabel 8350 4025 2    50   Output ~ 0
+Text HLabel 9500 4025 2    50   Output ~ 0
 ISTAT
 Wire Wire Line
-	6425 4025 6525 4025
-Wire Wire Line
 	1775 5175 2125 5175
 Connection ~ 2525 5175
@@
 Connection ~ 3125 5175
 Wire Wire Line
-	3125 5175 3750 5175
+	3125 5175 3550 5175
 Wire Wire Line
 	2525 4625 2525 4175
-Connection ~ 3750 5175
+Connection ~ 3550 5175
 Wire Wire Line
-	3750 5175 4825 5175
+	3550 5175 4025 5175
 Wire Wire Line
-	4225 4625 3750 4625
+	4225 4625 4025 4625
 Wire Wire Line
 	4225 4425 3125 4425
@@
 	5825 4825 5825 5175
 Wire Wire Line
-	3750 4925 3750 5175
+	3550 4925 3550 5175
 Wire Wire Line
 	3125 4925 3125 5175
@@
 Text HLabel 1800 1700 0    50   Input ~ 0
 EXT
-$Comp
-L Device:D_Schottky D?
-U 1 1 5F37A7F4
-P 5325 1700
-AR Path="/5F301C23/5F37A7F4" Ref="D?"  Part="1"
-AR Path="/5F39A2F0/5F37A7F4" Ref="D?"  Part="1"
-AR Path="/5F4CFCEF/5F37A7F4" Ref="D?"  Part="1"
-F 0 "D?" H 5325 1483 50  0000 C CNN
-F 1 "D_Schottky" H 5325 1574 50  0000 C CNN
-F 2 "" H 5325 1700 50  0001 C CNN
-F 3 "~" H 5325 1700 50  0001 C CNN
-	1    5325 1700
-	-1   0    0    1
-$EndComp
 Wire Wire Line
 	1800 1700 2125 1700
@@
 Wire Wire Line
 	6525 4225 8350 4225
+Wire Wire Line
+	2125 3925 4225 3925
+Wire Wire Line
+	3975 2925 4025 2925
+Connection ~ 4025 2925
 $Comp
-L 1K_Custom_Symbol:TP_1x1 TP?
-U 1 1 5F430011
-P 6600 4075
-AR Path="/5F301C23/5F430011" Ref="TP?"  Part="1"
-AR Path="/5F39A2F0/5F430011" Ref="TP?"  Part="1"
-AR Path="/5F4CFCEF/5F430011" Ref="TP?"  Part="1"
-F 0 "TP?" V 6600 4375 50  0000 C CNN
-F 1 "TP_1x1" V 6675 4150 50  0000 C CNN
-F 2 "TestPoint:TestPoint_THTPad_1.0x1.0mm_Drill0.5mm" H 6800 4075 50  0001 C CNN
-F 3 "~" H 6800 4075 50  0001 C CNN
-	1    6600 4075
-	0    1    1    0
+L Device:D_Schottky D?
+U 1 1 61553601
+P 5325 1700
+AR Path="/61553601" Ref="D?"  Part="1"
+AR Path="/5F301B61/61553601" Ref="D?"  Part="1"
+AR Path="/5F3BB61D/61553601" Ref="D?"  Part="1"
+AR Path="/5F3BED82/61553601" Ref="D?"  Part="1"
+AR Path="/5F3BD959/61553601" Ref="D?"  Part="1"
+AR Path="/5F3BC7D4/61553601" Ref="D?"  Part="1"
+AR Path="/5F3C01C1/61553601" Ref="D?"  Part="1"
+AR Path="/5F301C23/61553601" Ref="D?"  Part="1"
+AR Path="/5F4CFCEF/61553601" Ref="D?"  Part="1"
+F 0 "D?" H 5325 1483 50  0000 C CNN
+F 1 "NRVB120VLSFT1G" H 5325 1574 50  0000 C CNN
+F 2 "footprint_custom:D_SOD-123FL_handsolder" H 5325 1700 50  0001 C CNN
+F 3 "https://www.onsemi.com/pub/Collateral/MBR120VLSFT1-D.PDF" H 5325 1700 50  0001 C CNN
+F 4 "NRVB120VLSFT1G" H 5325 1700 50  0001 C CNN "Mfr. #"
+F 5 "https://www.digikey.com/product-detail/en/on-semiconductor/NRVB120VLSFT1G/NRVB120VLSFT1GOSCT-ND/8538727" H 5325 1700 50  0001 C CNN "Order"
+	1    5325 1700
+	-1   0    0    1
 $EndComp
+$Comp
+L Device:R R?
+U 1 1 5FC28CDC
+P 9150 4200
+AR Path="/5F301C23/5FC28CDC" Ref="R?"  Part="1"
+AR Path="/5F39A2F0/5FC28CDC" Ref="R?"  Part="1"
+AR Path="/5F4CFCEF/5FC28CDC" Ref="R?"  Part="1"
+F 0 "R?" H 9080 4154 50  0000 R CNN
+F 1 "10K" H 9080 4245 50  0000 R CNN
+F 2 "Resistor_SMD:R_0603_1608Metric_Pad1.05x0.95mm_HandSolder" V 9080 4200 50  0001 C CNN
+F 3 "~" H 9150 4200 50  0001 C CNN
+	1    9150 4200
+	-1   0    0    1
+$EndComp
+Text HLabel 9500 4400 2    50   Input ~ 0
+GND
 Wire Wire Line
-	6600 4075 6525 4075
+	9150 4350 9150 4400
 Wire Wire Line
-	6525 4025 6525 4075
-Connection ~ 6525 4025
+	9150 4400 9500 4400
 Wire Wire Line
-	6525 4025 8350 4025
+	9150 4050 9150 4025
+Connection ~ 9150 4025
 Wire Wire Line
-	2125 3925 4225 3925
+	9150 4025 9500 4025
+Text Notes 9425 4225 0    50   ~ 0
+10K = 10mA
+Text Notes 2500 5450 0    50   ~ 0
+Input current limit = 0.1A\nIcl(A) = 1000V/(10k ohms)
+Text Notes 875  4875 0    50   ~ 0
+Charge current = 50mA\nIchg(A) = 50000V/1000000
+Text Notes 3800 5550 0    50   ~ 0
+Charge Timer: \n136hours = 3400mAh/25mA charge rate\n136*0.1uF*100k/Rprog/3.0 = Ctimer = 4.5uF
+$Comp
+L Device:C C?
+U 1 1 5F76909E
+P 4025 4775
+AR Path="/5F301C23/5F76909E" Ref="C?"  Part="1"
+AR Path="/5F39A2F0/5F76909E" Ref="C?"  Part="1"
+AR Path="/5F4CFCEF/5F76909E" Ref="C?"  Part="1"
+F 0 "C?" H 4140 4821 50  0000 L CNN
+F 1 "DNP" H 4140 4730 50  0000 L CNN
+F 2 "" H 4063 4625 50  0001 C CNN
+F 3 "~" H 4025 4775 50  0001 C CNN
+	1    4025 4775
+	1    0    0    -1
+$EndComp
+Connection ~ 4025 4625
 Wire Wire Line
-	3975 2925 4025 2925
-Connection ~ 4025 2925
+	4025 4625 3550 4625
+Wire Wire Line
+	4025 4925 4025 5175
+Connection ~ 4025 5175
+Wire Wire Line
+	4025 5175 4825 5175
+Wire Wire Line
+	6425 4025 9150 4025
 $EndSCHEMATC

Commit message: Essentially done with EPS schematic
Parts:
- added C187, C188, C189: 4.7uF, Capacitor_SMD:C_0603_1608Metric_Pad1.05x0.95mm_HandSolder, symbol Device:C
- added R323, R324: 1, Resistor_SMD:R_0603_1608Metric_Pad1.05x0.95mm_HandSolder, symbol Device:R
- C22: renamed from C?; footprint (none) -> Capacitor_SMD:C_0603_1608Metric_Pad1.05x0.95mm_HandSolder; Mfr. # (none) -> C1608X7S1A475K080AC; Order (none) -> https://www.digikey.com/product-detail/en/tdk-corporation/C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; Voltage (none) -> 10V
- C23: renamed from C?; footprint (none) -> Capacitor_SMD:C_0603_1608Metric_Pad1.05x0.95mm_HandSolder
- R61: renamed from R?; Mfr. # (none) -> RK73H1JTTD2672F; Order (none) -> https://www.digikey.com/en/products/detail/koa-speer-electr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
- R62, R66: renamed from R?; Mfr. # (none) -> RMCF0603FT10K0; Order (none) -> https://www.digikey.com/en/products/detail/stackpole-electr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
- R63: renamed from R?; Mfr. # (none) -> RMCF0603JT1M00; Order (none) -> https://www.digikey.com/en/products/detail/stackpole-electr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
- R64: renamed from R?; value 10k -> 10K; Mfr. # (none) -> RMCF0603FT10K0; Order (none) -> https://www.digikey.com/en/products/detail/stackpole-electr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
- R65: renamed from R?; Mfr. # (none) -> RMCF0603FT100K; Order (none) -> https://www.digikey.com/en/products/detail/stackpole-electr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
- gave numbers to parts that had none: 8
Connections:
- net BAT: now also C189.1
- net GND: now also C188.2, R323.2, R324.1
- net VIN: now also C187.1
- net VOUT: now also C188.1
- new net: C189.2, R324.2
- new net: C187.2, R323.1

Commit message: EPS V1.0 Complete
Parts:
- U9: footprint Package_DFN_QFN:QFN-24-1EP_4x4mm_P0.5mm_EP2.6x2.6mm_ThermalVias -> footprint_custom:QFN-24-1EP_4x4mm_P0.5mm_EP2.6x2.6mm_0.4mmThermalVias
Changed lines of the file:
@@
 $Descr A 11000 8500
 encoding utf-8
-Sheet 5 39
+Sheet 3 39
 Title "LTC4066"
 Date "2020-08-09"
@@
 F 0 "U12" H 5325 4790 50  0000 C CNN
 F 1 "LTC4066" H 5325 4699 50  0000 C CNN
-F 2 "Package_DFN_QFN:QFN-24-1EP_4x4mm_P0.5mm_EP2.6x2.6mm_ThermalVias" H 5275 1725 50  0001 C CNN
+F 2 "footprint_custom:QFN-24-1EP_4x4mm_P0.5mm_EP2.6x2.6mm_0.4mmThermalVias" H 5275 1725 50  0001 C CNN
 F 3 "https://www.analog.com/media/en/technical-documentation/data-sheets/4066fc.pdf" H 5325 3625 50  0001 C CNN
 F 4 "LTC4066EUF#PBF" H 5325 3725 50  0001 C CNN "Mfr. #"
