File: eps_board/CURRENT_MONITOR.sch (KiCad schematic (older format))
At the start: 22 parts

Commit message: Essentially done with EPS schematic
Parts:
- C47, C49, C50, C53: renamed from C?; Mfr. # (none) -> CL10B104KA8NNNC; Order (none) -> https://www.digikey.com/product-detail/en/samsung-electro-m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; Voltage (none) -> 25V
- C51: renamed from C?; Mfr. # (none) -> CL10B105KP8NFNC; Order (none) -> https://www.digikey.com/product-detail/en/samsung-electro-m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; Voltage (none) -> 10V
- C52: renamed from C?; Mfr. # (none) -> C1608X7S1A475K080AC; Order (none) -> https://www.digikey.com/product-detail/en/tdk-corporation/C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; Voltage (none) -> 10V
- R143, R146, R149: renamed from R?; Mfr. # (none) -> RK73Z1JTTD; Order (none) -> https://www.digikey.com/product-detail/en/koa-speer-electro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
- R144: renamed from R?; value 100k -> 100K; Mfr. # (none) -> RMCF0603FT100K; Order (none) -> https://www.digikey.com/en/products/detail/stackpole-electr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
- R145, R147, R148: renamed from R?; Mfr. # (none) -> RMCF0603JT1M00; Order (none) -> https://www.digikey.com/en/products/detail/stackpole-electr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
- gave numbers to parts that had none: 9

Commit message: EPS layout in progress
Parts:
- removed R146: 0, Resistor_SMD:R_0603_1608Metric_Pad1.05x0.95mm_HandSolder, symbol Device:R
- C46, C48: footprint Capacitor_SMD:C_0603_1608Metric_Pad1.05x0.95mm_HandSolder -> Capacitor_SMD:C_0603_1608Metric
- Q1, Q2: footprint Package_TO_SOT_SMD:SOT-23_Handsoldering -> Package_TO_SOT_SMD:SOT-23
- U19: footprint Package_TO_SOT_SMD:SOT-363_SC-70-6_Handsoldering -> Package_TO_SOT_SMD:SOT-363_SC-70-6
- U20: footprint Package_TO_SOT_SMD:SOT-353_SC-70-5_Handsoldering -> Package_TO_SOT_SMD:SOT-353_SC-70-5; symbol 74xGxx:74LVC1G07 -> 1K_Custom_Symbol:74LVC1G07
- U21: footprint Package_TO_SOT_SMD:SOT-23-6_Handsoldering -> Package_TO_SOT_SMD:SOT-23-6
Connections:
- net at C51.2, R145.1, U20.4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: now also Q1.1 (G)
- net VCC: no longer names the net of C47.1, C49.2, C50.2, R143.1, R150.2, U19.3 (Vs), U20.5, U21.6 (V+)
Other:
- moved on the sheet: C155, R249

Commit message: EPS V1.0 Complete
Changed lines of the file:
@@
 $Descr A 11000 8500
 encoding utf-8
-Sheet 24 39
+Sheet 14 39
 Title "Current Monitor"
 Date "2020-09-06"
@@
 AR Path="/60177EB3/620FFEBA/5F9ECAFD" Ref="U?"  Part="1"
 AR Path="/60177EB3/620FFEC8/5F9ECAFD" Ref="U?"  Part="1"
-F 0 "U71" H 2075 4375 50  0000 C CNN
+F 0 "U79" H 2075 4375 50  0000 C CNN
 F 1 "NCS211" H 2050 3725 50  0000 C CNN
 F 2 "Package_TO_SOT_SMD:SOT-363_SC-70-6" H 2325 4025 50  0001 C CNN
@@
 AR Path="/60177EB3/620FFEBA/5F9ECB1A" Ref="U?"  Part="1"
 AR Path="/60177EB3/620FFEC8/5F9ECB1A" Ref="U?"  Part="1"
-F 0 "U73" H 4825 4075 50  0000 L CNN
+F 0 "U81" H 4825 4075 50  0000 L CNN
 F 1 "MCP65R46" H 4825 3725 50  0000 L CNN
 F 2 "Package_TO_SOT_SMD:SOT-23-6" H 4725 3925 50  0001 C CNN
@@
 AR Path="/60177EB3/620FFEBA/5F9ECB21" Ref="R?"  Part="1"
 AR Path="/60177EB3/620FFEC8/5F9ECB21" Ref="R?"  Part="1"
-F 0 "R248" H 3750 4600 50  0000 C CNN
+F 0 "R264" H 3750 4600 50  0000 C CNN
 F 1 "100K" H 3750 4700 50  0000 C CNN
 F 2 "Resistor_SMD:R_0603_1608Metric_Pad1.05x0.95mm_HandSolder" V 3530 4650 50  0001 C CNN
@@
 AR Path="/60177EB3/620FFEBA/5FA1CB12" Ref="R?"  Part="1"
 AR Path="/60177EB3/620FFEC8/5FA1CB12" Ref="R?"  Part="1"
-F 0 "R247" H 2500 1900 50  0000 C CNN
+F 0 "R263" H 2500 1900 50  0000 C CNN
 F 1 "0" H 2225 2050 50  0000 C CNN
 F 2 "Resistor_SMD:R_0603_1608Metric_Pad1.05x0.95mm_HandSolder" V 2255 1975 50  0001 C CNN
@@
 AR Path="/60177EB3/620FFEBA/5FA1D16A" Ref="R?"  Part="1"
 AR Path="/60177EB3/620FFEC8/5FA1D16A" Ref="R?"  Part="1"
-F 0 "R254" V 7600 3125 50  0000 C CNN
+F 0 "R270" V 7600 3125 50  0000 C CNN
 F 1 "DNP" V 7775 3125 50  0000 C CNN
 F 2 "Resistor_SMD:R_0603_1608Metric_Pad1.05x0.95mm_HandSolder" V 7630 3125 50  0001 C CNN
@@
 AR Path="/60177EB3/620FFEBA/5FA244B4" Ref="C?"  Part="1"
 AR Path="/60177EB3/620FFEC8/5FA244B4" Ref="C?"  Part="1"
-F 0 "C154" V 4750 3550 50  0000 L CNN
+F 0 "C170" V 4750 3550 50  0000 L CNN
 F 1 "0.1uF" V 4750 3275 50  0000 L CNN
 F 2 "Capacitor_SMD:C_0603_1608Metric_Pad1.05x0.95mm_HandSolder" H 4913 3350 50  0001 C CNN
@@
 AR Path="/60177EB3/620FFEBA/5FA34D09" Ref="U?"  Part="1"
 AR Path="/60177EB3/620FFEC8/5FA34D09" Ref="U?"  Part="1"
-F 0 "U74" H 8075 2615 50  0000 C CNN
+F 0 "U82" H 8075 2615 50  0000 C CNN
 F 1 "FPF2123" H 8075 2524 50  0000 C CNN
 F 2 "Package_TO_SOT_SMD:SOT-23-5_HandSoldering" H 8125 1100 50  0001 C CNN
@@
 AR Path="/60177EB3/620FFEBA/5FA3E628" Ref="C?"  Part="1"
 AR Path="/60177EB3/620FFEC8/5FA3E628" Ref="C?"  Part="1"
-F 0 "C156" H 7275 2150 50  0000 L CNN
+F 0 "C172" H 7275 2150 50  0000 L CNN
 F 1 "4.7uF" H 7275 2325 50  0000 L CNN
 F 2 "Capacitor_SMD:C_0603_1608Metric_Pad1.05x0.95mm_HandSolder" H 7538 2075 50  0001 C CNN
@@
 AR Path="/60177EB3/620FFEBA/5FA4AE93" Ref="R?"  Part="1"
 AR Path="/60177EB3/620FFEC8/5FA4AE93" Ref="R?"  Part="1"
-F 0 "R252" H 6975 1375 50  0000 C CNN
+F 0 "R268" H 6975 1375 50  0000 C CNN
 F 1 "1M" H 6950 1525 50  0000 C CNN
 F 2 "Resistor_SMD:R_0603_1608Metric_Pad1.05x0.95mm_HandSolder" V 6755 1450 50  0001 C CNN
@@
 AR Path="/60177EB3/620FFEBA/5FA5478F" Ref="C?"  Part="1"
 AR Path="/60177EB3/620FFEC8/5FA5478F" Ref="C?"  Part="1"
-F 0 "C157" H 8375 2150 50  0000 L CNN
+F 0 "C173" H 8375 2150 50  0000 L CNN
 F 1 "0.1uF" H 8350 2325 50  0000 L CNN
 F 2 "Capacitor_SMD:C_0603_1608Metric_Pad1.05x0.95mm_HandSolder" H 8638 2075 50  0001 C CNN
@@
 AR Path="/60177EB3/620FFEBA/5FD8572E" Ref="C?"  Part="1"
 AR Path="/60177EB3/620FFEC8/5FD8572E" Ref="C?"  Part="1"
-F 0 "C152" H 2850 4575 50  0000 L CNN
+F 0 "C168" H 2850 4575 50  0000 L CNN
 F 1 "DNP" H 2875 4350 50  0000 L CNN
 F 2 "Capacitor_SMD:C_0603_1608Metric" H 3113 4300 50  0001 C CNN
@@
 AR Path="/60177EB3/620FFEBA/5FD8CD80" Ref="C?"  Part="1"
 AR Path="/60177EB3/620FFEC8/5FD8CD80" Ref="C?"  Part="1"
-F 0 "C150" H 1725 4150 50  0000 L CNN
+F 0 "C166" H 1725 4150 50  0000 L CNN
 F 1 "DNP" H 1675 3925 50  0000 L CNN
 F 2 "Capacitor_SMD:C_0603_1608Metric" H 1663 3875 50  0001 C CNN
@@
 AR Path="/60177EB3/620FFEBA/5F58A815" Ref="C?"  Part="1"
 AR Path="/60177EB3/620FFEC8/5F58A815" Ref="C?"  Part="1"
-F 0 "C155" H 5450 4400 50  0000 L CNN
+F 0 "C171" H 5450 4400 50  0000 L CNN
 F 1 "1uF" H 5500 4475 50  0000 L CNN
 F 2 "Capacitor_SMD:C_0603_1608Metric_Pad1.05x0.95mm_HandSolder" H 5788 4300 50  0001 C CNN
@@
 AR Path="/60177EB3/620FFEBA/5F647D01" Ref="R?"  Part="1"
 AR Path="/60177EB3/620FFEC8/5F647D01" Ref="R?"  Part="1"
-F 0 "R249" H 5925 3325 50  0000 C CNN
+F 0 "R265" H 5925 3325 50  0000 C CNN
 F 1 "1M" H 5875 3450 50  0000 C CNN
 F 2 "Resistor_SMD:R_0603_1608Metric_Pad1.05x0.95mm_HandSolder" V 5680 3375 50  0001 C CNN
@@
 AR Path="/60177EB3/620FFEBA/61F1D561" Ref="U?"  Part="1"
 AR Path="/60177EB3/620FFEC8/61F1D561" Ref="U?"  Part="1"
-F 0 "U72" H 3625 2550 50  0000 C CNN
+F 0 "U80" H 3625 2550 50  0000 C CNN
 F 1 "74LVC1G07" H 4125 2375 50  0000 C CNN
 F 2 "Package_TO_SOT_SMD:SOT-353_SC-70-5" H 3875 2450 50  0001 C CNN
@@
 AR Path="/60177EB3/620FFEBA/61F20F44" Ref="C?"  Part="1"
 AR Path="/60177EB3/620FFEC8/61F20F44" Ref="C?"  Part="1"
-F 0 "C153" V 3950 2300 50  0000 L CNN
+F 0 "C169" V 3950 2300 50  0000 L CNN
 F 1 "0.1uF" V 3950 2025 50  0000 L CNN
 F 2 "Capacitor_SMD:C_0603_1608Metric_Pad1.05x0.95mm_HandSolder" H 4113 2100 50  0001 C CNN
@@
 AR Path="/60177EB3/620FFEBA/61F63EEF" Ref="R?"  Part="1"
 AR Path="/60177EB3/620FFEC8/61F63EEF" Ref="R?"  Part="1"
-F 0 "R251" H 6450 3325 50  0000 C CNN
+F 0 "R267" H 6450 3325 50  0000 C CNN
 F 1 "1M" H 6400 3450 50  0000 C CNN
 F 2 "Resistor_SMD:R_0603_1608Metric_Pad1.05x0.95mm_HandSolder" V 6205 3375 50  0001 C CNN
@@
 AR Path="/60177EB3/620FFEBA/61FD78C4" Ref="C?"  Part="1"
 AR Path="/60177EB3/620FFEC8/61FD78C4" Ref="C?"  Part="1"
-F 0 "C151" V 1925 3550 50  0000 L CNN
+F 0 "C167" V 1925 3550 50  0000 L CNN
 F 1 "0.1uF" V 1925 3275 50  0000 L CNN
 F 2 "Capacitor_SMD:C_0603_1608Metric_Pad1.05x0.95mm_HandSolder" H 2088 3350 50  0001 C CNN
@@
 AR Path="/60177EB3/620FFEBA/620C88DE" Ref="R?"  Part="1"
 AR Path="/60177EB3/620FFEC8/620C88DE" Ref="R?"  Part="1"
-F 0 "R253" H 6675 3300 50  0000 C CNN
+F 0 "R269" H 6675 3300 50  0000 C CNN
 F 1 "0" H 6750 3425 50  0000 C CNN
 F 2 "Resistor_SMD:R_0603_1608Metric_Pad1.05x0.95mm_HandSolder" V 6755 3375 50  0001 C CNN
@@
 AR Path="/60177EB3/620FFEBA/620F5F48" Ref="Q?"  Part="1"
 AR Path="/60177EB3/620FFEC8/620F5F48" Ref="Q?"  Part="1"
-F 0 "Q28" H 6925 3850 50  0000 L CNN
+F 0 "Q32" H 6925 3850 50  0000 L CNN
 F 1 "2N7002K" H 6850 3775 50  0000 L CNN
 F 2 "Package_TO_SOT_SMD:SOT-23" H 6925 3850 50  0001 L CIN
@@
 AR Path="/60177EB3/620FFEBA/620FC359" Ref="Q?"  Part="1"
 AR Path="/60177EB3/620FFEC8/620FC359" Ref="Q?"  Part="1"
-F 0 "Q27" H 6375 3850 50  0000 L CNN
+F 0 "Q31" H 6375 3850 50  0000 L CNN
 F 1 "2N7002K" H 6300 3775 50  0000 L CNN
 F 2 "Package_TO_SOT_SMD:SOT-23" H 6375 3850 50  0001 L CIN
