File: eps_board/EPS.kicad_pcb (KiCad board)
At the start: 2 copper layers, 705 parts, among them J1 Conn_01x04_MountingPin, J10 Conn_01x04_MountingPin, J11 Conn_01x04_MountingPin, J12 Conn_01x05, J13 Conn_01x04_Male, J14 USB_B_Micro, J2 Conn_01x02_Female, J4 Conn_01x02_Female, J6 Conn_02x20_Odd_Even, J7 Conn_01x04_MountingPin, J8 Conn_01x04_MountingPin, J9 Conn_01x04_MountingPin, Q1 2N7002K, Q10 2N7002K, Q11 2N7002K, Q12 2N7002K, Q13 2N7002K, Q14 2N7002K, Q15 2N7002K, Q16 2N7002K, Q17 2N7002K, Q18 2N7002K, Q19 2N7002K, Q2 2N7002K, Q20 2N7002K, Q21 2N7002K, Q22 2N7002K, Q23 2N7002K, Q24 2N7002K, Q25 2N7002K, Q26 2N7002K, Q27 2N7002K, Q28 2N7002K, Q29 2N7002K, Q3 2N7002K, Q30 2N7002K, Q31 2N7002K, Q32 2N7002K, Q4 2N7002K, Q5 2N7002K, Q6 2N7002K, Q7 2N7002K, Q8 2N7002K, Q9 2N7002K, SW1 SW_DIP_x01, SW2 SW_Push, U1 STM32L496ZGTx, U10 MCP65R46, U11 FPF2123, U12 LTC4066, U13 MCP65R46, U14 FPF2123, U15 LTC4415, U16 LTC3130-1, U17 TPS270, U18 TPS270, U19 NCS211, U2 MR25H10, U20 74LVC1G07, U21 MCP65R46, U22 FPF2123, U23 NCS211, U24 74LVC1G07, U25 MCP65R46, U26 FPF2123, U27 NCS211, U28 74LVC1G07, U29 MCP65R46, U3 TPL5010, U30 FPF2123, U31 NCS211, U32 74LVC1G07, U33 MCP65R46, U34 FPF2123, U35 NCS211, U36 74LVC1G07, U37 MCP65R46, U38 FPF2123, U39 NCS211, U4 TPS270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

Commit message: EPS layout in progress
Parts:
- removed J10, J11: Conn_01x04_MountingPin, Connector_Molex:Molex_Pico-Lock_504050-0491_1x04-1MP_P1.50mm_Horizontal
- removed R146, R154, R162, R170, R178, R186, R194, R202, R210, R218, R226, R234, R242, R250, R258, R266, R271, R272, R273, R274, R275, R276, R277, R278, R279, R280, R281, R282, R283, R284, R285, R286, R287, R288, R289, R290, R291, R292, R293, R294, R295, R296, R297, R298, R299, R300, R301, R302, R303: 0, Resistor_SMD:R_0603_1608Metric_Pad1.05x0.95mm_HandSolder
- removed R44, R45: 100K, Resistor_SMD:R_0603_1608Metric_Pad1.05x0.95mm_HandSolder
- removed TP6: TP_1.5x1.5, TestPoint:TestPoint_THTPad_1.5x1.5mm_Drill0.7mm
- added H1: MountingHole, MountingHole:MountingHole_2.1mm, F.Cu at (150.2, 129.5)
- added H2: MountingHole_Pad, MountingHole:MountingHole_3.2mm_M3_Pad_Via, F.Cu at (172.9, 139.0)
- added H3: MountingHole_Pad, MountingHole:MountingHole_3.2mm_M3_Pad_Via, F.Cu at (98.0, 139.0)
- added H4: MountingHole_Pad, MountingHole:MountingHole_3.2mm_M3_Pad_Via, F.Cu at (98.0, 64.0)
- added H5: MountingHole_Pad, MountingHole:MountingHole_3.2mm_M3_Pad_Via, F.Cu at (172.9, 64.0)
- added J3: Conn_01x04, Connector_PinHeader_2.54mm:PinHeader_1x04_P2.54mm_Vertical, F.Cu at (175.9, 80.9)
- added J5: Conn_01x04, Connector_PinHeader_2.54mm:PinHeader_1x04_P2.54mm_Vertical, F.Cu at (175.9, 92.2)
- BT1, BT2: footprint footprint_custom:BatteryHolder_Keystone_54_1x18650 -> footprint_custom:BatteryHolder_Keystone_54_v2_1x18650
- C1, C10, C103, C105, C106, C107, C108, C109, C11, C12, C13, C14, C143, C145, C146, C147, C148, C149, C15, C151, C153, C154, C155, C156, C157, C159, C16, C161, C162, C163, C164, C165, C17, C18, C2, C3, C32, C33, C34, C35, C37, C38, C39, C4, C40, C41, C42, C43, C5, C6, C7, C8, C9, D9, L1, R1, R110, R117, R118, R12, R13, R131, R132, R133, R135, R136, R137, R138, R139, R140, R16, R17, R18, R199, R200, R201, R203, R204, R205, R206, R239, R240, R241, R243, R244, R245, R246, R247, R248, R249, R251, R252, R253, R254, R255, R256, R257, R259, R260, R261, R262, R304, R305, R32, R33, R34, R35, R36, R37, R38, R39, R40, R41, R42, R43, R46, R47, R48, R49, R5, R50, R51, R52, R6, R7, R87, R88, R89, R90, U1, U16, U2, U5, U50, U70, U74, U78, U8: moved to B.Cu
- C102, C104, C142, C144, C150, C152, C158, C160: footprint Capacitor_SMD:C_0603_1608Metric_Pad1.05x0.95mm_HandSolder -> Capacitor_SMD:C_0603_1608Metric; moved to B.Cu
- C110, C112, C118, C120, C126, C128, C134, C136, C166, C168, C46, C48, C54, C56, C62, C64, C70, C72, C78, C80, C86, C88, C94, C96: footprint Capacitor_SMD:C_0603_1608Metric_Pad1.05x0.95mm_HandSolder -> Capacitor_SMD:C_0603_1608Metric
- J1, J7, J8, J9: value Conn_01x04_MountingPin -> Conn_01x04; footprint Connector_Molex:Molex_Pico-Lock_504050-0491_1x04-1MP_P1.50mm_Horizontal -> Connector_PinHeader_2.54mm:PinHeader_1x04_P2.54mm_Vertical
- Q1, Q10, Q11, Q12, Q13, Q14, Q17, Q18, Q19, Q2, Q20, Q21, Q22, Q23, Q24, Q3, Q31, Q32, Q4, Q5, Q6, Q7, Q8, Q9: footprint Package_TO_SOT_SMD:SOT-23_Handsoldering -> Package_TO_SOT_SMD:SOT-23
- Q15, Q16, Q25, Q26, Q27, Q28, Q29, Q30: footprint Package_TO_SOT_SMD:SOT-23_Handsoldering -> Package_TO_SOT_SMD:SOT-23; moved to B.Cu
- TP1, TP2, TP4, TP5: footprint TestPoint:TestPoint_Pad_1.0x1.0mm -> TestPoint:TestPoint_THTPad_1.0x1.0mm_Drill0.5mm; moved to B.Cu
- TP3: value TP_1.5x1.5 -> TP_smt_1x1; footprint TestPoint:TestPoint_THTPad_1.5x1.5mm_Drill0.7mm -> TestPoint:TestPoint_THTPad_1.0x1.0mm_Drill0.5mm; moved to B.Cu
- TP8, TP9: footprint TestPoint:TestPoint_Pad_1.0x1.0mm -> TestPoint:TestPoint_THTPad_1.0x1.0mm_Drill0.5mm
- U19, U23, U27, U31, U35, U39, U43, U51, U55, U59, U63, U79: footprint Package_TO_SOT_SMD:SOT-363_SC-70-6_Handsoldering -> Package_TO_SOT_SMD:SOT-363_SC-70-6
- U20, U24, U28, U32, U36, U40, U44, U52, U56, U60, U64, U80: footprint Package_TO_SOT_SMD:SOT-353_SC-70-5_Handsoldering -> Package_TO_SOT_SMD:SOT-353_SC-70-5
- U21, U25, U29, U33, U37, U41, U45, U53, U57, U61, U65, U81: footprint Package_TO_SOT_SMD:SOT-23-6_Handsoldering -> Package_TO_SOT_SMD:SOT-23-6
- U47, U67, U71, U75: footprint Package_TO_SOT_SMD:SOT-363_SC-70-6_Handsoldering -> Package_TO_SOT_SMD:SOT-363_SC-70-6; moved to B.Cu
- U48, U68, U72, U76: footprint Package_TO_SOT_SMD:SOT-353_SC-70-5_Handsoldering -> Package_TO_SOT_SMD:SOT-353_SC-70-5; moved to B.Cu
- U49, U69, U73, U77: footprint Package_TO_SOT_SMD:SOT-23-6_Handsoldering -> Package_TO_SOT_SMD:SOT-23-6; moved to B.Cu
- moved C86 198.9 mm to (123.2, 94.6)
- moved C89 196.0 mm to (123.3, 97.7)
- moved R187 195.2 mm to (122.3, 81.0), turned to 90 degrees
- moved R183 194.8 mm to (123.3, 96.2), turned to 180 degrees
- moved C93 192.7 mm to (123.2, 85.1), turned to 180 degrees
- moved U42 189.5 mm to (123.2, 88.3), turned to 90 degrees
- moved R185 188.8 mm to (126.8, 83.5), turned to 180 degrees
- moved R188 187.6 mm to (123.3, 99.3)
- moved C92 186.7 mm to (123.3, 91.5), turned to 180 degrees
- moved R196 186.3 mm to (121.6, 75.3), turned to 270 degrees
- moved U39 185.6 mm to (126.6, 94.5), turned to 180 degrees
- moved C90 184.4 mm to (128.9, 91.4), turned to 270 degrees
- moved R184 182.6 mm to (125.8, 91.4), turned to 90 degrees
- moved C94 180.4 mm to (124.4, 74.7)
- moved R189 180.0 mm to (120.6, 88.0), turned to 90 degrees
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Connections:
- C103 pad 1: +3V3 -> Net-(C103-Pad1)
- C105 pad 2: +3V3 -> Net-(C103-Pad1)
- C106 pad 2: +3V3 -> Net-(C103-Pad1)
- C111 pad 1: +3V3 -> Net-(C111-Pad1)
- C113 pad 2: +3V3 -> Net-(C111-Pad1)
- C114 pad 2: +3V3 -> Net-(C111-Pad1)
- C119 pad 1: +3V3 -> Net-(C119-Pad1)
- C121 pad 2: +3V3 -> Net-(C119-Pad1)
- C122 pad 2: +3V3 -> Net-(C119-Pad1)
- C127 pad 1: +3V3 -> Net-(C127-Pad1)
- C129 pad 2: +3V3 -> Net-(C127-Pad1)
- C130 pad 2: +3V3 -> Net-(C127-Pad1)
- C135 pad 1: +3V3 -> Net-(C135-Pad1)
- C137 pad 2: +3V3 -> Net-(C135-Pad1)
- C138 pad 2: +3V3 -> Net-(C135-Pad1)
- C143 pad 1: +3V3 -> Net-(C143-Pad1)
- C145 pad 2: +3V3 -> Net-(C143-Pad1)
- C146 pad 2: +3V3 -> Net-(C143-Pad1)
- C151 pad 1: +3V3 -> Net-(C151-Pad1)
- C153 pad 2: +3V3 -> Net-(C151-Pad1)
- C154 pad 2: +3V3 -> Net-(C151-Pad1)
- C159 pad 1: +3V3 -> Net-(C159-Pad1)
- C161 pad 2: +3V3 -> Net-(C159-Pad1)
- C162 pad 2: +3V3 -> Net-(C159-Pad1)
- C167 pad 1: +3V3 -> Net-(C167-Pad1)
- C169 pad 2: +3V3 -> Net-(C167-Pad1)
- C170 pad 2: +3V3 -> Net-(C167-Pad1)
- C18 pad 1: /3.3V_EPS_MRAM -> Net-(C18-Pad1)
- C36 pad 1: /PMIC/3.3V_STM_CORE -> Net-(C36-Pad1)
- C47 pad 1: +3V3 -> Net-(C47-Pad1)
- C49 pad 2: +3V3 -> Net-(C47-Pad1)
- C50 pad 2: +3V3 -> Net-(C47-Pad1)
- C55 pad 1: +3V3 -> Net-(C55-Pad1)
- C57 pad 2: +3V3 -> Net-(C55-Pad1)
- C58 pad 2: +3V3 -> Net-(C55-Pad1)
- C63 pad 1: +3V3 -> Net-(C63-Pad1)
- C65 pad 2: +3V3 -> Net-(C63-Pad1)
- C66 pad 2: +3V3 -> Net-(C63-Pad1)
- C71 pad 1: +3V3 -> Net-(C71-Pad1)
- C73 pad 2: +3V3 -> Net-(C71-Pad1)
- C74 pad 2: +3V3 -> Net-(C71-Pad1)
- C79 pad 1: +3V3 -> Net-(C79-Pad1)
- C81 pad 2: +3V3 -> Net-(C79-Pad1)
- C82 pad 2: +3V3 -> Net-(C79-Pad1)
- C87 pad 1: +3V3 -> Net-(C87-Pad1)
- C89 pad 2: +3V3 -> Net-(C87-Pad1)
- C90 pad 2: +3V3 -> Net-(C87-Pad1)
- C95 pad 1: +3V3 -> Net-(C95-Pad1)
- C97 pad 2: +3V3 -> Net-(C95-Pad1)
- C98 pad 2: +3V3 -> Net-(C95-Pad1)
- D18 pad 1: /VEXT -> Net-(D18-Pad1)
- J14 pad 1: Net-(J14-Pad1) -> Net-(D18-Pad1)
- J7 pad 1: Net-(D13-Pad2) -> Net-(D15-Pad2)
- J7 pad 2: Net-(D13-Pad2) -> Net-(D15-Pad2)
- J8 pad 1: Net-(D14-Pad2) -> Net-(D16-Pad2)
- J8 pad 2: Net-(D14-Pad2) -> Net-(D16-Pad2)
- J9 pad 1: Net-(D15-Pad2) -> Net-(D17-Pad2)
- J9 pad 2: Net-(D15-Pad2) -> Net-(D17-Pad2)
- Q1 pad 1: Net-(Q1-Pad1) -> Net-(C51-Pad2)
- Q11 pad 1: Net-(Q11-Pad1) -> Net-(C91-Pad2)
- Q13 pad 1: Net-(Q13-Pad1) -> Net-(C99-Pad2)
- Q15 pad 1: Net-(Q15-Pad1) -> Net-(C107-Pad2)
- Q17 pad 1: Net-(Q17-Pad1) -> Net-(C115-Pad2)
- Q19 pad 1: Net-(Q19-Pad1) -> Net-(C123-Pad2)
- Q21 pad 1: Net-(Q21-Pad1) -> Net-(C131-Pad2)
- Q23 pad 1: Net-(Q23-Pad1) -> Net-(C139-Pad2)
- Q25 pad 1: Net-(Q25-Pad1) -> Net-(C147-Pad2)
- Q27 pad 1: Net-(Q27-Pad1) -> Net-(C155-Pad2)
- Q29 pad 1: Net-(Q29-Pad1) -> Net-(C163-Pad2)
- Q3 pad 1: Net-(Q3-Pad1) -> Net-(C59-Pad2)
- Q31 pad 1: Net-(Q31-Pad1) -> Net-(C171-Pad2)
- Q5 pad 1: Net-(Q5-Pad1) -> Net-(C67-Pad2)
- Q7 pad 1: Net-(Q7-Pad1) -> Net-(C75-Pad2)
- Q9 pad 1: Net-(Q9-Pad1) -> Net-(C83-Pad2)
- R143 pad 1: +3V3 -> Net-(C47-Pad1)
- R150 pad 2: +3V3 -> Net-(C47-Pad1)
- R151 pad 1: +3V3 -> Net-(C55-Pad1)
- R158 pad 2: +3V3 -> Net-(C55-Pad1)
- R159 pad 1: +3V3 -> Net-(C63-Pad1)
- R166 pad 2: +3V3 -> Net-(C63-Pad1)
- R167 pad 1: +3V3 -> Net-(C71-Pad1)
- R174 pad 2: +3V3 -> Net-(C71-Pad1)
- R175 pad 1: +3V3 -> Net-(C79-Pad1)
- R182 pad 2: +3V3 -> Net-(C79-Pad1)
- R183 pad 1: +3V3 -> Net-(C87-Pad1)
- R190 pad 2: +3V3 -> Net-(C87-Pad1)
- R191 pad 1: +3V3 -> Net-(C95-Pad1)
- R198 pad 2: +3V3 -> Net-(C95-Pad1)
- R199 pad 1: +3V3 -> Net-(C103-Pad1)
- R206 pad 2: +3V3 -> Net-(C103-Pad1)
- R207 pad 1: +3V3 -> Net-(C111-Pad1)
- R214 pad 2: +3V3 -> Net-(C111-Pad1)
- R215 pad 1: +3V3 -> Net-(C119-Pad1)
- R222 pad 2: +3V3 -> Net-(C119-Pad1)
- R223 pad 1: +3V3 -> Net-(C127-Pad1)
- R230 pad 2: +3V3 -> Net-(C127-Pad1)
- R231 pad 1: +3V3 -> Net-(C135-Pad1)
- R238 pad 2: +3V3 -> Net-(C135-Pad1)
- R239 pad 1: +3V3 -> Net-(C143-Pad1)
- R246 pad 2: +3V3 -> Net-(C143-Pad1)
- R247 pad 1: +3V3 -> Net-(C151-Pad1)
- R254 pad 2: +3V3 -> Net-(C151-Pad1)
- R255 pad 1: +3V3 -> Net-(C159-Pad1)
- R262 pad 2: +3V3 -> Net-(C159-Pad1)
- R263 pad 1: +3V3 -> Net-(C167-Pad1)
- R270 pad 2: +3V3 -> Net-(C167-Pad1)
- R30 pad 1: Net-(R30-Pad1) -> Net-(C36-Pad1)
- R30 pad 2: /PMIC/3.3V_STM_CORE -> /3.3V_EPS_STM
- R31 pad 2: Net-(R30-Pad1) -> Net-(C36-Pad1)
- R328 pad 2: Net-(J14-Pad1) -> Net-(D18-Pad1)
- R329 pad 2: /VEXT -> Net-(D18-Pad1)
- R47 pad 1: /PGOOD_SOLAR -> /PG_SOLAR
- R7 pad 1: Net-(R7-Pad1) -> Net-(C18-Pad1)
- U1 pad 1: Net-(R283-Pad1) -> /CURRENT_MONITORS/PWR1_11_ON
- U1 pad 10: Net-(R278-Pad1) -> /PMIC/INT_1
- U1 pad 11: Net-(R295-Pad1) -> /PMIC/INT_2
- U1 pad 114: /PGOOD_SOLAR -> /PG_SOLAR
- U1 pad 124: Net-(R291-Pad1) -> /PMIC/INT_9
- U1 pad 125: Net-(R275-Pad1) -> (no net)
- U1 pad 126: Net-(R292-Pad1) -> (no net)
- U1 pad 127: Net-(R276-Pad1) -> (no net)
- U1 pad 128: Net-(R293-Pad1) -> /~IDEAL_WARN1
- U1 pad 129: Net-(R277-Pad1) -> /~IDEAL_STATUS1
- U1 pad 132: Net-(R294-Pad1) -> /~IDEAL_STATUS2
- U1 pad 142: Net-(R299-Pad1) -> /CURRENT_MONITORS/PWR1_10_ON
- U1 pad 19: Net-(R279-Pad1) -> /PMIC/INT_3
- U1 pad 2: Net-(R300-Pad1) -> /CURRENT_MONITORS/PWR1_12_ON
- U1 pad 21: Net-(R296-Pad1) -> /PMIC/INT_4
- U1 pad 3: Net-(R284-Pad1) -> /CURRENT_MONITORS/PWR1_13_ON
- U1 pad 4: Net-(R301-Pad1) -> /PMIC/INT_8
- U1 pad 42: /PMIC/ADC1_IN11 -> (no net)
- U1 pad 49: Net-(R280-Pad1) -> /PMIC/INT_5
- U1 pad 5: Net-(R285-Pad1) -> /PMIC/INT_9
- U1 pad 50: Net-(R297-Pad1) -> /PMIC/INT_6
- U1 pad 53: Net-(R281-Pad1) -> /PMIC/INT_7
- U1 pad 54: Net-(R298-Pad1) -> /CURRENT_MONITORS/PWR1_8_ON
- U1 pad 55: Net-(R282-Pad1) -> /CURRENT_MONITORS/PWR1_9_ON
- U1 pad 56: Net-(R287-Pad1) -> /PMIC/INT_1
- U1 pad 58: Net-(R302-Pad1) -> /CURRENT_MONITORS/PWR1_16_ON
- U1 pad 59: Net-(R286-Pad1) -> /CURRENT_MONITORS/PWR2_1_ON
- U1 pad 60: Net-(R303-Pad1) -> /CURRENT_MONITORS/PWR2_2_ON
- U1 pad 87: Net-(R271-Pad1) -> /PMIC/INT_2
- U1 pad 88: Net-(R288-Pad1) -> /PMIC/INT_3
- U1 pad 89: Net-(R272-Pad1) -> /PMIC/INT_4
- U1 pad 90: Net-(R289-Pad1) -> /PMIC/INT_5
- U1 pad 91: Net-(R273-Pad1) -> /PMIC/INT_6
- U1 pad 92: Net-(R290-Pad1) -> /PMIC/INT_7
- U1 pad 93: Net-(R274-Pad1) -> /PMIC/INT_8
- U19 pad 3: +3V3 -> Net-(C47-Pad1)
- U2 pad 8: Net-(R7-Pad1) -> Net-(C18-Pad1)
- U20 pad 5: +3V3 -> Net-(C47-Pad1)
- U21 pad 6: +3V3 -> Net-(C47-Pad1)
- U23 pad 3: +3V3 -> Net-(C55-Pad1)
- U24 pad 5: +3V3 -> Net-(C55-Pad1)
- U25 pad 6: +3V3 -> Net-(C55-Pad1)
- U27 pad 3: +3V3 -> Net-(C63-Pad1)
- U28 pad 5: +3V3 -> Net-(C63-Pad1)
- U29 pad 6: +3V3 -> Net-(C63-Pad1)
- U31 pad 3: +3V3 -> Net-(C71-Pad1)
- U32 pad 5: +3V3 -> Net-(C71-Pad1)
- U33 pad 6: +3V3 -> Net-(C71-Pad1)
- U35 pad 3: +3V3 -> Net-(C79-Pad1)
- U36 pad 5: +3V3 -> Net-(C79-Pad1)
- U37 pad 6: +3V3 -> Net-(C79-Pad1)
- U39 pad 3: +3V3 -> Net-(C87-Pad1)
- U40 pad 5: +3V3 -> Net-(C87-Pad1)
- U41 pad 6: +3V3 -> Net-(C87-Pad1)
- U43 pad 3: +3V3 -> Net-(C95-Pad1)
- U44 pad 5: +3V3 -> Net-(C95-Pad1)
- U45 pad 6: +3V3 -> Net-(C95-Pad1)
- U47 pad 3: +3V3 -> Net-(C103-Pad1)
- U48 pad 5: +3V3 -> Net-(C103-Pad1)
- U49 pad 6: +3V3 -> Net-(C103-Pad1)
- U51 pad 3: +3V3 -> Net-(C111-Pad1)
- U52 pad 5: +3V3 -> Net-(C111-Pad1)
- U53 pad 6: +3V3 -> Net-(C111-Pad1)
- U55 pad 3: +3V3 -> Net-(C119-Pad1)
- U56 pad 5: +3V3 -> Net-(C119-Pad1)
- U57 pad 6: +3V3 -> Net-(C119-Pad1)
- U59 pad 3: +3V3 -> Net-(C127-Pad1)
- U60 pad 5: +3V3 -> Net-(C127-Pad1)
- U61 pad 6: +3V3 -> Net-(C127-Pad1)
- U63 pad 3: +3V3 -> Net-(C135-Pad1)
- U64 pad 5: +3V3 -> Net-(C135-Pad1)
- U65 pad 6: +3V3 -> Net-(C135-Pad1)
- U67 pad 3: +3V3 -> Net-(C143-Pad1)
- U68 pad 5: +3V3 -> Net-(C143-Pad1)
- U69 pad 6: +3V3 -> Net-(C143-Pad1)
- U71 pad 3: +3V3 -> Net-(C151-Pad1)
- U72 pad 5: +3V3 -> Net-(C151-Pad1)
- U73 pad 6: +3V3 -> Net-(C151-Pad1)
- U75 pad 3: +3V3 -> Net-(C159-Pad1)
- U76 pad 5: +3V3 -> Net-(C159-Pad1)
- U77 pad 6: +3V3 -> Net-(C159-Pad1)
- U79 pad 3: +3V3 -> Net-(C167-Pad1)
- U80 pad 5: +3V3 -> Net-(C167-Pad1)
- U81 pad 6: +3V3 -> Net-(C167-Pad1)
- U84 pad 5: (no net) -> GND
- X1 pad 2: Net-(R30-Pad1) -> Net-(C36-Pad1)
- X1 pad 3: Net-(R30-Pad1) -> Net-(C36-Pad1)
Routing:
- net GND: track 0.00 -> 716.6 mm, vias 0 -> 73
- net +3V3: track 0.00 -> 440.2 mm, vias 0 -> 6
- net /3.3V_EPS_STM: track 0.00 -> 206.4 mm, vias 0 -> 10
- net /VRAW_SOLAR: track 0.00 -> 94.5 mm, vias 0 -> 2
- net Net-(C10-Pad1): track 0.00 -> 91.2 mm, vias 0 -> 10
- net Net-(C15-Pad2): track 0.00 -> 89.5 mm, vias 0 -> 3
- net /3.3V_EPS_MRAM: track 0.00 -> 83.5 mm, vias 0 -> 1
- net /VOUT2: track 0.00 -> 80.8 mm, vias 0 -> 6
- net /SOLAR_5V: track 0.00 -> 80.3 mm, vias 0 -> 3
- net /BATTERY/NTC: track 0.00 -> 68.7 mm, vias 0 -> 1
- net /3.3V_EPS_CAN: track 0.00 -> 63.1 mm, vias 0 -> 2
- net /VOUT1: track 0.00 -> 59.6 mm, vias 0 -> 1
- net /sheet5F4CFCDE/NTC: track 0.00 -> 55.6 mm, vias 0 -> 1
- net Net-(C26-Pad1): track 0.00 -> 53.6 mm
- net /PMIC/QUADSPI_BK1_IO0: track 0.00 -> 52.9 mm
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- added copper zone on F.Cu, net +5V
- added copper zone on In1.Cu, net /BATTERY_CHARGER/BAT
- added copper zone on In1.Cu, net /SOLAR_5V
- added copper zone on B.Cu, net /SOLAR_MPPT_5V/VOUT
- added copper zone on In1.Cu, net /VOUT2
- added copper zone on B.Cu, net /VRAW_SOLAR
- added copper zone on In1.Cu, net /sheet5F4CFCDE/BAT
- added copper zone on F.Cu, net /sheet5FCD3934/VOUT
- added copper zone on B.Cu, net GND
- added copper zone on F.Cu, net GND
- added copper zone on In2.Cu, net GND
- added copper zone on F.Cu, net Net-(BT1-Pad1)
- added copper zone on F.Cu, net Net-(BT2-Pad1)
- added copper zone on In1.Cu, net Net-(C10-Pad1)
- added copper zone on F.Cu, net Net-(C177-Pad1)
- added copper zone on F.Cu, net Net-(C177-Pad2)
- added copper zone on F.Cu, net Net-(C178-Pad1)
- added copper zone on F.Cu, net Net-(C178-Pad2)
- added copper zone on B.Cu, net Net-(C35-Pad1)
- added copper zone on B.Cu, net Net-(C35-Pad2)
- added copper zone on B.Cu, net Net-(C37-Pad1)
- added copper zone on B.Cu, net Net-(C37-Pad2)
- added copper zone on F.Cu, net Net-(L3-Pad1)
- added copper zone on F.Cu, net VBUS
- added copper zone on In1.Cu, net VBUS
Other:
- board outline added: 85 x 85 mm
- copper layers 2 -> 4
- net class Power added: clearance 0.2, trace_width 0.4, via_dia 0.8, via_drill 0.4
- net class thin added: clearance 0.13, trace_width 0.2, via_dia 0.8, via_drill 0.4
- board text added: "1"

Commit message: EPS V1.0 Complete
Parts:
- removed TP38, TP40, TP41: TP_1.5x1.5, TestPoint:TestPoint_THTPad_1.5x1.5mm_Drill0.7mm
- added FID4: Fiducial, Calibration_Scale:Gauge_10mm_Type1_SilkScreenTop, F.Cu at (153.4, 84.9)
- added G***: LOGO, footprint_custom:qrr, B.Cu at (162.3, 88.8)
- C110, C111, C112, C113, C114, C115, C116, C117, C118, C119, C120, C121, C122, C123, C124, C125, C126, C127, C128, C129, C130, C131, C132, C133, C134, C135, C136, C137, C138, C139, C140, C141, C167, C168, C170, C171, C174, C19, C20, Q17, Q18, Q19, Q20, Q21, Q22, Q23, Q24, R119, R120, R121, R122, R123, R124, R125, R126, R127, R128, R129, R130, R207, R208, R209, R211, R212, R213, R214, R215, R216, R217, R219, R220, R221, R222, R223, R224, R225, R227, R228, R229, R230, R231, R232, R233, R235, R236, R237, R238, R267, R57, R58, U51, U52, U53, U54, U55, U56, U57, U58, U59, U6, U60, U61, U62, U63, U64, U65, U66, U7: moved to B.Cu
- J13: footprint Connector_PinHeader_2.54mm:PinHeader_1x04_P2.54mm_Horizontal -> Connector_PinHeader_2.54mm:PinHeader_1x04_P2.54mm_Vertical
- TP37, TP39: footprint TestPoint:TestPoint_THTPad_1.5x1.5mm_Drill0.7mm -> TestPoint:TestPoint_THTPad_1.0x1.0mm_Drill0.5mm
- U12, U9: footprint Package_DFN_QFN:QFN-24-1EP_4x4mm_P0.5mm_EP2.6x2.6mm_ThermalVias -> footprint_custom:QFN-24-1EP_4x4mm_P0.5mm_EP2.6x2.6mm_0.4mmThermalVias
- U15, U16, U83: footprint Package_SO:MSOP-16-1EP_3x4.039mm_P0.5mm_EP1.651x2.845mm_ThermalVias -> footprint_custom:MSOP-16-1EP_3x4.039mm_P0.5mm_EP1.651x2.845mm_0.3mmThermalVias
- moved Q17 105.2 mm to (101.0, 90.2), turned to 180 degrees
- moved R211 102.2 mm to (100.1, 83.0), turned to 90 degrees
- moved C115 101.1 mm to (104.7, 91.0), turned to 180 degrees
- moved Q18 99.8 mm to (101.0, 86.4), turned to 180 degrees
- moved R209 99.0 mm to (103.5, 88.3), turned to 90 degrees
- moved R124 96.4 mm to (105.2, 88.1), turned to 90 degrees
- moved C112 96.3 mm to (108.1, 91.0), turned to 0 degrees
- moved R214 93.6 mm to (103.7, 84.5), turned to 270 degrees
- moved U53 93.1 mm to (107.8, 88.4), turned to 0 degrees
- moved C117 91.5 mm to (105.1, 84.5), turned to 90 degrees
- moved C114 90.8 mm to (111.4, 90.4), turned to 0 degrees
- moved R123 88.6 mm to (111.4, 88.8), turned to 180 degrees
- moved U54 87.2 mm to (108.3, 84.7), turned to 180 degrees
- moved R208 86.5 mm to (111.4, 87.3), turned to 180 degrees
- moved C111 86.3 mm to (114.7, 90.5), turned to 0 degrees
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Connections:
- J6 pad 1: /3.3V_STM_CORE -> /3.3V_11
- J6 pad 10: /3.3V_9 -> GND
- J6 pad 11: GND -> /3.3V_MRAM
- J6 pad 12: /3.3V_10 -> /INTERBOARD_CONNECTOR/EPS_RESET
- J6 pad 13: /3.3V_ACS_LOGIC -> /UART_RXI
- J6 pad 14: GND -> /UART_TXO
- J6 pad 15: /3.3V_GYRO -> (no net)
- J6 pad 16: /3.3V_11 -> /INTERBOARD_CONNECTOR/AVI_RESET
- J6 pad 19: /5V0_1 -> (no net)
- J6 pad 2: GND -> /3.3V_ACS_LOGIC
- J6 pad 21: /5V0_2 -> (no net)
- J6 pad 22: /5V0_2 -> (no net)
- J6 pad 23: GND -> /3.3V_GYRO
- J6 pad 24: GND -> /3.3V_GPS
- J6 pad 25: (no net) -> /3.3V_CLK
- J6 pad 26: (no net) -> /3.3V_STM_CORE
- J6 pad 28: (no net) -> GND
- J6 pad 3: /3.3V_GPS -> GND
- J6 pad 30: (no net) -> /5V0_1
- J6 pad 31: (no net) -> GND
- J6 pad 32: (no net) -> GND
- J6 pad 33: /CANH -> /5V0_2
- J6 pad 34: (no net) -> /5V0_2
- J6 pad 35: /CANL -> GND
- J6 pad 37: /UART_RXI -> GND
- J6 pad 38: /INTERBOARD_CONNECTOR/EPS_RESET -> GND
- J6 pad 39: /UART_TXO -> /CANL
- J6 pad 4: /3.3V_MAG -> GND
- J6 pad 40: /INTERBOARD_CONNECTOR/AVI_RESET -> /CANH
- J6 pad 5: GND -> /3.3V_AVI_CAN
- J6 pad 6: /3.3V_CLK -> /3.3V_10
- J6 pad 7: /3.3V_MRAM -> (no net)
- J6 pad 8: GND -> /3.3V_MAG
- J6 pad 9: /3.3V_AVI_CAN -> /3.3V_9
Routing:
- net +3V3: track 440.2 -> 635.5 mm, vias 6 -> 29
- net GND: track 716.6 -> 883.8 mm, vias 73 -> 231
- net /BATTERY/VNTC: track 3.56 -> 147.3 mm, vias 1 -> 4
- net /BC_1_POL: track 11.0 -> 142.4 mm, vias 1 -> 4
- net /BC_2_SUSP: track 3.81 -> 127.0 mm, vias 0 -> 3
- net /BC_2_POL: track 13.9 -> 132.3 mm, vias 1 -> 5
- net /AVI_EXTRN_RST: track 0.00 -> 97.9 mm, vias 0 -> 12
- net /sheet5F4CFCDE/VNTC: track 5.14 -> 99.8 mm, vias 1 -> 2
- net /CURRENT_MONITORS/PWR1_11_ON: track 4.91 -> 97.7 mm, vias 0 -> 2
- net /IDEAL_EN1: track 8.67 -> 98.7 mm, vias 1 -> 3
- net /~IDEAL_EN2: track 11.2 -> 99.8 mm, vias 1 -> 3
- net /CANL: track 11.8 -> 98.3 mm
- net /CURRENT_MONITORS/PWR1_10_ON: track 4.82 -> 89.8 mm, vias 0 -> 4
- net /CANH: track 11.1 -> 95.7 mm
- net /PMIC/INT_5: track 25.8 -> 105.1 mm, vias 0 -> 7
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- added copper zone on B.Cu, net Net-(C39-Pad1)
- added copper zone on B.Cu, net VBUS
Other:
- rule pad_to_mask_clearance: 0.05 -> 0
- board text added: "$1K CubeSat"
- board text added: "10"
- board text added: "11"
- board text added: "12"
- board text added: "13"
- board text added: "14"
- board text added: "15"
- board text added: "16"
- board text added: "2"
- board text added: "3"
- board text added: "4"
- board text added: "5"
- board text added: "5V_1"
- board text added: "5V_2"
- board text added: "6"
- board text added: "7"
- board text added: "8"
- board text added: "9"
- board text added: "CAN"
- board text added: "EPS V1.0"
- board text added: "MRAM"
- board text removed: "90 cm"
