File: eps_board/IDEAL_DIODE.sch (KiCad schematic (older format))
At the start: 5 parts

Commit message: Progress on EPS
Parts:
- removed R?: 1K, Resistor_SMD:R_0603_1608Metric_Pad1.05x0.95mm_HandSolder, symbol Device:R
- removed R? (x2): 100K, Resistor_SMD:R_0603_1608Metric_Pad1.05x0.95mm_HandSolder, symbol Device:R
- added R?: 150, Resistor_SMD:R_0603_1608Metric_Pad1.05x0.95mm_HandSolder, symbol Device:R
- R?: value 1K -> 150
Connections:
- net GND: now also R?.2
- net at U?.5 (CLIM2): now also R?.1
Other:
- note added: "3.33A current limit per diode"
- note added: "Maximum 4A current limit for each diode"
- note added: "STAT\nOpen-drain output pulls down during forward diode conduction. \nThis pin can be left open or grounded when not used."
- note added: "WARN\nOpen-drain output pulls down when the diode current exceeds its\ncurrent limit or die temperature is close to thermal shutdown."
- note removed: "0.5A current limit is set"
Changed lines of the file:
@@
 EELAYER 30 0
 EELAYER END
-$Descr A4 11693 8268
+$Descr A 11000 8500
 encoding utf-8
-Sheet 4 14
-Title ""
-Date ""
+Sheet 7 39
+Title "LTC4415"
+Date "2020-09-06"
 Rev ""
 Comp ""
@@
 AR Path="/5F71F783/5F33369A" Ref="R?"  Part="1"
 F 0 "R?" V 4550 3350 50  0000 C CNN
-F 1 "1K" V 4550 3525 50  0000 C CNN
+F 1 "150" V 4550 3525 50  0000 C CNN
 F 2 "Resistor_SMD:R_0603_1608Metric_Pad1.05x0.95mm_HandSolder" V 4580 3450 50  0001 C CNN
 F 3 "~" H 4650 3450 50  0001 C CNN
@@
 Wire Wire Line
 	4800 3750 5100 3750
+Text HLabel 4125 3450 0    50   Input ~ 0
+GND
+Wire Wire Line
+	4125 3450 4300 3450
+Wire Wire Line
+	4300 3450 4300 3750
+Wire Wire Line
+	4300 3750 4500 3750
+Connection ~ 4300 3450
+Wire Wire Line
+	4300 3450 4500 3450
+Text Notes 3175 3675 0    50   ~ 0
+3.33A current limit per diode
+Text Notes 1025 5800 0    50   ~ 0
+Voltage Threasholds for the Enable pins:\nVenth = 0.8V with Venhyst = 0.055V
+Text Notes 2000 3225 0    50   ~ 0
+Weekly pullup EN1, so EN1 is always enabled\n
+Text Notes 1925 4025 0    50   ~ 0
+Weekly pulldown EN2, so EN2 is always enabled
+Text Notes 6125 2000 0    50   ~ 0
+STAT\nOpen-drain output pulls down during forward diode conduction. \nThis pin can be left open or grounded when not used.
+Text Notes 6125 2375 0    50   ~ 0
+WARN\nOpen-drain output pulls down when the diode current exceeds its\ncurrent limit or die temperature is close to thermal shutdown.
+Text Notes 4975 4950 0    50   ~ 0
+Maximum 4A current limit for each diode
 $Comp
 L Device:R R?
-U 1 1 5F334C9A
+U 1 1 5F7F3229
 P 4650 3750
-AR Path="/5F301BD2/5F334C9A" Ref="R?"  Part="1"
-AR Path="/5F33AC42/5F334C9A" Ref="R?"  Part="1"
-AR Path="/5F35742D/5F334C9A" Ref="R?"  Part="1"
-AR Path="/5F3589F2/5F334C9A" Ref="R?"  Part="1"
-AR Path="/5F3DE515/5F334C9A" Ref="R?"  Part="1"
-AR Path="/5F3E03A5/5F334C9A" Ref="R?"  Part="1"
-AR Path="/5F40A177/5F334C9A" Ref="R?"  Part="1"
-AR Path="/5F71F783/5F334C9A" Ref="R?"  Part="1"
+AR Path="/5F301BD2/5F7F3229" Ref="R?"  Part="1"
+AR Path="/5F33AC42/5F7F3229" Ref="R?"  Part="1"
+AR Path="/5F35742D/5F7F3229" Ref="R?"  Part="1"
+AR Path="/5F3589F2/5F7F3229" Ref="R?"  Part="1"
+AR Path="/5F3DE515/5F7F3229" Ref="R?"  Part="1"
+AR Path="/5F3E03A5/5F7F3229" Ref="R?"  Part="1"
+AR Path="/5F40A177/5F7F3229" Ref="R?"  Part="1"
+AR Path="/5F71F783/5F7F3229" Ref="R?"  Part="1"
 F 0 "R?" V 4550 3650 50  0000 C CNN
-F 1 "1K" V 4550 3825 50  0000 C CNN
+F 1 "150" V 4550 3825 50  0000 C CNN
 F 2 "Resistor_SMD:R_0603_1608Metric_Pad1.05x0.95mm_HandSolder" V 4580 3750 50  0001 C CNN
 F 3 "~" H 4650 3750 50  0001 C CNN
@@
 	0    1    1    0
 $EndComp
-Text HLabel 4125 3450 0    50   Input ~ 0
-GND
-Wire Wire Line
-	4125 3450 4300 3450
-Wire Wire Line
-	4300 3450 4300 3750
-Wire Wire Line
-	4300 3750 4500 3750
-Connection ~ 4300 3450
-Wire Wire Line
-	4300 3450 4500 3450
-Text Notes 3275 3650 0    50   ~ 0
-0.5A current limit is set
-Text Notes 1025 5800 0    50   ~ 0
-Voltage Threasholds for the Enable pins:\nVenth = 0.8V with Venhyst = 0.055V
-Text HLabel 2100 3575 0    50   Input ~ 0
-VIN1
-Text HLabel 2100 3875 0    50   Input ~ 0
-EN1
-$Comp
-L Device:R R?
-U 1 1 5F33798B
-P 2375 3725
-AR Path="/5F301BD2/5F33798B" Ref="R?"  Part="1"
-AR Path="/5F33AC42/5F33798B" Ref="R?"  Part="1"
-AR Path="/5F35742D/5F33798B" Ref="R?"  Part="1"
-AR Path="/5F3589F2/5F33798B" Ref="R?"  Part="1"
-AR Path="/5F3DE515/5F33798B" Ref="R?"  Part="1"
-AR Path="/5F3E03A5/5F33798B" Ref="R?"  Part="1"
-AR Path="/5F40A177/5F33798B" Ref="R?"  Part="1"
-AR Path="/5F71F783/5F33798B" Ref="R?"  Part="1"
-F 0 "R?" H 2250 3600 50  0000 C CNN
-F 1 "100K" H 2200 3850 50  0000 C CNN
-F 2 "Resistor_SMD:R_0603_1608Metric_Pad1.05x0.95mm_HandSolder" V 2305 3725 50  0001 C CNN
-F 3 "~" H 2375 3725 50  0001 C CNN
-	1    2375 3725
-	-1   0    0    1
-$EndComp
-Wire Wire Line
-	2100 3875 2375 3875
-Wire Wire Line
-	2100 3575 2375 3575
-Text Notes 1025 3450 0    50   ~ 0
-Weekly pullup EN1, so EN1 is always enabled\n
-Text HLabel 2100 4150 0    50   Input ~ 0
-~EN2
-$Comp
-L Device:R R?
-U 1 1 5F3398C4
-P 2375 4300
-AR Path="/5F301BD2/5F3398C4" Ref="R?"  Part="1"
-AR Path="/5F33AC42/5F3398C4" Ref="R?"  Part="1"
-AR Path="/5F35742D/5F3398C4" Ref="R?"  Part="1"
-AR Path="/5F3589F2/5F3398C4" Ref="R?"  Part="1"
-AR Path="/5F3DE515/5F3398C4" Ref="R?"  Part="1"
-AR Path="/5F3E03A5/5F3398C4" Ref="R?"  Part="1"
-AR Path="/5F40A177/5F3398C4" Ref="R?"  Part="1"
-AR Path="/5F71F783/5F3398C4" Ref="R?"  Part="1"
-F 0 "R?" H 2250 4175 50  0000 C CNN
-F 1 "100K" H 2200 4425 50  0000 C CNN
-F 2 "Resistor_SMD:R_0603_1608Metric_Pad1.05x0.95mm_HandSolder" V 2305 4300 50  0001 C CNN
-F 3 "~" H 2375 4300 50  0001 C CNN
-	1    2375 4300
-	-1   0    0    1
-$EndComp
-Wire Wire Line
-	2100 4150 2375 4150
-Text HLabel 2100 4450 0    50   Input ~ 0
-GND
-Wire Wire Line
-	2100 4450 2375 4450
-Text Notes 1000 4050 0    50   ~ 0
-Weekly pulldown EN2, so EN2 is always enabled
 $EndSCHEMATC

Commit message: Essentially done with EPS schematic
Parts:
- R85, R86: renamed from R?; Mfr. # (none) -> RMCF0603JT150R; Order (none) -> https://www.digikey.com/en/products/detail/stackpole-electr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
- gave numbers to parts that had none: 1
Changed lines of the file:
@@
 AR Path="/5F3E03A5/5F32EDA5" Ref="U?"  Part="1"
 AR Path="/5F40A177/5F32EDA5" Ref="U?"  Part="1"
-AR Path="/5F71F783/5F32EDA5" Ref="U?"  Part="1"
-F 0 "U?" H 5700 5025 50  0000 C CNN
+AR Path="/5F71F783/5F32EDA5" Ref="U15"  Part="1"
+F 0 "U15" H 5700 5025 50  0000 C CNN
 F 1 "LTC4415" H 5700 5150 50  0000 C CNN
 F 2 "Package_SO:MSOP-16-1EP_3x4.039mm_P0.5mm_EP1.651x2.845mm_ThermalVias" H 5700 2900 50  0001 C CNN
@@
 AR Path="/5F3E03A5/5F33369A" Ref="R?"  Part="1"
 AR Path="/5F40A177/5F33369A" Ref="R?"  Part="1"
-AR Path="/5F71F783/5F33369A" Ref="R?"  Part="1"
-F 0 "R?" V 4550 3350 50  0000 C CNN
+AR Path="/5F71F783/5F33369A" Ref="R85"  Part="1"
+F 0 "R85" V 4550 3350 50  0000 C CNN
 F 1 "150" V 4550 3525 50  0000 C CNN
 F 2 "Resistor_SMD:R_0603_1608Metric_Pad1.05x0.95mm_HandSolder" V 4580 3450 50  0001 C CNN
 F 3 "~" H 4650 3450 50  0001 C CNN
+F 4 "RMCF0603JT150R" H 4650 3450 50  0001 C CNN "Mfr. #"
+F 5 "https://www.digikey.com/en/products/detail/stackpole-electronics-inc/RMCF0603JT150R/1757965" H 4650 3450 50  0001 C CNN "Order"
 	1    4650 3450
 	0    1    1    0
@@
 Wire Wire Line
 	4300 3450 4500 3450
-Text Notes 3175 3675 0    50   ~ 0
+Text Notes 3150 3675 0    50   ~ 0
 3.33A current limit per diode
 Text Notes 1025 5800 0    50   ~ 0
@@
 AR Path="/5F3E03A5/5F7F3229" Ref="R?"  Part="1"
 AR Path="/5F40A177/5F7F3229" Ref="R?"  Part="1"
-AR Path="/5F71F783/5F7F3229" Ref="R?"  Part="1"
-F 0 "R?" V 4550 3650 50  0000 C CNN
+AR Path="/5F71F783/5F7F3229" Ref="R86"  Part="1"
+F 0 "R86" V 4550 3650 50  0000 C CNN
 F 1 "150" V 4550 3825 50  0000 C CNN
 F 2 "Resistor_SMD:R_0603_1608Metric_Pad1.05x0.95mm_HandSolder" V 4580 3750 50  0001 C CNN
 F 3 "~" H 4650 3750 50  0001 C CNN
+F 4 "RMCF0603JT150R" H 4650 3750 50  0001 C CNN "Mfr. #"
+F 5 "https://www.digikey.com/en/products/detail/stackpole-electronics-inc/RMCF0603JT150R/1757965" H 4650 3750 50  0001 C CNN "Order"
 	1    4650 3750
 	0    1    1    0

Commit message: EPS V1.0 Complete
Parts:
- U15: footprint Package_SO:MSOP-16-1EP_3x4.039mm_P0.5mm_EP1.651x2.845mm_ThermalVias -> footprint_custom:MSOP-16-1EP_3x4.039mm_P0.5mm_EP1.651x2.845mm_0.3mmThermalVias
Changed lines of the file:
@@
 F 0 "U15" H 5700 5025 50  0000 C CNN
 F 1 "LTC4415" H 5700 5150 50  0000 C CNN
-F 2 "Package_SO:MSOP-16-1EP_3x4.039mm_P0.5mm_EP1.651x2.845mm_ThermalVias" H 5700 2900 50  0001 C CNN
+F 2 "footprint_custom:MSOP-16-1EP_3x4.039mm_P0.5mm_EP1.651x2.845mm_0.3mmThermalVias" H 5700 2900 50  0001 C CNN
 F 3 "https://www.analog.com/media/en/technical-documentation/data-sheets/4415fa.pdf" H 5700 3850 50  0001 C CNN
 F 4 "LTC4415EMSE#PBF" H 5700 2600 50  0001 C CNN "Mfr. #"
