File: eps_board/LTC3130.sch (KiCad schematic (older format))
At the start: 15 parts, among them U83 LTC3130-1

Commit message: EPS V1.0 Complete
Parts:
- U83: footprint Package_SO:MSOP-16-1EP_3x4.039mm_P0.5mm_EP1.651x2.845mm_ThermalVias -> footprint_custom:MSOP-16-1EP_3x4.039mm_P0.5mm_EP1.651x2.845mm_0.3mmThermalVias
Changed lines of the file:
@@
 $Descr A 11000 8500
 encoding utf-8
-Sheet 8 39
+Sheet 39 39
 Title "LTC3130"
 Date "2020-08-09"
@@
 AR Path="/5F62C305/5F325818" Ref="C?"  Part="1"
 AR Path="/5FCD393E/5F325818" Ref="C175"  Part="1"
-F 0 "C33" H 2375 3625 50  0000 L CNN
+F 0 "C175" H 2375 3625 50  0000 L CNN
 F 1 "4.7uF" H 2375 3550 50  0000 L CNN
 F 2 "Capacitor_SMD:C_0603_1608Metric_Pad1.05x0.95mm_HandSolder" H 2313 3425 50  0001 C CNN
@@
 AR Path="/5F62C305/5F316C45" Ref="R?"  Part="1"
 AR Path="/5FCD393E/5F316C45" Ref="R318"  Part="1"
-F 0 "R89" V 3725 3975 50  0000 C CNN
+F 0 "R318" V 3725 3975 50  0000 C CNN
 F 1 "0" V 3725 4100 50  0000 C CNN
 F 2 "Resistor_SMD:R_0603_1608Metric_Pad1.05x0.95mm_HandSolder" V 3755 4025 50  0001 C CNN
@@
 AR Path="/5F62C305/5F3159CA" Ref="R?"  Part="1"
 AR Path="/5FCD393E/5F3159CA" Ref="R319"  Part="1"
-F 0 "R90" V 6350 3575 50  0000 C CNN
+F 0 "R319" V 6350 3575 50  0000 C CNN
 F 1 "0" V 6350 3700 50  0000 C CNN
 F 2 "Resistor_SMD:R_0603_1608Metric_Pad1.05x0.95mm_HandSolder" V 6380 3625 50  0001 C CNN
@@
 AR Path="/5F62C305/5F30F8B8" Ref="C?"  Part="1"
 AR Path="/5FCD393E/5F30F8B8" Ref="C180"  Part="1"
-F 0 "C41" H 6900 3550 50  0000 L CNN
+F 0 "C180" H 6900 3550 50  0000 L CNN
 F 1 "47uF" H 6900 3475 50  0000 L CNN
 F 2 "Capacitor_SMD:C_1210_3225Metric_Pad1.42x2.65mm_HandSolder" H 6838 3325 50  0001 C CNN
@@
 AR Path="/5F62C305/5F30E2F4" Ref="C?"  Part="1"
 AR Path="/5FCD393E/5F30E2F4" Ref="C177"  Part="1"
-F 0 "C35" V 4521 2500 50  0000 C CNN
+F 0 "C177" V 4521 2500 50  0000 C CNN
 F 1 "22nF" V 4612 2500 50  0000 C CNN
 F 2 "Capacitor_SMD:C_0603_1608Metric_Pad1.05x0.95mm_HandSolder" H 4750 2500 50  0001 C CNN
@@
 AR Path="/5F62C305/5F30C7DB" Ref="L?"  Part="1"
 AR Path="/5FCD393E/5F30C7DB" Ref="L2"  Part="1"
-F 0 "L1" V 5400 2500 50  0000 C CNN
+F 0 "L2" V 5400 2500 50  0000 C CNN
 F 1 "4.7uH" V 5325 2500 50  0000 C CNN
 F 2 "Inductor_SMD:L_Coilcraft_LPS4018" H 5250 2500 50  0001 C CNN
@@
 AR Path="/5F62C305/5F30A62E" Ref="C?"  Part="1"
 AR Path="/5FCD393E/5F30A62E" Ref="C179"  Part="1"
-F 0 "C40" H 6525 4550 50  0000 L CNN
+F 0 "C179" H 6525 4550 50  0000 L CNN
 F 1 "4.7uF" H 6525 4475 50  0000 L CNN
 F 2 "Capacitor_SMD:C_0603_1608Metric_Pad1.05x0.95mm_HandSolder" H 6463 4350 50  0001 C CNN
@@
 AR Path="/5F62C305/5F5775AC" Ref="R?"  Part="1"
 AR Path="/5FCD393E/5F5775AC" Ref="R317"  Part="1"
-F 0 "R88" V 3725 4375 50  0000 C CNN
+F 0 "R317" V 3725 4375 50  0000 C CNN
 F 1 "0" V 3725 4500 50  0000 C CNN
 F 2 "Resistor_SMD:R_0603_1608Metric_Pad1.05x0.95mm_HandSolder" V 3755 4425 50  0001 C CNN
@@
 AR Path="/5F62C305/5F5775B2" Ref="R?"  Part="1"
 AR Path="/5FCD393E/5F5775B2" Ref="R316"  Part="1"
-F 0 "R87" V 3725 4175 50  0000 C CNN
+F 0 "R316" V 3725 4175 50  0000 C CNN
 F 1 "0" V 3725 4300 50  0000 C CNN
 F 2 "Resistor_SMD:R_0603_1608Metric_Pad1.05x0.95mm_HandSolder" V 3755 4225 50  0001 C CNN
@@
 AR Path="/5F62C305/5F915D60" Ref="C?"  Part="1"
 AR Path="/5FCD393E/5F915D60" Ref="C178"  Part="1"
-F 0 "C37" V 5525 2500 50  0000 C CNN
+F 0 "C178" V 5525 2500 50  0000 C CNN
 F 1 "22nF" V 5600 2500 50  0000 C CNN
 F 2 "Capacitor_SMD:C_0603_1608Metric_Pad1.05x0.95mm_HandSolder" H 5750 2500 50  0001 C CNN
@@
 AR Path="/5F62C305/5F918110" Ref="C?"  Part="1"
 AR Path="/5FCD393E/5F918110" Ref="C181"  Part="1"
-F 0 "C42" H 7365 3521 50  0000 L CNN
+F 0 "C181" H 7365 3521 50  0000 L CNN
 F 1 "DNP" H 7365 3430 50  0000 L CNN
 F 2 "Capacitor_SMD:C_1210_3225Metric_Pad1.42x2.65mm_HandSolder" H 7288 3325 50  0001 C CNN
@@
 AR Path="/5F62C305/5F91837D" Ref="C?"  Part="1"
 AR Path="/5FCD393E/5F91837D" Ref="C182"  Part="1"
-F 0 "C43" H 7815 3521 50  0000 L CNN
+F 0 "C182" H 7815 3521 50  0000 L CNN
 F 1 "DNP" H 7815 3430 50  0000 L CNN
 F 2 "Capacitor_SMD:C_0603_1608Metric_Pad1.05x0.95mm_HandSolder" H 7738 3325 50  0001 C CNN
@@
 AR Path="/5F62C305/5F91FDED" Ref="C?"  Part="1"
 AR Path="/5FCD393E/5F91FDED" Ref="C176"  Part="1"
-F 0 "C34" H 2825 3625 50  0000 L CNN
+F 0 "C176" H 2825 3625 50  0000 L CNN
 F 1 "1uF" H 2825 3550 50  0000 L CNN
 F 2 "Capacitor_SMD:C_0603_1608Metric_Pad1.05x0.95mm_HandSolder" H 2763 3425 50  0001 C CNN
@@
 AR Path="/5F62C305/5F92B281" Ref="C?"  Part="1"
 AR Path="/5FCD393E/5F92B281" Ref="C174"  Part="1"
-F 0 "C32" H 1925 3625 50  0000 L CNN
+F 0 "C174" H 1925 3625 50  0000 L CNN
 F 1 "47uF" H 1925 3550 50  0000 L CNN
 F 2 "Capacitor_SMD:C_1210_3225Metric_Pad1.42x2.65mm_HandSolder" H 1863 3425 50  0001 C CNN
@@
 AR Path="/5F301AC2/638BE07D" Ref="U16"  Part="1"
 AR Path="/638BE07D" Ref="U83"  Part="1"
-F 0 "U16" H 5275 3825 50  0000 C CNN
+F 0 "U83" H 5275 3825 50  0000 C CNN
 F 1 "LTC3130-1" H 5250 3425 50  0000 C CNN
-F 2 "Package_SO:MSOP-16-1EP_3x4.039mm_P0.5mm_EP1.651x2.845mm_ThermalVias" H 5300 2575 50  0001 C CNN
+F 2 "footprint_custom:MSOP-16-1EP_3x4.039mm_P0.5mm_EP1.651x2.845mm_0.3mmThermalVias" H 5300 2575 50  0001 C CNN
 F 3 "https://www.analog.com/media/en/technical-documentation/data-sheets/3130f.pdf" H 5250 3825 50  0001 C CNN
 F 4 "LTC3130EMSE-1#PBF" H 5250 3975 50  0001 C CNN "Mfr. #"
