File: eps_board/INTERBOARD_CONNECTOR.sch (KiCad schematic (older format))
At the start: 1 part, among them J8 Conn_02x20_Odd_Even

Commit message: Progress on EPS
Parts:
- removed J8: Conn_02x20_Odd_Even, Connector_PinHeader_2.54mm:PinHeader_2x20_P2.54mm_Vertical, symbol Connector_Generic:Conn_02x20_Odd_Even
- added J?: Conn_02x20_Odd_Even, Connector_PinHeader_2.54mm:PinHeader_2x20_P2.54mm_Vertical, symbol Connector_Generic:Conn_02x20_Odd_Even
Connections:
- net CANH: now also J?.33 (Pin_33)
- net CANL: now also J?.35 (Pin_35)
- net EPS_RESET: now also J?.31 (Pin_31)
- net GND: now also J?.10 (Pin_10), J?.12 (Pin_12), J?.14 (Pin_14), J?.16 (Pin_16), J?.18 (Pin_18), J?.2 (Pin_2), J?.20 (Pin_20), J?.22 (Pin_22), J?.24 (Pin_24), J?.26 (Pin_26), J?.28 (Pin_28), J?.4 (Pin_4), J?.6 (Pin_6), J?.8 (Pin_8)
- net SPARE_1: now also J?.30 (Pin_30)
- net SPARE_2: now also J?.32 (Pin_32)
- net SPARE_3: now also J?.34 (Pin_34)
- net SPARE_4: now also J?.36 (Pin_36)
- new net 3V3_1: J?.1 (Pin_1)
- new net 3V3_10: J?.19 (Pin_19)
- new net 3V3_11: J?.21 (Pin_21)
- new net 3V3_12: J?.23 (Pin_23)
- new net 3V3_2: J?.3 (Pin_3)
- new net 3V3_3: J?.5 (Pin_5)
- new net 3V3_4: J?.7 (Pin_7)
- new net 3V3_5: J?.9 (Pin_9)
- new net 3V3_6: J?.11 (Pin_11)
- new net 3V3_7: J?.13 (Pin_13)
- new net 3V3_8: J?.15 (Pin_15)
- new net 3V3_9: J?.17 (Pin_17)
- new net 5V0_1: J?.25 (Pin_25)
- new net 5V0_2: J?.27 (Pin_27)
- new net AVI_RESET: J?.29 (Pin_29)
- new net UART_A_RXI: J?.39 (Pin_39)
- new net UART_A_TXO: J?.37 (Pin_37)
- new net UART_B_RXI: J?.40 (Pin_40)
- new net UART_B_TXO: J?.38 (Pin_38)
Changed lines of the file:
@@
 $Descr A 11000 8500
 encoding utf-8
-Sheet 23 24
-Title "Interboard Connector"
+Sheet 26 39
+Title "Current Monitor"
 Date "2020-05-25"
 Rev ""
@@
 $EndDescr
 $Comp
-L Connector_Generic:Conn_02x20_Odd_Even J8
-U 1 1 61C172A8
+L Connector_Generic:Conn_02x20_Odd_Even J?
+U 1 1 6310C580
 P 5775 3775
-F 0 "J8" H 5825 4892 50  0000 C CNN
+AR Path="/5EA31C93/6310AFB3/5FD3BACF/6310C580" Ref="J?"  Part="1"
+AR Path="/5EA31C93/631545C7/6310C580" Ref="J?"  Part="1"
+AR Path="/5FD3BACF/6310C580" Ref="J?"  Part="1"
+F 0 "J?" H 5825 4892 50  0000 C CNN
 F 1 "Conn_02x20_Odd_Even" H 5825 4801 50  0000 C CNN
 F 2 "Connector_PinHeader_2.54mm:PinHeader_2x20_P2.54mm_Vertical" H 5775 3775 50  0001 C CNN
@@
 $EndComp
 Text HLabel 5100 2875 0    50   Output ~ 0
-PWR_STM_CORE
-Text HLabel 5100 3775 0    50   Output ~ 0
-AVO_RESET
-Text HLabel 5100 2975 0    50   Output ~ 0
-PWR_GPS
-Text HLabel 5100 3075 0    50   Output ~ 0
-PWR_IRIDIUM
-Text HLabel 5100 3175 0    50   Output ~ 0
-PWR_ACS_COIL
-Text HLabel 5100 3275 0    50   Output ~ 0
-PWR_ACS_LOGIC
-Text HLabel 5100 3375 0    50   Output ~ 0
-PWR_GYRO
-Text HLabel 5100 3475 0    50   Output ~ 0
-PWR_MAG
-Text HLabel 5100 3575 0    50   Output ~ 0
-PWR_TEMPERATURE
-Text HLabel 5100 4475 0    50   Output ~ 0
+3V3_1
+Text HLabel 5100 4275 0    50   Output ~ 0
+AVI_RESET
+Text HLabel 5100 4475 0    50   BiDi ~ 0
 CANH
-Text HLabel 5100 4575 0    50   Output ~ 0
+Text HLabel 5100 4575 0    50   BiDi ~ 0
 CANL
 Text HLabel 5100 4675 0    50   Output ~ 0
-UART_TXO
-Text HLabel 5100 4775 0    50   Output ~ 0
-UART_RXI
+UART_A_TXO
+Text HLabel 5100 4775 0    50   Input ~ 0
+UART_A_RXI
 Text HLabel 6550 2875 2    50   Output ~ 0
 GND
@@
 Wire Wire Line
 	6075 3675 6550 3675
-Text HLabel 6550 4775 2    50   Output ~ 0
-GND
 Wire Wire Line
 	6075 4775 6550 4775
-Text HLabel 6550 4675 2    50   Output ~ 0
-GND
 Wire Wire Line
 	6075 4675 6550 4675
-Text HLabel 6550 4575 2    50   Output ~ 0
-GND
 Wire Wire Line
 	6075 4575 6550 4575
-Text HLabel 6550 4475 2    50   Output ~ 0
+Text HLabel 6550 4175 2    50   Output ~ 0
 GND
 Wire Wire Line
@@
 Wire Wire Line
 	5100 4775 5575 4775
-Text HLabel 5100 4275 0    50   Output ~ 0
-SPARE_8
-Text HLabel 5100 4175 0    50   Output ~ 0
-SPARE_6
-Text HLabel 5100 4075 0    50   Output ~ 0
-SPARE_4
-Text HLabel 5100 3975 0    50   Output ~ 0
+Text HLabel 6550 4375 2    50   Output ~ 0
 SPARE_2
 Wire Wire Line
@@
 Wire Wire Line
 	6075 4275 6550 4275
-Text HLabel 6550 4175 2    50   Output ~ 0
-SPARE_7
+Text HLabel 6550 4475 2    50   Output ~ 0
+SPARE_3
 Text HLabel 6550 4275 2    50   Output ~ 0
-SPARE_9
-Text HLabel 6550 4075 2    50   Output ~ 0
-SPARE_5
-Text HLabel 6550 3975 2    50   Output ~ 0
-SPARE_3
-Text HLabel 6550 3875 2    50   Output ~ 0
 SPARE_1
 Wire Wire Line
@@
 Wire Wire Line
 	6075 3975 6550 3975
-Text HLabel 5100 3675 0    50   Output ~ 0
-PWR_MRAM
 Text HLabel 6550 3775 2    50   Output ~ 0
 GND
@@
 Wire Wire Line
 	5100 3775 5575 3775
-Text HLabel 5100 4375 0    50   Output ~ 0
-PWR_CAN
 Wire Wire Line
 	5100 4375 5575 4375
-Text HLabel 6550 4375 2    50   Output ~ 0
+Text HLabel 6550 4075 2    50   Output ~ 0
 GND
 Wire Wire Line
 	6075 4375 6550 4375
+Text HLabel 5100 4375 0    50   Output ~ 0
+EPS_RESET
+Text HLabel 5100 2975 0    50   Output ~ 0
+3V3_2
+Text HLabel 5100 3075 0    50   Output ~ 0
+3V3_3
+Text HLabel 5100 3175 0    50   Output ~ 0
+3V3_4
+Text HLabel 5100 3275 0    50   Output ~ 0
+3V3_5
+Text HLabel 5100 3375 0    50   Output ~ 0
+3V3_6
+Text HLabel 5100 3475 0    50   Output ~ 0
+3V3_7
+Text HLabel 5100 3575 0    50   Output ~ 0
+3V3_8
+Text HLabel 5100 3675 0    50   Output ~ 0
+3V3_9
+Text HLabel 5100 3775 0    50   Output ~ 0
+3V3_10
 Text HLabel 5100 3875 0    50   Output ~ 0
-EPS_RESET
+3V3_11
+Text HLabel 5100 3975 0    50   Output ~ 0
+3V3_12
+Text HLabel 5100 4075 0    50   Output ~ 0
+5V0_1
+Text HLabel 5100 4175 0    50   Output ~ 0
+5V0_2
+Text HLabel 6550 3875 2    50   Output ~ 0
+GND
+Text HLabel 6550 3975 2    50   Output ~ 0
+GND
+Text HLabel 6550 4575 2    50   Output ~ 0
+SPARE_4
+Text HLabel 6550 4675 2    50   Output ~ 0
+UART_B_TXO
+Text HLabel 6550 4775 2    50   Input ~ 0
+UART_B_RXI
 $EndSCHEMATC

Commit message: Essentially done with EPS schematic
Parts:
- gave numbers to parts that had none: 1
Connections:
- net 3V3_10: now also J1.12 (Pin_12); no longer J1.19 (Pin_19)
- net 3V3_11: now also J1.16 (Pin_16); no longer J1.21 (Pin_21)
- net 3V3_12: now also J1.18 (Pin_18); no longer J1.23 (Pin_23)
- net 3V3_3: now also J1.7 (Pin_7); no longer J1.5 (Pin_5)
- net 3V3_4: now also J1.9 (Pin_9); no longer J1.7 (Pin_7)
- net 3V3_5: now also J1.13 (Pin_13); no longer J1.9 (Pin_9)
- net 3V3_6: now also J1.15 (Pin_15); no longer J1.11 (Pin_11)
- net 3V3_7: now also J1.4 (Pin_4); no longer J1.13 (Pin_13)
- net 3V3_8: now also J1.6 (Pin_6); no longer J1.15 (Pin_15)
- net 3V3_9: now also J1.10 (Pin_10); no longer J1.17 (Pin_17)
- net 5V0_1: now also J1.19 (Pin_19); no longer J1.25 (Pin_25)
- net 5V0_2: now also J1.21 (Pin_21), J1.22 (Pin_22); no longer J1.27 (Pin_27)
- net AVI_RESET: now also J1.40 (Pin_40); no longer J1.29 (Pin_29)
- net EPS_RESET: now also J1.38 (Pin_38); no longer J1.31 (Pin_31)
- net GND: now also J1.11 (Pin_11), J1.17 (Pin_17), J1.23 (Pin_23), J1.5 (Pin_5); no longer J1.10 (Pin_10), J1.12 (Pin_12), J1.16 (Pin_16), J1.18 (Pin_18), J1.22 (Pin_22), J1.26 (Pin_26), J1.28 (Pin_28), J1.4 (Pin_4), J1.6 (Pin_6)
- net SPARE_1: now also J1.25 (Pin_25); no longer J1.30 (Pin_30)
- net SPARE_2: now also J1.27 (Pin_27); no longer J1.32 (Pin_32)
- net SPARE_3: now also J1.29 (Pin_29); no longer J1.34 (Pin_34)
- net SPARE_4: now also J1.31 (Pin_31); no longer J1.36 (Pin_36)
- net UART_B_RXI: now also J1.32 (Pin_32); no longer J1.40 (Pin_40)
- net UART_B_TXO: now also J1.30 (Pin_30); no longer J1.38 (Pin_38)
- new net SPARE_5: J1.26 (Pin_26)
- new net SPARE_6: J1.28 (Pin_28)
- new net UART_B_CTS: J1.34 (Pin_34)
- new net UART_B_RTS: J1.36 (Pin_36)
Other:
- note added: "There are a lot of options that could work:\nhttps://www.digikey.com/short/znc31r"
Changed lines of the file:
@@
 $Descr A 11000 8500
 encoding utf-8
-Sheet 26 39
+Sheet 9 39
 Title "Current Monitor"
 Date "2020-05-25"
@@
 P 5775 3775
 AR Path="/5EA31C93/6310AFB3/5FD3BACF/6310C580" Ref="J?"  Part="1"
-AR Path="/5EA31C93/631545C7/6310C580" Ref="J?"  Part="1"
-AR Path="/5FD3BACF/6310C580" Ref="J?"  Part="1"
-F 0 "J?" H 5825 4892 50  0000 C CNN
+AR Path="/5EA31C93/631545C7/6310C580" Ref="J1"  Part="1"
+AR Path="/5FD3BACF/6310C580" Ref="J6"  Part="1"
+AR Path="/5EA31C93/639EBCB0/6310C580" Ref="J?"  Part="1"
+F 0 "J6" H 5825 4892 50  0000 C CNN
 F 1 "Conn_02x20_Odd_Even" H 5825 4801 50  0000 C CNN
 F 2 "Connector_PinHeader_2.54mm:PinHeader_2x20_P2.54mm_Vertical" H 5775 3775 50  0001 C CNN
@@
 Text HLabel 5100 2875 0    50   Output ~ 0
 3V3_1
-Text HLabel 5100 4275 0    50   Output ~ 0
+Text HLabel 6550 4775 2    50   Output ~ 0
 AVI_RESET
 Text HLabel 5100 4475 0    50   BiDi ~ 0
@@
 Text HLabel 5100 4775 0    50   Input ~ 0
 UART_A_RXI
-Text HLabel 6550 2875 2    50   Output ~ 0
-GND
 Wire Wire Line
 	5100 2875 5575 2875
 Wire Wire Line
 	6075 2875 6550 2875
-Text HLabel 6550 2975 2    50   Output ~ 0
-GND
 Wire Wire Line
 	6075 2975 6550 2975
-Text HLabel 6550 3075 2    50   Output ~ 0
-GND
 Wire Wire Line
 	6075 3075 6550 3075
-Text HLabel 6550 3175 2    50   Output ~ 0
-GND
 Wire Wire Line
 	6075 3175 6550 3175
-Text HLabel 6550 3275 2    50   Output ~ 0
-GND
 Wire Wire Line
 	6075 3275 6550 3275
-Text HLabel 6550 3375 2    50   Output ~ 0
-GND
 Wire Wire Line
 	6075 3375 6550 3375
-Text HLabel 6550 3475 2    50   Output ~ 0
+Text HLabel 5100 3075 0    50   Output ~ 0
 GND
 Wire Wire Line
 	6075 3475 6550 3475
-Text HLabel 6550 3575 2    50   Output ~ 0
+Text HLabel 5100 3375 0    50   Output ~ 0
 GND
 Wire Wire Line
 	6075 3575 6550 3575
-Text HLabel 6550 3675 2    50   Output ~ 0
+Text HLabel 6550 2875 2    50   Output ~ 0
 GND
 Wire Wire Line
@@
 Wire Wire Line
 	6075 4575 6550 4575
-Text HLabel 6550 4175 2    50   Output ~ 0
-GND
 Wire Wire Line
 	6075 4475 6550 4475
@@
 Wire Wire Line
 	5100 4775 5575 4775
-Text HLabel 6550 4375 2    50   Output ~ 0
+Text HLabel 5100 4175 0    50   Output ~ 0
 SPARE_2
 Wire Wire Line
@@
 Wire Wire Line
 	6075 4275 6550 4275
-Text HLabel 6550 4475 2    50   Output ~ 0
+Text HLabel 5100 4275 0    50   Output ~ 0
 SPARE_3
-Text HLabel 6550 4275 2    50   Output ~ 0
+Text HLabel 5100 4075 0    50   Output ~ 0
 SPARE_1
 Wire Wire Line
@@
 Wire Wire Line
 	6075 3975 6550 3975
-Text HLabel 6550 3775 2    50   Output ~ 0
+Text HLabel 6550 3175 2    50   Output ~ 0
 GND
 Wire Wire Line
@@
 Wire Wire Line
 	5100 4375 5575 4375
-Text HLabel 6550 4075 2    50   Output ~ 0
+Text HLabel 5100 3675 0    50   Output ~ 0
 GND
 Wire Wire Line
 	6075 4375 6550 4375
-Text HLabel 5100 4375 0    50   Output ~ 0
+Text HLabel 6550 4675 2    50   Output ~ 0
 EPS_RESET
 Text HLabel 5100 2975 0    50   Output ~ 0
 3V3_2
-Text HLabel 5100 3075 0    50   Output ~ 0
+Text HLabel 5100 3175 0    50   Output ~ 0
 3V3_3
-Text HLabel 5100 3175 0    50   Output ~ 0
+Text HLabel 5100 3275 0    50   Output ~ 0
 3V3_4
-Text HLabel 5100 3275 0    50   Output ~ 0
+Text HLabel 5100 3475 0    50   Output ~ 0
 3V3_5
-Text HLabel 5100 3375 0    50   Output ~ 0
+Text HLabel 5100 3575 0    50   Output ~ 0
 3V3_6
-Text HLabel 5100 3475 0    50   Output ~ 0
+Text HLabel 6550 2975 2    50   Output ~ 0
 3V3_7
-Text HLabel 5100 3575 0    50   Output ~ 0
+Text HLabel 6550 3075 2    50   Output ~ 0
 3V3_8
-Text HLabel 5100 3675 0    50   Output ~ 0
+Text HLabel 6550 3275 2    50   Output ~ 0
 3V3_9
+Text HLabel 6550 3375 2    50   Output ~ 0
+3V3_10
+Text HLabel 6550 3575 2    50   Output ~ 0
+3V3_11
+Text HLabel 6550 3675 2    50   Output ~ 0
+3V3_12
 Text HLabel 5100 3775 0    50   Output ~ 0
-3V3_10
+5V0_1
 Text HLabel 5100 3875 0    50   Output ~ 0
-3V3_11
+5V0_2
+Text HLabel 6550 3475 2    50   Output ~ 0
+GND
+Text HLabel 6550 3775 2    50   Output ~ 0
+GND
+Text HLabel 5100 4375 0    50   Output ~ 0
+SPARE_4
+Text HLabel 6550 4275 2    50   Output ~ 0
+UART_B_TXO
+Text HLabel 6550 4375 2    50   Input ~ 0
+UART_B_RXI
+Text HLabel 6550 3875 2    50   Output ~ 0
+5V0_2
+Text HLabel 6550 4475 2    50   Input ~ 0
+UART_B_CTS
+Text HLabel 6550 4575 2    50   Output ~ 0
+UART_B_RTS
 Text HLabel 5100 3975 0    50   Output ~ 0
-3V3_12
-Text HLabel 5100 4075 0    50   Output ~ 0
-5V0_1
-Text HLabel 5100 4175 0    50   Output ~ 0
-5V0_2
-Text HLabel 6550 3875 2    50   Output ~ 0
 GND
 Text HLabel 6550 3975 2    50   Output ~ 0
 GND
-Text HLabel 6550 4575 2    50   Output ~ 0
-SPARE_4
-Text HLabel 6550 4675 2    50   Output ~ 0
-UART_B_TXO
-Text HLabel 6550 4775 2    50   Input ~ 0
-UART_B_RXI
+Text HLabel 6550 4075 2    50   Output ~ 0
+SPARE_5
+Text HLabel 6550 4175 2    50   Output ~ 0
+SPARE_6
+Text Notes 4950 5225 0    50   ~ 0
+There are a lot of options that could work:\nhttps://www.digikey.com/short/znc31r
 $EndSCHEMATC

Commit message: EPS V1.0 Complete
Connections:
- net SPARE_5 is gone; now on net 3V3_1: J1.26 (Pin_26)
- net SPARE_6 is gone; now on net GND: J1.28 (Pin_28)
- net 3V3_1: no longer J1.1 (Pin_1)
- net 3V3_10: now also J1.6 (Pin_6); no longer J1.12 (Pin_12)
- net 3V3_11: now also J1.1 (Pin_1); no longer J1.16 (Pin_16)
- net 3V3_2: now also J1.24 (Pin_24); no longer J1.3 (Pin_3)
- net 3V3_3: now also J1.11 (Pin_11); no longer J1.7 (Pin_7)
- net 3V3_4: now also J1.5 (Pin_5); no longer J1.9 (Pin_9)
- net 3V3_5: now also J1.2 (Pin_2); no longer J1.13 (Pin_13)
- net 3V3_6: now also J1.23 (Pin_23); no longer J1.15 (Pin_15)
- net 3V3_7: now also J1.8 (Pin_8); no longer J1.4 (Pin_4)
- net 3V3_8: now also J1.25 (Pin_25); no longer J1.6 (Pin_6)
- net 3V3_9: now also J1.9 (Pin_9); no longer J1.10 (Pin_10)
- net 5V0_1: now also J1.30 (Pin_30); no longer J1.19 (Pin_19)
- net 5V0_2: now also J1.33 (Pin_33), J1.34 (Pin_34); no longer J1.21 (Pin_21), J1.22 (Pin_22)
- net AVI_RESET: now also J1.16 (Pin_16); no longer J1.40 (Pin_40)
- net CANH: now also J1.40 (Pin_40); no longer J1.33 (Pin_33)
- net CANL: now also J1.39 (Pin_39); no longer J1.35 (Pin_35)
- net EPS_RESET: now also J1.12 (Pin_12); no longer J1.38 (Pin_38)
- net GND: now also J1.10 (Pin_10), J1.3 (Pin_3), J1.31 (Pin_31), J1.32 (Pin_32), J1.35 (Pin_35), J1.37 (Pin_37), J1.38 (Pin_38), J1.4 (Pin_4); no longer J1.11 (Pin_11), J1.14 (Pin_14), J1.2 (Pin_2), J1.23 (Pin_23), J1.24 (Pin_24), J1.5 (Pin_5), J1.8 (Pin_8)
- net SPARE_1: now also J1.7 (Pin_7); no longer J1.25 (Pin_25)
- net SPARE_4: now also J1.36 (Pin_36); no longer J1.31 (Pin_31)
- net UART_A_RXI: now also J1.14 (Pin_14); no longer J1.39 (Pin_39)
- net UART_A_TXO: now also J1.13 (Pin_13); no longer J1.37 (Pin_37)
- net UART_B_CTS: now also J1.19 (Pin_19); no longer J1.34 (Pin_34)
- net UART_B_RTS: now also J1.15 (Pin_15); no longer J1.36 (Pin_36)
- net UART_B_RXI: now also J1.22 (Pin_22); no longer J1.32 (Pin_32)
- net UART_B_TXO: now also J1.21 (Pin_21); no longer J1.30 (Pin_30)
Changed lines of the file:
@@
 	1    0    0    -1
 $EndComp
-Text HLabel 5100 2875 0    50   Output ~ 0
+Text HLabel 6550 4075 2    50   Output ~ 0
 3V3_1
-Text HLabel 6550 4775 2    50   Output ~ 0
+Text HLabel 6550 3575 2    50   Output ~ 0
 AVI_RESET
-Text HLabel 5100 4475 0    50   BiDi ~ 0
+Text HLabel 6550 4775 2    50   BiDi ~ 0
 CANH
-Text HLabel 5100 4575 0    50   BiDi ~ 0
+Text HLabel 5100 4775 0    50   BiDi ~ 0
 CANL
-Text HLabel 5100 4675 0    50   Output ~ 0
+Text HLabel 5100 3475 0    50   Output ~ 0
 UART_A_TXO
-Text HLabel 5100 4775 0    50   Input ~ 0
+Text HLabel 6550 3475 2    50   Input ~ 0
 UART_A_RXI
 Wire Wire Line
@@
 Wire Wire Line
 	6075 3375 6550 3375
-Text HLabel 5100 3075 0    50   Output ~ 0
+Text HLabel 5100 2975 0    50   Output ~ 0
 GND
 Wire Wire Line
 	6075 3475 6550 3475
-Text HLabel 5100 3375 0    50   Output ~ 0
+Text HLabel 6550 4675 2    50   Output ~ 0
 GND
 Wire Wire Line
 	6075 3575 6550 3575
-Text HLabel 6550 2875 2    50   Output ~ 0
+Text HLabel 6550 4175 2    50   Output ~ 0
 GND
 Wire Wire Line
@@
 Text HLabel 5100 4275 0    50   Output ~ 0
 SPARE_3
-Text HLabel 5100 4075 0    50   Output ~ 0
+Text HLabel 5100 3175 0    50   Output ~ 0
 SPARE_1
 Wire Wire Line
@@
 Wire Wire Line
 	6075 3975 6550 3975
-Text HLabel 6550 3175 2    50   Output ~ 0
+Text HLabel 6550 3275 2    50   Output ~ 0
 GND
 Wire Wire Line
@@
 Wire Wire Line
 	6075 4375 6550 4375
-Text HLabel 6550 4675 2    50   Output ~ 0
+Text HLabel 6550 3375 2    50   Output ~ 0
 EPS_RESET
-Text HLabel 5100 2975 0    50   Output ~ 0
-3V3_2
-Text HLabel 5100 3175 0    50   Output ~ 0
+Text HLabel 5100 3375 0    50   Output ~ 0
 3V3_3
+Text HLabel 5100 3075 0    50   Output ~ 0
+3V3_4
+Text HLabel 6550 2875 2    50   Output ~ 0
+3V3_5
+Text HLabel 6550 3175 2    50   Output ~ 0
+3V3_7
+Text HLabel 5100 4075 0    50   Output ~ 0
+3V3_8
 Text HLabel 5100 3275 0    50   Output ~ 0
-3V3_4
-Text HLabel 5100 3475 0    50   Output ~ 0
-3V3_5
-Text HLabel 5100 3575 0    50   Output ~ 0
-3V3_6
-Text HLabel 6550 2975 2    50   Output ~ 0
-3V3_7
+3V3_9
 Text HLabel 6550 3075 2    50   Output ~ 0
-3V3_8
-Text HLabel 6550 3275 2    50   Output ~ 0
-3V3_9
-Text HLabel 6550 3375 2    50   Output ~ 0
 3V3_10
-Text HLabel 6550 3575 2    50   Output ~ 0
+Text HLabel 5100 2875 0    50   Output ~ 0
 3V3_11
 Text HLabel 6550 3675 2    50   Output ~ 0
 3V3_12
-Text HLabel 5100 3775 0    50   Output ~ 0
+Text HLabel 6550 4275 2    50   Output ~ 0
 5V0_1
-Text HLabel 5100 3875 0    50   Output ~ 0
+Text HLabel 6550 4475 2    50   Output ~ 0
 5V0_2
-Text HLabel 6550 3475 2    50   Output ~ 0
+Text HLabel 5100 4575 0    50   Output ~ 0
 GND
 Text HLabel 6550 3775 2    50   Output ~ 0
 GND
+Text HLabel 6550 4575 2    50   Output ~ 0
+SPARE_4
+Text HLabel 5100 3875 0    50   Output ~ 0
+UART_B_TXO
+Text HLabel 6550 3875 2    50   Input ~ 0
+UART_B_RXI
+Text HLabel 5100 4475 0    50   Output ~ 0
+5V0_2
 Text HLabel 5100 4375 0    50   Output ~ 0
-SPARE_4
-Text HLabel 6550 4275 2    50   Output ~ 0
-UART_B_TXO
-Text HLabel 6550 4375 2    50   Input ~ 0
-UART_B_RXI
-Text HLabel 6550 3875 2    50   Output ~ 0
-5V0_2
-Text HLabel 6550 4475 2    50   Input ~ 0
-UART_B_CTS
-Text HLabel 6550 4575 2    50   Output ~ 0
-UART_B_RTS
-Text HLabel 5100 3975 0    50   Output ~ 0
 GND
-Text HLabel 6550 3975 2    50   Output ~ 0
+Text HLabel 6550 4375 2    50   Output ~ 0
 GND
-Text HLabel 6550 4075 2    50   Output ~ 0
-SPARE_5
-Text HLabel 6550 4175 2    50   Output ~ 0
-SPARE_6
 Text Notes 4950 5225 0    50   ~ 0
 There are a lot of options that could work:\nhttps://www.digikey.com/short/znc31r
+Text HLabel 5100 3575 0    50   Output ~ 0
+UART_B_RTS
+Text HLabel 6550 3975 2    50   Output ~ 0
+3V3_2
+Text HLabel 5100 3775 0    50   Input ~ 0
+UART_B_CTS
+Text HLabel 5100 3975 0    50   Output ~ 0
+3V3_6
+Text HLabel 5100 4675 0    50   Output ~ 0
+GND
+Text HLabel 6550 2975 2    50   Output ~ 0
+GND
 $EndSCHEMATC

Commit message: Update Avionics part names to match KiCad update. Update Avionics board to use new interboard connector
Changed lines of the file:
@@
 $Descr A 11000 8500
 encoding utf-8
-Sheet 9 39
+Sheet 23 23
 Title "Current Monitor"
 Date "2020-05-25"
@@
 AR Path="/5EA31C93/631545C7/6310C580" Ref="J1"  Part="1"
 AR Path="/5FD3BACF/6310C580" Ref="J6"  Part="1"
-AR Path="/5EA31C93/639EBCB0/6310C580" Ref="J?"  Part="1"
-F 0 "J6" H 5825 4892 50  0000 C CNN
+AR Path="/5EA31C93/639EBCB0/6310C580" Ref="J1"  Part="1"
+F 0 "J1" H 5825 4892 50  0000 C CNN
 F 1 "Conn_02x20_Odd_Even" H 5825 4801 50  0000 C CNN
 F 2 "Connector_PinHeader_2.54mm:PinHeader_2x20_P2.54mm_Vertical" H 5775 3775 50  0001 C CNN
